Commit message: 3arm urdf model spawns in gazebo and rviz

File: open_manipulator_p/open_manipulator_p_description/urdf/open_manipulator_p.transmission.xacro (robot description, xacro)
@@ -2,11 +2,11 @@
 <robot xmlns:xacro="http://ros.org/wiki/xacro">
   <!-- Transmission macro -->
-  <xacro:macro name="SimpleTransmissionPosition" params="joint n">
-    <transmission name="tran${n}">
+  <xacro:macro name="SimpleTransmissionPosition" params="joint n id">
+    <transmission name="robot${id}/tran${n}">
       <type>transmission_interface/SimpleTransmission</type>
-      <joint name="${joint}">
+      <joint name="robot${id}/${joint}">
         <hardwareInterface>hardware_interface/PositionJointInterface</hardwareInterface>
       </joint>
-      <actuator name="motor${n}">
+      <actuator name="robot${id}/motor${n}">
         <mechanicalReduction>1</mechanicalReduction>
       </actuator>
@@ -14,11 +14,11 @@
   </xacro:macro>
   <!-- Transmission macro -->
-  <xacro:macro name="SimpleTransmissionEffort" params="joint n">
-    <transmission name="tran${n}">
+  <xacro:macro name="SimpleTransmissionEffort" params="joint n id">
+    <transmission name="robot${id}/tran${n}">
       <type>transmission_interface/SimpleTransmission</type>
-      <joint name="${joint}">
+      <joint name="robot${id}/${joint}">
         <hardwareInterface>hardware_interface/EffortJointInterface</hardwareInterface>
       </joint>
-      <actuator name="motor${n}">
+      <actuator name="robot${id}/motor${n}">
         <mechanicalReduction>1</mechanicalReduction>
       </actuator>
@@ -26,14 +26,26 @@
   </xacro:macro>
   <!-- Transmission 1 -->
-  <xacro:SimpleTransmissionPosition n="1" joint="joint1" />
+  <xacro:SimpleTransmissionPosition n="1" joint="joint1" id="1" />
+  <xacro:SimpleTransmissionPosition n="1" joint="joint1" id="2" />
+  <xacro:SimpleTransmissionPosition n="1" joint="joint1" id="3" />
   <!-- Transmission 2 -->
-  <xacro:SimpleTransmissionPosition n="2" joint="joint2" />
+  <xacro:SimpleTransmissionPosition n="2" joint="joint2" id="1" />
+  <xacro:SimpleTransmissionPosition n="2" joint="joint2" id="2" />
+  <xacro:SimpleTransmissionPosition n="2" joint="joint2" id="3" />
   <!-- Transmission 3 -->
-  <xacro:SimpleTransmissionPosition n="3" joint="joint3" />
+  <xacro:SimpleTransmissionPosition n="3" joint="joint3" id="1" />
+  <xacro:SimpleTransmissionPosition n="3" joint="joint3" id="2" />
+  <xacro:SimpleTransmissionPosition n="3" joint="joint3" id="3" />
   <!-- Transmission 4 -->
-  <xacro:SimpleTransmissionPosition n="4" joint="joint4" />
+  <xacro:SimpleTransmissionPosition n="4" joint="joint4" id="1" />
+  <xacro:SimpleTransmissionPosition n="4" joint="joint4" id="2" />
+  <xacro:SimpleTransmissionPosition n="4" joint="joint4" id="3" />
   <!-- Transmission 5 -->
-  <xacro:SimpleTransmissionPosition n="5" joint="joint5" />
+  <xacro:SimpleTransmissionPosition n="5" joint="joint5" id="1" />
+  <xacro:SimpleTransmissionPosition n="5" joint="joint5" id="2" />
+  <xacro:SimpleTransmissionPosition n="5" joint="joint5" id="3" />
   <!-- Transmission 6 -->
-  <xacro:SimpleTransmissionPosition n="6" joint="joint6" />
+  <xacro:SimpleTransmissionPosition n="6" joint="joint6" id="1" />
+  <xacro:SimpleTransmissionPosition n="6" joint="joint6" id="2" />
+  <xacro:SimpleTransmissionPosition n="6" joint="joint6" id="3" />
 </robot>

File: open_manipulator_p/open_manipulator_p_description/urdf/papras_group_moveit.urdf.xacro (robot description, xacro)
@@ -2,44 +2,28 @@
 <robot name="open_manipulator_p" xmlns:xacro="http://www.ros.org/wiki/xacro">
   <!-- Import Rviz colors -->
-  <xacro:include filename="$(find open_manipulator_p_description)/urdf/materials.xacro" />
+  <xacro:include filename="$(find open_manipulator_p_description)/urdf/materials.xacro"/>
   <!-- Import all Gazebo-customization elements, including Gazebo colors -->
-  <xacro:include filename="$(find open_manipulator_p_description)/urdf/open_manipulator_p.gazebo.xacro" />
+  <xacro:include filename="$(find open_manipulator_p_description)/urdf/open_manipulator_p.gazebo.xacro"/>
   <!-- Import Transmission -->
-  <xacro:include filename="$(find open_manipulator_p_description)/urdf/open_manipulator_p.transmission.xacro" />
+  <xacro:include filename="$(find open_manipulator_p_description)/urdf/open_manipulator_p.transmission.xacro"/>
   <xacro:arg name="base_offset" default ="0.046375"/>
-  <xacro:arg name="robot1_base_x" default="0"/>
-  <xacro:property name="robot1_base_x" value="0"/>
-  <xacro:arg name="robot1_base_y" default="0"/>
-  <xacro:property name="robot1_base_y" value="0"/>
-  <xacro:arg name="robot1_base_z" default="0"/>
-  <xacro:property name="robot1_base_z" value="0"/>
-  <xacro:arg name="robot2_base_x" default="0"/>
-  <xacro:property name="robot2_base_x" value="0.5"/>
-  <xacro:arg name="robot2_base_y" default="0"/>
-  <xacro:property name="robot2_base_y" value="0.5"/>
-  <xacro:arg name="robot2_base_z" default="0"/>
-  <xacro:property name="robot2_base_z" value="0"/>
-  <xacro:arg name="robot3_base_x" default="0"/>
-  <xacro:property name="robot3_base_x" value="1"/>
-  <xacro:arg name="robot3_base_y" default="0"/>
-  <xacro:property name="robot3_base_y" value="0"/>
-  <xacro:arg name="robot3_base_z" default="0"/>
-  <xacro:property name="robot3_base_z" value="0"/>
+  <xacro:arg name="robot1_base_x" default="-0.3"/>
+  <xacro:arg name="robot1_base_y" default="0.1"/>
+  <xacro:arg name="robot1_base_z" default="0.9"/>
+  <xacro:arg name="robot1_base_yaw" default="1.57"/>
+  <xacro:arg name="robot2_base_x" default="-0.3"/>
+  <xacro:arg name="robot2_base_y" default="-0.5"/>
+  <xacro:arg name="robot2_base_z" default="0.9"/>
+  <xacro:arg name="robot2_base_yaw" default="1.57"/>
+  <xacro:arg name="robot3_base_x" default="0.3"/>
+  <xacro:arg name="robot3_base_y" default="0.0"/>
+  <xacro:arg name="robot3_base_z" default="0.9"/>
+  <xacro:arg name="robot3_base_yaw" default="-1.57"/>
   <xacro:macro name="omp_arm" params="id">
-    <!-- <joint name="robot${prefix}/fixed" type="fixed">
-      <parent link="world"/>
-      <origin xyz="$(eval robot${prefix}_base_x) $(eval robot${prefix}_base_y) $(eval robot${prefix}_base_z-base_offset)"/>
-      <child link="robot${prefix}/base_link"/>
-    </joint>
-    <link name="robot${prefix}/floating_world_0"/>
-    <joint name="robot${prefix}/base_link_floating_world" type="fixed">
-      <parent link="robot${prefix}/base_link"/>
-      <origin xyz="0 0 ${base_offset}" />
-      <child link="robot${prefix}/floating_world_0"/>
-    </joint> -->
     <joint name="robot${id}/world_fixed" type="fixed">
         <parent link="world" />
         <child link="robot${id}/link1" />
-        <origin xyz="$(eval robot${id}_base_x) $(eval robot${id}_base_y) $(eval robot${id}_base_z-base_offset)"/>
+        <origin xyz="$(eval robot${id}_base_x) $(eval robot${id}_base_y) $(eval robot${id}_base_z-base_offset)"
+                rpy="0 0 $(eval robot${id}_base_yaw)"/>
     </joint>
     <!-- link 1 -->

Commit message: fixed vibrating arm issue and faster sim ratio

File: open_manipulator_p/open_manipulator_p_description/urdf/open_manipulator_p.transmission.xacro (robot description, xacro)
@@ -2,11 +2,11 @@
 <robot xmlns:xacro="http://ros.org/wiki/xacro">
   <!-- Transmission macro -->
-  <xacro:macro name="SimpleTransmissionPosition" params="joint n id">
-    <transmission name="robot${id}/tran${n}">
+  <xacro:macro name="SimpleTransmissionPosition" params="joint n">
+    <transmission name="tran${n}">
       <type>transmission_interface/SimpleTransmission</type>
-      <joint name="robot${id}/${joint}">
+      <joint name="${joint}">
         <hardwareInterface>hardware_interface/PositionJointInterface</hardwareInterface>
       </joint>
-      <actuator name="robot${id}/motor${n}">
+      <actuator name="motor${n}">
         <mechanicalReduction>1</mechanicalReduction>
       </actuator>
@@ -14,11 +14,11 @@
   </xacro:macro>
   <!-- Transmission macro -->
-  <xacro:macro name="SimpleTransmissionEffort" params="joint n id">
-    <transmission name="robot${id}/tran${n}">
+  <xacro:macro name="SimpleTransmissionEffort" params="joint n">
+    <transmission name="tran${n}">
       <type>transmission_interface/SimpleTransmission</type>
-      <joint name="robot${id}/${joint}">
+      <joint name="${joint}">
         <hardwareInterface>hardware_interface/EffortJointInterface</hardwareInterface>
       </joint>
-      <actuator name="robot${id}/motor${n}">
+      <actuator name="motor${n}">
         <mechanicalReduction>1</mechanicalReduction>
       </actuator>
@@ -26,26 +26,14 @@
   </xacro:macro>
   <!-- Transmission 1 -->
-  <xacro:SimpleTransmissionPosition n="1" joint="joint1" id="1" />
-  <xacro:SimpleTransmissionPosition n="1" joint="joint1" id="2" />
-  <xacro:SimpleTransmissionPosition n="1" joint="joint1" id="3" />
+  <xacro:SimpleTransmissionPosition n="1" joint="joint1" />
   <!-- Transmission 2 -->
-  <xacro:SimpleTransmissionPosition n="2" joint="joint2" id="1" />
-  <xacro:SimpleTransmissionPosition n="2" joint="joint2" id="2" />
-  <xacro:SimpleTransmissionPosition n="2" joint="joint2" id="3" />
+  <xacro:SimpleTransmissionPosition n="2" joint="joint2" />
   <!-- Transmission 3 -->
-  <xacro:SimpleTransmissionPosition n="3" joint="joint3" id="1" />
-  <xacro:SimpleTransmissionPosition n="3" joint="joint3" id="2" />
-  <xacro:SimpleTransmissionPosition n="3" joint="joint3" id="3" />
+  <xacro:SimpleTransmissionPosition n="3" joint="joint3" />
   <!-- Transmission 4 -->
-  <xacro:SimpleTransmissionPosition n="4" joint="joint4" id="1" />
-  <xacro:SimpleTransmissionPosition n="4" joint="joint4" id="2" />
-  <xacro:SimpleTransmissionPosition n="4" joint="joint4" id="3" />
+  <xacro:SimpleTransmissionPosition n="4" joint="joint4" />
   <!-- Transmission 5 -->
-  <xacro:SimpleTransmissionPosition n="5" joint="joint5" id="1" />
-  <xacro:SimpleTransmissionPosition n="5" joint="joint5" id="2" />
-  <xacro:SimpleTransmissionPosition n="5" joint="joint5" id="3" />
+  <xacro:SimpleTransmissionPosition n="5" joint="joint5" />
   <!-- Transmission 6 -->
-  <xacro:SimpleTransmissionPosition n="6" joint="joint6" id="1" />
-  <xacro:SimpleTransmissionPosition n="6" joint="joint6" id="2" />
-  <xacro:SimpleTransmissionPosition n="6" joint="joint6" id="3" />
+  <xacro:SimpleTransmissionPosition n="6" joint="joint6" />
 </robot>

File: open_manipulator_p/open_manipulator_p_description/urdf/papras_group_moveit.urdf.xacro (robot description, xacro)
@@ -6,17 +6,17 @@
   <xacro:include filename="$(find open_manipulator_p_description)/urdf/open_manipulator_p.gazebo.xacro"/>
   <!-- Import Transmission -->
-  <xacro:include filename="$(find open_manipulator_p_description)/urdf/open_manipulator_p.transmission.xacro"/>
+  <xacro:include filename="$(find open_manipulator_p_description)/urdf/3arm_moveit.transmission.xacro"/>
   <xacro:arg name="base_offset" default ="0.046375"/>
   <xacro:arg name="robot1_base_x" default="-0.3"/>
   <xacro:arg name="robot1_base_y" default="0.1"/>
-  <xacro:arg name="robot1_base_z" default="0.9"/>
+  <xacro:arg name="robot1_base_z" default="1.1"/>
   <xacro:arg name="robot1_base_yaw" default="1.57"/>
   <xacro:arg name="robot2_base_x" default="-0.3"/>
   <xacro:arg name="robot2_base_y" default="-0.5"/>
-  <xacro:arg name="robot2_base_z" default="0.9"/>
+  <xacro:arg name="robot2_base_z" default="1.1"/>
   <xacro:arg name="robot2_base_yaw" default="1.57"/>
   <xacro:arg name="robot3_base_x" default="0.3"/>
   <xacro:arg name="robot3_base_y" default="0.0"/>
-  <xacro:arg name="robot3_base_z" default="0.9"/>
+  <xacro:arg name="robot3_base_z" default="1.1"/>
   <xacro:arg name="robot3_base_yaw" default="-1.57"/>
   <xacro:macro name="omp_arm" params="id">
