Commit message: coffee demo working on hardware with gripper using moveit planner :) (#12)
* one arm correct joint states on rviz

* increased joint 2 lower limit for disabled pose

* set joint 4 limit in omp.cpp, arm3 moveit control

* initial cup_demo code+package

* set joint 4 limit in omp.cpp, arm3 moveit control pt2

* new rviz config

* generic task pose fails

* moveit gripper pkg, gripper not closing

* cartesian poses still fail

* cup_demo arm1 moves

* arm 1 no gripper

* cup_demo works on sim without gripper

* gripper working on moveit, gripper 111 not communicating

* issue with multiple hw controllers due to same node name

* hardware single arm group control on all arms using single u2d2, w/o gripper

Co-authored-by: Dhruv Mathur <dmathur2@illinois.edu>

File: open_manipulator_p/open_manipulator_p_description/urdf/papras_group_moveit_gazebo.urdf (robot description, URDF)
Before this commit: robot open_manipulator_p, 23 links, 22 joints
Joints:
- joint robot1/joint2: limit lower=-1.5707963267948966 upper=1.5707963267948966 effort=1000 velocity=6.5 -> lower=-2.0 upper=1.5707963267948966 effort=1000 velocity=6.5
- joint robot2/joint2: limit lower=-1.5707963267948966 upper=1.5707963267948966 effort=1000 velocity=6.5 -> lower=-2.0 upper=1.5707963267948966 effort=1000 velocity=6.5
- joint robot3/joint2: limit lower=-1.5707963267948966 upper=1.5707963267948966 effort=1000 velocity=6.5 -> lower=-2.0 upper=1.5707963267948966 effort=1000 velocity=6.5

File: open_manipulator_p/open_manipulator_p_description/urdf/papras_group_moveit_with_gripper.urdf.xacro (robot description, xacro)
@@ -6,5 +6,5 @@
   <xacro:include filename="$(find open_manipulator_p_description)/urdf/open_manipulator_p.gazebo.xacro"/>
   <!-- Import Transmission -->
-  <xacro:include filename="$(find open_manipulator_p_description)/urdf/3arm_moveit.transmission.xacro"/>
+  <xacro:include filename="$(find open_manipulator_p_description)/urdf/3arm_moveit_with_gripper.transmission.xacro"/>
   <xacro:arg name="robot1_base_x" default="-0.3795"/>
   <xacro:arg name="robot1_base_y" default="0.0435"/>
@@ -237,4 +237,122 @@
         <inertia ixx="1.0" ixy="0.0" ixz="0.0" iyy="1.0" iyz="0.0" izz="1.0" />
         <!--<inertia ixx="0.00000938" ixy="0.0" ixz="0.0" iyy="0.00000338" iyz="0.0" izz="0.00000635" />-->
+      </inertial>
+    </link>
+     <!-- gripper main fixed joint-->
+    <joint name="robot${id}/end_link_fixed" type="fixed">
+      <parent link="robot${id}/end_link"/>
+      <child link="robot${id}/gripper_main_link"/>
+      <origin xyz="0.007 0.0 0.0" rpy="0 0 0" />
+    </joint>
+    <!-- gripper main link -->
+    <link name="robot${id}/gripper_main_link">
+      <visual>
+        <origin xyz="0 0 0" rpy="0 0 0" />
+        <geometry>
+          <mesh filename="package://open_manipulator_p_description/meshes/gripper_main_link.stl" scale="0.001 0.001 0.001"/>
+        </geometry>
+        <material name="grey"/>
+      </visual>
+      <collision>
+        <origin xyz="0 0 0" rpy="0 0 0" />
+        <geometry>
+          <mesh filename="package://open_manipulator_p_description/meshes/gripper_main_link.stl" scale="0.001 0.001 0.001"/>
+        </geometry>
+      </collision>
+      <inertial>
+        <origin xyz="0.0 0.0 0.0" rpy="0 0 0"/>
+        <mass value="0.509"/>
+        <inertia ixx="1.0" ixy="0.0" ixz="0.0" iyy="1.0" iyz="0.0" izz="1.0" />
+      </inertial>
+    </link>
+    <!-- gripper joint -->
+    <joint name="robot${id}/gripper" type="revolute">
+      <axis xyz="0 0 1" />
+      <origin xyz="0.0552 -0.0400 0" rpy="0 0 -0.4"/>
+      <parent link="robot${id}/gripper_main_link"/>
+      <child link="robot${id}/gripper_link"/>
+      <limit velocity="6.5" effort="1000" lower="0.0" upper="1.1" />
+      <dynamics damping="0.1" friction="0.0" />
+    </joint>
+    <!-- gripper link -->
+    <link name="robot${id}/gripper_link">
+      <visual>
+        <origin xyz="0 0 0" rpy="0 0 0" />
+        <geometry>
+          <mesh filename="package://open_manipulator_p_description/meshes/gripper_link.stl" scale="0.001 0.001 0.001"/>
+        </geometry>
+        <material name="grey"/>
+      </visual>
+      <collision>
+        <origin xyz="0 0 0" rpy="0 0 0" />
+        <geometry>
+          <mesh filename="package://open_manipulator_p_description/meshes/gripper_link.stl" scale="0.001 0.001 0.001"/>
+        </geometry>
+        <material name="grey"/>
+      </collision>
+      <inertial>
+        <origin xyz="0 0 0" rpy="0 0 0"/>
+        <mass value="0.013"/>
+        <inertia ixx="1.0" ixy="0.0" ixz="0.0" iyy="1.0" iyz="0.0" izz="1.0" />
+      </inertial>
+    </link>
+    <!-- gripper joint 1 -->
+    <joint name="robot${id}/gripper_sub" type="revolute">
+      <axis xyz="0 0 -1" />
+      <origin xyz="0.0552 0.0400 0" rpy="0 0 0.4"/>
+      <parent link="robot${id}/gripper_main_link"/>
+      <child link="robot${id}/gripper_sub_link"/>
+      <limit velocity="6.5" effort="1000" lower="0.0" upper="1.1" />
+      <dynamics damping="0.1" friction="0.0" />
+      <mimic joint="robot${id}/gripper" multiplier="1"/>
+    </joint>
+    <!-- gripper 1 link -->
+    <link name="robot${id}/gripper_sub_link">
+      <visual>
+        <origin xyz="0 0 0" rpy="0 0 0" />
+        <geometry>
+          <mesh filename="package://open_manipulator_p_description/meshes/gripper_sub_link.stl" scale="0.001 0.001 0.001"/>
+        </geometry>
+        <material name="grey"/>
+      </visual>
+      <collision>
+        <origin xyz="0 0 0" rpy="0 0 0" />
+        <geometry>
+          <mesh filename="package://open_manipulator_p_description/meshes/gripper_sub_link.stl" scale="0.001 0.001 0.001"/>
+        </geometry>
+        <material name="grey"/>
+      </collision>
+      <inertial>
+        <origin xyz="0 0 0" rpy="0 0 0"/>
+        <mass value="0.013"/>
+        <inertia ixx="1.0" ixy="0.0" ixz="0.0" iyy="1.0" iyz="0.0" izz="1.0" />
+      </inertial>
+    </link>
+    <!-- gripper main fixed joint-->
+    <joint name="robot${id}/end_effector_joint" type="fixed">
+      <parent link="robot${id}/gripper_main_link"/>
+      <child link="robot${id}/end_effector_link"/>
+      <origin xyz="0.14 0.0 0.0" rpy="0 0 0" />
+    </joint>
+    <!-- End Effector -->
+    <link name="robot${id}/end_effector_link">
+      <visual>
+        <origin xyz="0.0 0.0 0.0" rpy="0 0 0" />
+        <geometry>
+          <box size = "0.01 0.01 0.01"/>
+        </geometry>
+        <material name="red"/>
+      </visual>
+      <collision>
+        <origin xyz="0.0 0.0 0.0" rpy="0 0 0" />
+        <geometry>
+          <box size = "0.01 0.01 0.01"/>
+        </geometry>
+        <material name="red"/>
+      </collision>
+      <inertial>
+        <origin xyz="0.0 0.0 0.0" rpy="0 0 0" />
+        <mass value="0.001" />
+        <inertia ixx="1.0" ixy="0.0" ixz="0.0" iyy="1.0" iyz="0.0" izz="1.0" />
       </inertial>
     </link>
