Commit message: simplified collision meshes in URDF for faster collision detection (#9)

File: open_manipulator_p/open_manipulator_p_description/urdf/papras_group_moveit.urdf.xacro (robot description, xacro)
@@ -101,5 +101,5 @@
         <origin xyz="0.067 0.008 -0.019" rpy="0 0 3.14"/>
         <geometry>
-          <mesh filename="package://open_manipulator_p_description/meshes/link3_papras.stl" scale="0.001 0.001 0.001"/>
+          <mesh filename="package://open_manipulator_p_description/meshes/link3_papras_simple.stl" scale="0.001 0.001 0.001"/>
         </geometry>
       </collision>
@@ -133,5 +133,5 @@
         <origin xyz="0.227 0.0085 -0.024" rpy="0 0 3.14"/>
         <geometry>
-          <mesh filename="package://open_manipulator_p_description/meshes/link4_papras.stl" scale="0.001 0.001 0.001"/>
+          <mesh filename="package://open_manipulator_p_description/meshes/link4_papras_simple.stl" scale="0.001 0.001 0.001"/>
         </geometry>
       </collision>
@@ -197,5 +197,5 @@
         <origin xyz="-0.034 -0.098 -0.028" rpy="0 0 0"/>
         <geometry>
-          <mesh filename="package://open_manipulator_p_description/meshes/link6_papras.stl" scale="0.001 0.001 0.001"/>
+          <mesh filename="package://open_manipulator_p_description/meshes/link6_papras_simple.stl" scale="0.001 0.001 0.001"/>
         </geometry>
       </collision>

Commit message: full 2arm coffee demo with props (#37)
* move cup_demo script into papras_gazebo pkg

* cup_demo with pose goals in sim

* fix moveit_config_w_gripper config/launch files #30

* more fixes for #30

* #31: Modularized arm movements

* script based gripper control (modularized per #31)

* script based modular arm and gripper control on hardware (#31, #32)

* coffee demo mission plan yaml file

* testing kettle moves in sim

* added dripper and cup moves

* update yaml file configuration (#35)

* script based control via YAML file (#35)

* 2arm demo complete

* change commands from script to yaml

Co-authored-by: Dhruv Mathur <dmathur2@illinois.edu>

File: open_manipulator_p/open_manipulator_p_description/urdf/papras_group_moveit.urdf.xacro (robot description, xacro)
@@ -54,5 +54,5 @@
       <origin xyz="0.0 0.0 0.126" rpy="0 0 0"/>
       <axis xyz="0 0 1"/>
-      <limit velocity="6.5" effort="1000" lower="${-pi*0.5}" upper="${pi*0.5}" />
+      <limit velocity="6.5" effort="1000" lower="${-pi*1.0}" upper="${pi*1.0}" />
       <dynamics damping="0.7"/>
     </joint>
@@ -86,5 +86,5 @@
       <origin xyz="0.0 0.069 0.033" rpy="0 0 0"/>
       <axis xyz="0 1 0"/>
-      <limit velocity="6.5" effort="1000" lower="-2.0" upper="${pi*0.5}" />
+      <limit velocity="6.5" effort="1000" lower="-2.0" upper="${pi*1.0}" />
       <dynamics damping="0.7"/>
     </joint>
@@ -118,5 +118,5 @@
       <origin xyz="0.03000 -0.01150 0.26400" rpy="0 0 0"/>
       <axis xyz="0 1 0"/>
-      <limit velocity="6.5" effort="1000" lower="${-pi*0.5}" upper="${pi*0.5}" />
+      <limit velocity="6.5" effort="1000" lower="${-pi*1.0}" upper="${pi*1.0}" />
       <dynamics damping="0.7"/>
     </joint>
@@ -150,5 +150,5 @@
       <origin xyz="0.19500 -0.05750 0.03000" rpy="0 0 0"/>
       <axis xyz="1 0 0"/>
-      <limit velocity="6.5" effort="1000" lower="${-pi*0.5}" upper="${pi*0.5}" />
+      <limit velocity="6.5" effort="1000" lower="${-pi*0.875}" upper="${pi*0.875}" />
       <dynamics damping="0.7"/>
     </joint>
@@ -182,5 +182,5 @@
       <origin xyz="0.06300 0.04500 0.00000" rpy="0 0 0"/>
       <axis xyz="0 1 0"/>
-      <limit velocity="6.5" effort="1000" lower="${-pi*0.5}" upper="${pi*0.5}" />
+      <limit velocity="6.5" effort="1000" lower="${-pi*1.0}" upper="${pi*1.0}" />
       <dynamics damping="0.7"/>
     </joint>
@@ -214,5 +214,5 @@
       <origin xyz="0.12300 -0.04500 0.00000" rpy="0 0 0"/>
       <axis xyz="1 0 0"/>
-      <limit velocity="6.5" effort="1000" lower="${-pi*0.5}" upper="${pi*0.5}" />
+      <limit velocity="6.5" effort="1000" lower="${-pi*1.0}" upper="${pi*1.0}" />
       <dynamics damping="0.7"/>
     </joint>

File: open_manipulator_p/open_manipulator_p_description/urdf/papras_group_moveit_with_gripper.urdf.xacro (robot description, xacro)
@@ -14,5 +14,5 @@
   <xacro:arg name="robot2_base_y" default="-0.5545"/>
   <xacro:arg name="robot2_base_z" default="$(eval 0.77-0.084)"/>
-  <xacro:arg name="robot2_base_yaw" default="1.57"/>
+  <xacro:arg name="robot2_base_yaw" default="3.14"/>
   <xacro:arg name="robot3_base_x" default="0.3735"/>
   <xacro:arg name="robot3_base_y" default="-0.2535"/>
@@ -54,5 +54,5 @@
       <origin xyz="0.0 0.0 0.126" rpy="0 0 0"/>
       <axis xyz="0 0 1"/>
-      <limit velocity="6.5" effort="1000" lower="${-pi*0.5}" upper="${pi*0.5}" />
+      <limit velocity="6.5" effort="1000" lower="${-pi*1.0}" upper="${pi*1.0}" />
       <dynamics damping="0.7"/>
     </joint>
@@ -86,5 +86,5 @@
       <origin xyz="0.0 0.069 0.033" rpy="0 0 0"/>
       <axis xyz="0 1 0"/>
-      <limit velocity="6.5" effort="1000" lower="-2.0" upper="${pi*0.5}" />
+      <limit velocity="6.5" effort="1000" lower="-2.0" upper="${pi*1.0}" />
       <dynamics damping="0.7"/>
     </joint>
@@ -118,5 +118,5 @@
       <origin xyz="0.03000 -0.01150 0.26400" rpy="0 0 0"/>
       <axis xyz="0 1 0"/>
-      <limit velocity="6.5" effort="1000" lower="${-pi*0.5}" upper="${pi*0.5}" />
+      <limit velocity="6.5" effort="1000" lower="${-pi*1.0}" upper="${pi*1.0}" />
       <dynamics damping="0.7"/>
     </joint>
@@ -150,5 +150,5 @@
       <origin xyz="0.19500 -0.05750 0.03000" rpy="0 0 0"/>
       <axis xyz="1 0 0"/>
-      <limit velocity="6.5" effort="1000" lower="${-pi*0.5}" upper="${pi*0.5}" />
+      <limit velocity="6.5" effort="1000" lower="${-pi*0.875}" upper="${pi*0.875}" />
       <dynamics damping="0.7"/>
     </joint>
@@ -182,5 +182,5 @@
       <origin xyz="0.06300 0.04500 0.00000" rpy="0 0 0"/>
       <axis xyz="0 1 0"/>
-      <limit velocity="6.5" effort="1000" lower="${-pi*0.5}" upper="${pi*0.5}" />
+      <limit velocity="6.5" effort="1000" lower="${-pi*1.0}" upper="${pi*1.0}" />
       <dynamics damping="0.7"/>
     </joint>
@@ -214,5 +214,5 @@
       <origin xyz="0.12300 -0.04500 0.00000" rpy="0 0 0"/>
       <axis xyz="1 0 0"/>
-      <limit velocity="6.5" effort="1000" lower="${-pi*0.5}" upper="${pi*0.5}" />
+      <limit velocity="6.5" effort="1000" lower="${-pi*1.0}" upper="${pi*1.0}" />
       <dynamics damping="0.7"/>
     </joint>
