Commit message: bare-bones 2 arm stand urdf and launch file (#24) (#43)

File: open_manipulator_p/open_manipulator_p_description/urdf/2arm_stand_with_gripper.urdf.xacro (robot description, xacro)
@@ -4,25 +4,25 @@
   <xacro:include filename="$(find open_manipulator_p_description)/urdf/materials.xacro"/>
   <!-- Import all Gazebo-customization elements, including Gazebo colors -->
-  <xacro:include filename="$(find open_manipulator_p_description)/urdf/3arm_moveit.gazebo.xacro"/>
+  <xacro:include filename="$(find open_manipulator_p_description)/urdf/2arm_stand.gazebo.xacro"/>
   <!-- Import Transmission -->
-  <xacro:include filename="$(find open_manipulator_p_description)/urdf/3arm_moveit_with_gripper.transmission.xacro"/>
-  <xacro:arg name="robot1_base_x" default="-0.3795"/>
-  <xacro:arg name="robot1_base_y" default="0.0435"/>
-  <xacro:arg name="robot1_base_z" default="$(eval 0.77-0.084)"/>
-  <xacro:arg name="robot1_base_yaw" default="1.57"/>
-  <xacro:arg name="robot2_base_x" default="-0.3835"/>
-  <xacro:arg name="robot2_base_y" default="-0.5545"/>
-  <xacro:arg name="robot2_base_z" default="$(eval 0.77-0.084)"/>
-  <xacro:arg name="robot2_base_yaw" default="3.14"/>
-  <xacro:arg name="robot3_base_x" default="0.3735"/>
-  <xacro:arg name="robot3_base_y" default="-0.2535"/>
-  <xacro:arg name="robot3_base_z" default="$(eval 0.77-0.084)"/>
-  <xacro:arg name="robot3_base_yaw" default="-1.57"/>
+  <xacro:include filename="$(find open_manipulator_p_description)/urdf/2arm_stand_with_gripper.transmission.xacro"/>
+  <xacro:arg name="robotleft_base_x" default="0.0"/>
+  <xacro:arg name="robotleft_base_y" default="0.0565"/>
+  <xacro:arg name="robotleft_base_z" default="1.661"/>
+  <xacro:arg name="robotleft_base_roll" default="-1.571"/>
+  <xacro:arg name="robotleft_base_pitch" default="-1.571"/>
+  <xacro:arg name="robotleft_base_yaw" default="0.0"/>
+  <xacro:arg name="robotright_base_x" default="0.0"/>
+  <xacro:arg name="robotright_base_y" default="-0.0565"/>
+  <xacro:arg name="robotright_base_z" default="1.661"/>
+  <xacro:arg name="robotright_base_roll" default="1.571"/>
+  <xacro:arg name="robotright_base_pitch" default="-1.571"/>
+  <xacro:arg name="robotright_base_yaw" default="0.0"/>
   <xacro:macro name="omp_arm" params="id">
-    <joint name="robot${id}/arm_desk_fixed" type="fixed">
-        <parent link="papras_desk" />
+    <joint name="robot${id}/world_fixed" type="fixed">
+        <parent link="world" />
         <child link="robot${id}/link1" />
         <origin xyz="$(eval robot${id}_base_x) $(eval robot${id}_base_y) $(eval robot${id}_base_z)"
-                rpy="0 0 $(eval robot${id}_base_yaw)"/>
+                rpy="$(eval robot${id}_base_roll) $(eval robot${id}_base_pitch) $(eval robot${id}_base_yaw)"/>
     </joint>
     <!-- link 1 -->
@@ -358,28 +358,8 @@
     </link>
   </xacro:macro>
-  <!-- World with PAPRAS Desk-->
+  <!-- World without stand-->
   <link name="world"/>
-  <joint name="desk_world_fixed" type="fixed">
-      <parent link="world" />
-      <child link="papras_desk" />
-      <origin xyz="0 0 0" rpy="0 0 0"/>
-  </joint>
-  <link name="papras_desk">
-    <visual>
-      <origin xyz="0.0 0.0 0.77" rpy="0 0 0" />
-      <geometry>
-        <mesh filename="package://open_manipulator_p_description/meshes/desk.stl"/>
-      </geometry>
-    </visual>
-    <collision>
-      <origin xyz="0.0 0.0 0.77" rpy="0 0 0" />
-      <geometry>
-        <mesh filename="package://open_manipulator_p_description/meshes/desk.stl"/>
-      </geometry>
-    </collision>
-  </link>
   <!-- Arms -->
-  <xacro:omp_arm id="1"/>
-  <xacro:omp_arm id="2"/>
-  <xacro:omp_arm id="3"/>
+  <xacro:omp_arm id="left"/>
+  <xacro:omp_arm id="right"/>
 </robot>

File: open_manipulator_p/open_manipulator_p_description/urdf/papras_group_moveit.urdf.xacro (robot description, xacro)
@@ -4,5 +4,5 @@
   <xacro:include filename="$(find open_manipulator_p_description)/urdf/materials.xacro"/>
   <!-- Import all Gazebo-customization elements, including Gazebo colors -->
-  <xacro:include filename="$(find open_manipulator_p_description)/urdf/open_manipulator_p.gazebo.xacro"/>
+  <xacro:include filename="$(find open_manipulator_p_description)/urdf/3arm_moveit.gazebo.xacro"/>
   <!-- Import Transmission -->
   <xacro:include filename="$(find open_manipulator_p_description)/urdf/3arm_moveit.transmission.xacro"/>

Commit message: Remeasured hardware joint limits

File: open_manipulator_p/open_manipulator_p_description/urdf/2arm_stand_with_gripper.urdf.xacro (robot description, xacro)
@@ -86,5 +86,5 @@
       <origin xyz="0.0 0.069 0.033" rpy="0 0 0"/>
       <axis xyz="0 1 0"/>
-      <limit velocity="6.5" effort="1000" lower="-2.0" upper="${pi*1.0}" />
+      <limit velocity="6.5" effort="1000" lower="-2.0" upper="2.0" />
       <dynamics damping="0.7"/>
     </joint>
@@ -118,5 +118,5 @@
       <origin xyz="0.03000 -0.01150 0.26400" rpy="0 0 0"/>
       <axis xyz="0 1 0"/>
-      <limit velocity="6.5" effort="1000" lower="${-pi*1.0}" upper="${pi*1.0}" />
+      <limit velocity="6.5" effort="1000" lower="${-pi*1.0}" upper="${pi*0.5}" />
       <dynamics damping="0.7"/>
     </joint>
@@ -182,5 +182,5 @@
       <origin xyz="0.06300 0.04500 0.00000" rpy="0 0 0"/>
       <axis xyz="0 1 0"/>
-      <limit velocity="6.5" effort="1000" lower="${-pi*1.0}" upper="${pi*1.0}" />
+      <limit velocity="6.5" effort="1000" lower="${-pi*0.5}" upper="${pi*0.5}" />
       <dynamics damping="0.7"/>
     </joint>

File: open_manipulator_p/open_manipulator_p_description/urdf/open_manipulator_p.urdf.xacro (robot description, xacro)
@@ -29,5 +29,5 @@
     <origin xyz="0.0 0.0 0.126" rpy="0 0 0"/>
     <axis xyz="0 0 1"/>
-    <limit velocity="6.5" effort="1000" lower="${-pi*0.5}" upper="${pi*0.5}" />
+    <limit velocity="6.5" effort="1000" lower="${-pi*1.0}" upper="${pi*1.0}" />
     <dynamics damping="0.7"/>
   </joint>
@@ -61,5 +61,5 @@
     <origin xyz="0.0 0.069 0.033" rpy="0 0 0"/>
     <axis xyz="0 1 0"/>
-    <limit velocity="6.5" effort="1000" lower="${-pi*0.5}" upper="${pi*0.5}" />
+    <limit velocity="6.5" effort="1000" lower="$-2.0" upper="$2.0" />
     <dynamics damping="0.7"/>
   </joint>
@@ -93,5 +93,5 @@
     <origin xyz="0.03000 -0.01150 0.26400" rpy="0 0 0"/>
     <axis xyz="0 1 0"/>
-    <limit velocity="6.5" effort="1000" lower="${-pi*0.5}" upper="${pi*0.5}" />
+    <limit velocity="6.5" effort="1000" lower="${-pi*1.0}" upper="${pi*0.5}" />
     <dynamics damping="0.7"/>
   </joint>
@@ -125,5 +125,5 @@
     <origin xyz="0.19500 -0.05750 0.03000" rpy="0 0 0"/>
     <axis xyz="1 0 0"/>
-    <limit velocity="6.5" effort="1000" lower="${-pi*0.5}" upper="${pi*0.5}" />
+    <limit velocity="6.5" effort="1000" lower="${-pi*0.875}" upper="${pi*0.875}" />
     <dynamics damping="0.7"/>
   </joint>
@@ -189,5 +189,5 @@
     <origin xyz="0.12300 -0.04500 0.00000" rpy="0 0 0"/>
     <axis xyz="1 0 0"/>
-    <limit velocity="6.5" effort="1000" lower="${-pi*0.5}" upper="${pi*0.5}" />
+    <limit velocity="6.5" effort="1000" lower="${-pi*1.0}" upper="${pi*1.0}" />
     <dynamics damping="0.7"/>
   </joint>

File: open_manipulator_p/open_manipulator_p_description/urdf/open_manipulator_p_with_gripper.urdf.xacro (robot description, xacro)
@@ -29,5 +29,5 @@
     <origin xyz="0.0 0.0 0.126" rpy="0 0 0"/>
     <axis xyz="0 0 1"/>
-    <limit velocity="6.5" effort="1000" lower="${-pi*0.5}" upper="${pi*0.5}" />
+    <limit velocity="6.5" effort="1000" lower="${-pi*1.0}" upper="${pi*1.0}" />
     <dynamics damping="0.7"/>
   </joint>
@@ -61,5 +61,5 @@
     <origin xyz="0.0 0.069 0.033" rpy="0 0 0"/>
     <axis xyz="0 1 0"/>
-    <limit velocity="6.5" effort="1000" lower="${-pi*0.5}" upper="${pi*0.5}" />
+    <limit velocity="6.5" effort="1000" lower="-2.0" upper="2.0" />
     <dynamics damping="0.7"/>
   </joint>
@@ -93,5 +93,5 @@
     <origin xyz="0.03000 -0.01150 0.26400" rpy="0 0 0"/>
     <axis xyz="0 1 0"/>
-    <limit velocity="6.5" effort="1000" lower="${-pi*0.5}" upper="${pi*0.5}" />
+    <limit velocity="6.5" effort="1000" lower="${-pi*1.0}" upper="${pi*0.5}" />
     <dynamics damping="0.7"/>
   </joint>
@@ -125,5 +125,5 @@
     <origin xyz="0.19500 -0.05750 0.03000" rpy="0 0 0"/>
     <axis xyz="1 0 0"/>
-    <limit velocity="6.5" effort="1000" lower="${-pi*0.5}" upper="${pi*0.5}" />
+    <limit velocity="6.5" effort="1000" lower="${-pi*0.875}" upper="${pi*0.875}" />
     <dynamics damping="0.7"/>
   </joint>
@@ -189,5 +189,5 @@
     <origin xyz="0.12300 -0.04500 0.00000" rpy="0 0 0"/>
     <axis xyz="1 0 0"/>
-    <limit velocity="6.5" effort="1000" lower="${-pi*0.5}" upper="${pi*0.5}" />
+    <limit velocity="6.5" effort="1000" lower="${-pi*1.0}" upper="${pi*1.0}" />
     <dynamics damping="0.7"/>
   </joint>

File: open_manipulator_p/open_manipulator_p_description/urdf/papras_group_moveit.urdf.xacro (robot description, xacro)
@@ -86,5 +86,5 @@
       <origin xyz="0.0 0.069 0.033" rpy="0 0 0"/>
       <axis xyz="0 1 0"/>
-      <limit velocity="6.5" effort="1000" lower="-2.0" upper="${pi*1.0}" />
+      <limit velocity="6.5" effort="1000" lower="-2.0" upper="2.0" />
       <dynamics damping="0.7"/>
     </joint>
@@ -118,5 +118,5 @@
       <origin xyz="0.03000 -0.01150 0.26400" rpy="0 0 0"/>
       <axis xyz="0 1 0"/>
-      <limit velocity="6.5" effort="1000" lower="${-pi*1.0}" upper="${pi*1.0}" />
+      <limit velocity="6.5" effort="1000" lower="${-pi*1.0}" upper="${pi*0.5}" />
       <dynamics damping="0.7"/>
     </joint>
@@ -182,5 +182,5 @@
       <origin xyz="0.06300 0.04500 0.00000" rpy="0 0 0"/>
       <axis xyz="0 1 0"/>
-      <limit velocity="6.5" effort="1000" lower="${-pi*1.0}" upper="${pi*1.0}" />
+      <limit velocity="6.5" effort="1000" lower="${-pi*0.5}" upper="${pi*0.5}" />
       <dynamics damping="0.7"/>
     </joint>

File: open_manipulator_p/open_manipulator_p_description/urdf/papras_group_moveit_with_gripper.urdf.xacro (robot description, xacro)
@@ -86,5 +86,5 @@
       <origin xyz="0.0 0.069 0.033" rpy="0 0 0"/>
       <axis xyz="0 1 0"/>
-      <limit velocity="6.5" effort="1000" lower="-2.0" upper="${pi*1.0}" />
+      <limit velocity="6.5" effort="1000" lower="-2.0" upper="2.0" />
       <dynamics damping="0.7"/>
     </joint>
@@ -118,5 +118,5 @@
       <origin xyz="0.03000 -0.01150 0.26400" rpy="0 0 0"/>
       <axis xyz="0 1 0"/>
-      <limit velocity="6.5" effort="1000" lower="${-pi*1.0}" upper="${pi*1.0}" />
+      <limit velocity="6.5" effort="1000" lower="${-pi*1.0}" upper="${pi*0.5}" />
       <dynamics damping="0.7"/>
     </joint>
@@ -182,5 +182,5 @@
       <origin xyz="0.06300 0.04500 0.00000" rpy="0 0 0"/>
       <axis xyz="0 1 0"/>
-      <limit velocity="6.5" effort="1000" lower="${-pi*1.0}" upper="${pi*1.0}" />
+      <limit velocity="6.5" effort="1000" lower="${-pi*0.5}" upper="${pi*0.5}" />
       <dynamics damping="0.7"/>
     </joint>
