Commit message: Update urdf stl (#3)
* update original urdf with gripper

* update original urdf without gripper

* update 3arm urdf

File: open_manipulator_p/open_manipulator_p_description/urdf/open_manipulator_p.urdf.xacro (robot description, xacro)
@@ -67,14 +67,14 @@
   <link name="link3">
     <visual>
-      <origin xyz="0 0 0" rpy="0 0 0"/>
-      <geometry>
-        <mesh filename="package://open_manipulator_p_description/meshes/link3.stl" scale="0.001 0.001 0.001"/>
-      </geometry>
-      <material name="grey"/>
-    </visual>
-    <collision>
-      <origin xyz="0 0 0" rpy="0 0 0"/>
-      <geometry>
-        <mesh filename="package://open_manipulator_p_description/meshes/link3.stl" scale="0.001 0.001 0.001"/>
+      <origin xyz="0.067 0.008 -0.019" rpy="0 0 3.14"/>
+      <geometry>
+        <mesh filename="package://open_manipulator_p_description/meshes/link3_papras.stl" scale="0.001 0.001 0.001"/>
+      </geometry>
+      <material name="grey"/>
+    </visual>
+    <collision>
+      <origin xyz="0.067 0.008 -0.019" rpy="0 0 3.14"/>
+      <geometry>
+        <mesh filename="package://open_manipulator_p_description/meshes/link3_papras.stl" scale="0.001 0.001 0.001"/>
       </geometry>
     </collision>
@@ -99,14 +99,14 @@
   <link name="link4">
     <visual>
-      <origin xyz="0 0 0" rpy="0 0 0"/>
-      <geometry>
-        <mesh filename="package://open_manipulator_p_description/meshes/link4.stl" scale="0.001 0.001 0.001"/>
-      </geometry>
-      <material name="grey"/>
-    </visual>
-    <collision>
-      <origin xyz="0 0 0" rpy="0 0 0"/>
-      <geometry>
-        <mesh filename="package://open_manipulator_p_description/meshes/link4.stl" scale="0.001 0.001 0.001"/>
+      <origin xyz="0.227 0.0085 -0.024" rpy="0 0 3.14"/>
+      <geometry>
+        <mesh filename="package://open_manipulator_p_description/meshes/link4_papras.stl" scale="0.001 0.001 0.001"/>
+      </geometry>
+      <material name="grey"/>
+    </visual>
+    <collision>
+      <origin xyz="0.227 0.0085 -0.024" rpy="0 0 3.14"/>
+      <geometry>
+        <mesh filename="package://open_manipulator_p_description/meshes/link4_papras.stl" scale="0.001 0.001 0.001"/>
       </geometry>
     </collision>
@@ -163,14 +163,14 @@
   <link name="link6">
     <visual>
-      <origin xyz="0 0 0" rpy="0 0 0"/>
-      <geometry>
-        <mesh filename="package://open_manipulator_p_description/meshes/link6.stl" scale="0.001 0.001 0.001"/>
-      </geometry>
-      <material name="grey"/>
-    </visual>
-    <collision>
-      <origin xyz="0 0 0" rpy="0 0 0"/>
-      <geometry>
-        <mesh filename="package://open_manipulator_p_description/meshes/link6.stl" scale="0.001 0.001 0.001"/>
+      <origin xyz="-0.034 -0.098 -0.028" rpy="0 0 0"/>
+      <geometry>
+        <mesh filename="package://open_manipulator_p_description/meshes/link6_papras.stl" scale="0.001 0.001 0.001"/>
+      </geometry>
+      <material name="grey"/>
+    </visual>
+    <collision>
+      <origin xyz="-0.034 -0.098 -0.028" rpy="0 0 0"/>
+      <geometry>
+        <mesh filename="package://open_manipulator_p_description/meshes/link6_papras.stl" scale="0.001 0.001 0.001"/>
       </geometry>
     </collision>

File: open_manipulator_p/open_manipulator_p_description/urdf/open_manipulator_p_with_gripper.urdf.xacro (robot description, xacro)
@@ -67,14 +67,14 @@
   <link name="link3">
     <visual>
-      <origin xyz="0 0 0" rpy="0 0 0"/>
-      <geometry>
-        <mesh filename="package://open_manipulator_p_description/meshes/link3.stl" scale="0.001 0.001 0.001"/>
-      </geometry>
-      <material name="grey"/>
-    </visual>
-    <collision>
-      <origin xyz="0 0 0" rpy="0 0 0"/>
-      <geometry>
-        <mesh filename="package://open_manipulator_p_description/meshes/link3.stl" scale="0.001 0.001 0.001"/>
+      <origin xyz="0.067 0.008 -0.019" rpy="0 0 3.14"/>
+      <geometry>
+        <mesh filename="package://open_manipulator_p_description/meshes/link3_papras.stl" scale="0.001 0.001 0.001"/>
+      </geometry>
+      <material name="grey"/>
+    </visual>
+    <collision>
+      <origin xyz="0.067 0.008 -0.019" rpy="0 0 3.14"/>
+      <geometry>
+        <mesh filename="package://open_manipulator_p_description/meshes/link3_papras.stl" scale="0.001 0.001 0.001"/>
       </geometry>
     </collision>
@@ -99,14 +99,14 @@
   <link name="link4">
     <visual>
-      <origin xyz="0 0 0" rpy="0 0 0"/>
-      <geometry>
-        <mesh filename="package://open_manipulator_p_description/meshes/link4.stl" scale="0.001 0.001 0.001"/>
-      </geometry>
-      <material name="grey"/>
-    </visual>
-    <collision>
-      <origin xyz="0 0 0" rpy="0 0 0"/>
-      <geometry>
-        <mesh filename="package://open_manipulator_p_description/meshes/link4.stl" scale="0.001 0.001 0.001"/>
+      <origin xyz="0.227 0.0085 -0.024" rpy="0 0 3.14"/>
+      <geometry>
+        <mesh filename="package://open_manipulator_p_description/meshes/link4_papras.stl" scale="0.001 0.001 0.001"/>
+      </geometry>
+      <material name="grey"/>
+    </visual>
+    <collision>
+      <origin xyz="0.227 0.0085 -0.024" rpy="0 0 3.14"/>
+      <geometry>
+        <mesh filename="package://open_manipulator_p_description/meshes/link4_papras.stl" scale="0.001 0.001 0.001"/>
       </geometry>
     </collision>
@@ -163,14 +163,14 @@
   <link name="link6">
     <visual>
-      <origin xyz="0 0 0" rpy="0 0 0"/>
-      <geometry>
-        <mesh filename="package://open_manipulator_p_description/meshes/link6.stl" scale="0.001 0.001 0.001"/>
-      </geometry>
-      <material name="grey"/>
-    </visual>
-    <collision>
-      <origin xyz="0 0 0" rpy="0 0 0"/>
-      <geometry>
-        <mesh filename="package://open_manipulator_p_description/meshes/link6.stl" scale="0.001 0.001 0.001"/>
+      <origin xyz="-0.034 -0.098 -0.028" rpy="0 0 0"/>
+      <geometry>
+        <mesh filename="package://open_manipulator_p_description/meshes/link6_papras.stl" scale="0.001 0.001 0.001"/>
+      </geometry>
+      <material name="grey"/>
+    </visual>
+    <collision>
+      <origin xyz="-0.034 -0.098 -0.028" rpy="0 0 0"/>
+      <geometry>
+        <mesh filename="package://open_manipulator_p_description/meshes/link6_papras.stl" scale="0.001 0.001 0.001"/>
       </geometry>
     </collision>

File: open_manipulator_p/open_manipulator_p_description/urdf/papras_group_moveit.urdf.xacro (robot description, xacro)
@@ -93,14 +93,14 @@
     <link name="robot${id}/link3">
       <visual>
-        <origin xyz="0 0 0" rpy="0 0 0"/>
-        <geometry>
-          <mesh filename="package://open_manipulator_p_description/meshes/link3.stl" scale="0.001 0.001 0.001"/>
-        </geometry>
-        <material name="grey"/>
-      </visual>
-      <collision>
-        <origin xyz="0 0 0" rpy="0 0 0"/>
-        <geometry>
-          <mesh filename="package://open_manipulator_p_description/meshes/link3.stl" scale="0.001 0.001 0.001"/>
+        <origin xyz="0.067 0.008 -0.019" rpy="0 0 3.14"/>
+        <geometry>
+          <mesh filename="package://open_manipulator_p_description/meshes/link3_papras.stl" scale="0.001 0.001 0.001"/>
+        </geometry>
+        <material name="grey"/>
+      </visual>
+      <collision>
+        <origin xyz="0.067 0.008 -0.019" rpy="0 0 3.14"/>
+        <geometry>
+          <mesh filename="package://open_manipulator_p_description/meshes/link3_papras.stl" scale="0.001 0.001 0.001"/>
         </geometry>
       </collision>
@@ -125,14 +125,14 @@
     <link name="robot${id}/link4">
       <visual>
-        <origin xyz="0 0 0" rpy="0 0 0"/>
-        <geometry>
-          <mesh filename="package://open_manipulator_p_description/meshes/link4.stl" scale="0.001 0.001 0.001"/>
-        </geometry>
-        <material name="grey"/>
-      </visual>
-      <collision>
-        <origin xyz="0 0 0" rpy="0 0 0"/>
-        <geometry>
-          <mesh filename="package://open_manipulator_p_description/meshes/link4.stl" scale="0.001 0.001 0.001"/>
+        <origin xyz="0.227 0.0085 -0.024" rpy="0 0 3.14"/>
+        <geometry>
+          <mesh filename="package://open_manipulator_p_description/meshes/link4_papras.stl" scale="0.001 0.001 0.001"/>
+        </geometry>
+        <material name="grey"/>
+      </visual>
+      <collision>
+        <origin xyz="0.227 0.0085 -0.024" rpy="0 0 3.14"/>
+        <geometry>
+          <mesh filename="package://open_manipulator_p_description/meshes/link4_papras.stl" scale="0.001 0.001 0.001"/>
         </geometry>
       </collision>
@@ -189,14 +189,14 @@
     <link name="robot${id}/link6">
       <visual>
-        <origin xyz="0 0 0" rpy="0 0 0"/>
-        <geometry>
-          <mesh filename="package://open_manipulator_p_description/meshes/link6.stl" scale="0.001 0.001 0.001"/>
-        </geometry>
-        <material name="grey"/>
-      </visual>
-      <collision>
-        <origin xyz="0 0 0" rpy="0 0 0"/>
-        <geometry>
-          <mesh filename="package://open_manipulator_p_description/meshes/link6.stl" scale="0.001 0.001 0.001"/>
+        <origin xyz="-0.034 -0.098 -0.028" rpy="0 0 0"/>
+        <geometry>
+          <mesh filename="package://open_manipulator_p_description/meshes/link6_papras.stl" scale="0.001 0.001 0.001"/>
+        </geometry>
+        <material name="grey"/>
+      </visual>
+      <collision>
+        <origin xyz="-0.034 -0.098 -0.028" rpy="0 0 0"/>
+        <geometry>
+          <mesh filename="package://open_manipulator_p_description/meshes/link6_papras.stl" scale="0.001 0.001 0.001"/>
         </geometry>
       </collision>

Commit message: New hardware limits FIXED

File: open_manipulator_p/open_manipulator_p_description/urdf/open_manipulator_p.urdf.xacro (robot description, xacro)
@@ -61,5 +61,5 @@
     <origin xyz="0.0 0.069 0.033" rpy="0 0 0"/>
     <axis xyz="0 1 0"/>
-    <limit velocity="6.5" effort="1000" lower="$-2.0" upper="$2.0" />
+    <limit velocity="6.5" effort="1000" lower="-2.0" upper="2.0" />
     <dynamics damping="0.7"/>
   </joint>
