Commit message: Keynote vids (#51)
* post coffee and 2 arm stand demos

* created naive kitchen urdf

* start of yaml file for kitchen moves

* add cmd op yaml

* kitchen demo cmp op tested on sim

* Full yaml file with poses confirmed on hw

* update arm name in yaml

* post kitchen keynote vid

* Fix #39 - added mimic joint plugin for gripper in gazebo

* Full 1000 arm URDF and Moveit package (#24)

* rename for consistent naming

* 2arm launch file

* Merge branch 'keynote-vids' of https://github-dev.cs.illinois.edu/KIMLAB/PAPRAS into keynote-vids

* minor changes to clean up warning/error msgs

Co-authored-by: Dhruv Mathur <dmathur2@illinois.edu>

File: open_manipulator_p/open_manipulator_p_description/urdf/2arm_stand.gazebo.xacro (robot description, xacro)
@@ -15,4 +15,6 @@
   <!-- World -->
   <gazebo reference="world"/>
+  <!-- Stand Link -->
+  <gazebo reference="stand_link"/>
   <!-- Link1 -->
   <RefLink ref="link1"/>
@@ -29,4 +31,14 @@
   <!-- end_link -->
   <RefLink ref="end_link"/>
+  <!-- gripper_main_link -->
+  <RefLink ref="gripper_main_link"/>
+  <!-- gripper_link -->
+  <RefLink ref="gripper_link"/>
+  <!-- gripper_sub_link -->
+  <RefLink ref="gripper_sub_link"/>
+  <!-- end_effector_link -->
+  <gazebo reference="end_effector_link">
+    <material>Gazebo/Red</material>
+  </gazebo>
   <!-- ros_control plugin -->
   <gazebo>
@@ -35,3 +47,21 @@
     </plugin>
   </gazebo>
+  <gazebo>
+    <!-- loading plugin: mimic joints works in gazebo now -->
+    <plugin name="gazebo_left_gripper_ros_control" filename="libroboticsgroup_gazebo_mimic_joint_plugin.so">
+      <joint>robotleft/gripper</joint>
+      <mimicJoint>robotleft/gripper_sub</mimicJoint>
+      <multiplier>1.0</multiplier>
+      <offset>0.0</offset>
+    </plugin>
+  </gazebo>
+  <gazebo>
+    <!-- loading plugin: mimic joints works in gazebo now -->
+    <plugin name="gazebo_right_gripper_ros_control" filename="libroboticsgroup_gazebo_mimic_joint_plugin.so">
+      <joint>robotright/gripper</joint>
+      <mimicJoint>robotright/gripper_sub</mimicJoint>
+      <multiplier>1.0</multiplier>
+      <offset>0.0</offset>
+    </plugin>
+  </gazebo>
 </robot>

File: open_manipulator_p/open_manipulator_p_description/urdf/papras_group_moveit.urdf.xacro (robot description, xacro)
@@ -14,5 +14,5 @@
   <xacro:arg name="robot2_base_y" default="-0.5545"/>
   <xacro:arg name="robot2_base_z" default="$(eval 0.77-0.084)"/>
-  <xacro:arg name="robot2_base_yaw" default="1.57"/>
+  <xacro:arg name="robot2_base_yaw" default="0.0"/>
   <xacro:arg name="robot3_base_x" default="0.3735"/>
   <xacro:arg name="robot3_base_y" default="-0.2535"/>

File: open_manipulator_p/open_manipulator_p_description/urdf/papras_group_moveit_with_gripper.urdf.xacro (robot description, xacro)
@@ -4,5 +4,5 @@
   <xacro:include filename="$(find open_manipulator_p_description)/urdf/materials.xacro"/>
   <!-- Import all Gazebo-customization elements, including Gazebo colors -->
-  <xacro:include filename="$(find open_manipulator_p_description)/urdf/3arm_moveit.gazebo.xacro"/>
+  <xacro:include filename="$(find open_manipulator_p_description)/urdf/3arm_moveit_with_gripper.gazebo.xacro"/>
   <!-- Import Transmission -->
   <xacro:include filename="$(find open_manipulator_p_description)/urdf/3arm_moveit_with_gripper.transmission.xacro"/>
@@ -14,5 +14,5 @@
   <xacro:arg name="robot2_base_y" default="-0.5545"/>
   <xacro:arg name="robot2_base_z" default="$(eval 0.77-0.084)"/>
-  <xacro:arg name="robot2_base_yaw" default="3.14"/>
+  <xacro:arg name="robot2_base_yaw" default="0.0"/>
   <xacro:arg name="robot3_base_x" default="0.3735"/>
   <xacro:arg name="robot3_base_y" default="-0.2535"/>
