Commit message: Rearchitecture v1 (#61)
* add docker image, abstracted out unmodified pkgs

* abstract out ros openpose

* changed rospkg papras_gazebo to papras

* re: changed rospkg papras_gazebo to papras

* add gui docker

* Update README.md

* add realsense to urdf, improve dockerfile

Co-authored-by: Kazuki Shin <shinkazuki99@gmail.com>

File: open_manipulator_p/open_manipulator_p_description/urdf/papras_group_moveit_with_gripper.urdf.xacro (robot description, xacro)
@@ -357,4 +357,12 @@
       </inertial>
     </link>
+      <!-- Realsense Camera Joint Position -->
+      <joint name="robot${id}/camera_joint" type="fixed">
+        <axis xyz="0 1 0" />
+        <origin xyz="0.070 0.032 0.052" rpy="0 0 0"/>
+        <parent link="robot${id}/link5"/>
+        <child link="camera${id}_link"/>
+      </joint>
+      <link name="camera${id}_link"/>
   </xacro:macro>
   <!-- World with PAPRAS Desk-->

Commit message: Camera tf (#62)
* add gazebo2tf to dockerfile

* add robot_state_publisher, camera_joint to urdf/srdf, linked camera tf to rest of system

* add 3 cams running with coffee demo, check ControlT violations

File: open_manipulator_p/open_manipulator_p_description/urdf/papras_group_moveit_with_gripper.urdf.xacro (robot description, xacro)
@@ -361,5 +361,5 @@
         <axis xyz="0 1 0" />
         <origin xyz="0.070 0.032 0.052" rpy="0 0 0"/>
-        <parent link="robot${id}/link5"/>
+        <parent link="robot${id}/gripper_main_link"/>
         <child link="camera${id}_link"/>
       </joint>

Commit message: minor fix

File: open_manipulator_p/open_manipulator_p_description/urdf/papras_group_moveit_with_gripper.urdf.xacro (robot description, xacro)
@@ -357,12 +357,12 @@
       </inertial>
     </link>
-      <!-- Realsense Camera Joint Position -->
-      <joint name="robot${id}/camera_joint" type="fixed">
-        <axis xyz="0 1 0" />
-        <origin xyz="0.070 0.032 0.052" rpy="0 0 0"/>
-        <parent link="robot${id}/gripper_main_link"/>
-        <child link="camera${id}_link"/>
-      </joint>
-      <link name="camera${id}_link"/>
+    <!-- Realsense Camera Joint Position -->
+    <!-- <joint name="robot${id}/camera_joint" type="fixed">
+      <axis xyz="0 1 0" />
+      <origin xyz="0.070 0.032 0.052" rpy="0 0 0"/>
+      <parent link="robot${id}/gripper_main_link"/>
+      <child link="camera${id}_link"/>
+    </joint>
+    <link name="camera${id}_link"/> -->
   </xacro:macro>
   <!-- World with PAPRAS Desk-->
