Commit message: Cage jacket (#17)
* add stand 4 config

* update lamnda_stand launch file

* Update checklist.md add stand 4

* change demo coffee pkg to coffee_camera moveit config, remove arm2 from coffee_demo.cpp. update checklist.md

* confirmed coffee demo working on hardware

* stand 4 yaml file

* fix stand 4 yaml gripper comment out

* update kitchen poses for old gripper

* cage moveit config  w camera

* increase spot arm speed

* named poses for spot demo

* spot double gripper group

* Initial work on jacket removal

- Found relatively good poses for arms 3 and 4
- Bad trajectories for removing jacket
- Need to overhaul cpp script to include different planning groups and gripper commands

* control commands for for jacket demo

* control for demo jacket

* cage jacket works in sim

* jacket success, filmed

* cage demo on prof

Co-authored-by: Dhruv Mathur <dhruv.mathur3@gmail.com>

File: open_manipulator_p/open_manipulator_p_description/urdf/cage.gazebo.xacro (robot description, xacro)
@@ -54,15 +54,15 @@
   <!-- gripper_main_link -->
   <RefLink ref="robot1/gripper_main_link"/>
-  <RefLink ref="robot2/gripper_main_link"/>
+  <!-- <RefLink ref="robot2/gripper_main_link"/> -->
   <RefLink ref="robot3/gripper_main_link"/>
   <RefLink ref="robot4/gripper_main_link"/>
   <!-- gripper_link -->
   <RefLink ref="robot1/gripper_link"/>
-  <RefLink ref="robot2/gripper_link"/>
+  <!-- <RefLink ref="robot2/gripper_link"/> -->
   <RefLink ref="robot3/gripper_link"/>
   <RefLink ref="robot4/gripper_link"/>
   <!-- gripper_sub_link -->
   <RefLink ref="robot1/gripper_sub_link"/>
-  <RefLink ref="robot2/gripper_sub_link"/>
+  <!-- <RefLink ref="robot2/gripper_sub_link"/> -->
   <RefLink ref="robot3/gripper_sub_link"/>
   <RefLink ref="robot4/gripper_sub_link"/>
@@ -71,7 +71,7 @@
     <material>Gazebo/Red</material>
   </gazebo>
-  <gazebo reference="robot2/end_effector_link">
+  <!-- <gazebo reference="robot2/end_effector_link">
     <material>Gazebo/Red</material>
-  </gazebo>
+  </gazebo> -->
   <gazebo reference="robot3/end_effector_link">
     <material>Gazebo/Red</material>
@@ -80,4 +80,7 @@
     <material>Gazebo/Red</material>
   </gazebo>
+  <!-- camera_link -->
+  <gazebo reference="robot1/camera_link"/>
+  <gazebo reference="robot4/camera_link"/>
   <!-- ros_control plugin -->
   <gazebo>
@@ -95,6 +98,6 @@
     </plugin>
   </gazebo>
-  <gazebo>
-    <!-- loading plugin: mimic joints works in gazebo now -->
+  <!-- <gazebo>
+    loading plugin: mimic joints works in gazebo now
     <plugin name="gazebo_robot2_gripper_ros_control" filename="libroboticsgroup_gazebo_mimic_joint_plugin.so">
       <joint>robot2/gripper</joint>
@@ -103,5 +106,5 @@
       <offset>0.0</offset>
     </plugin>
-  </gazebo>
+  </gazebo> -->
   <gazebo>
     <!-- loading plugin: mimic joints works in gazebo now -->

File: open_manipulator_p/open_manipulator_p_description/urdf/cage.transmission.xacro (robot description, xacro)
@@ -57,10 +57,10 @@
   <!-- Transmission gripper -->
   <xacro:SimpleTransmissionEffort n="gripper" joint="gripper" id="1"/>
-  <xacro:SimpleTransmissionEffort n="gripper" joint="gripper" id="2"/>
+  <!-- <xacro:SimpleTransmissionEffort n="gripper" joint="gripper" id="2"/> -->
   <xacro:SimpleTransmissionEffort n="gripper" joint="gripper" id="3"/>
   <xacro:SimpleTransmissionEffort n="gripper" joint="gripper" id="4"/>
   <!-- Transmission gripper_sub -->
   <xacro:SimpleTransmissionEffort n="gripper_sub" joint="gripper_sub" id="1"/>
-  <xacro:SimpleTransmissionEffort n="gripper_sub" joint="gripper_sub" id="2"/>
+  <!-- <xacro:SimpleTransmissionEffort n="gripper_sub" joint="gripper_sub" id="2"/> -->
   <xacro:SimpleTransmissionEffort n="gripper_sub" joint="gripper_sub" id="3"/>
   <xacro:SimpleTransmissionEffort n="gripper_sub" joint="gripper_sub" id="4"/>

File: open_manipulator_p/open_manipulator_p_description/urdf/cage.urdf.xacro (robot description, xacro)
@@ -251,5 +251,7 @@
       </inertial>
     </link>
-     <!-- gripper main fixed joint-->
+  </xacro:macro>
+  <xacro:macro name="omp_gripper" params="id">
+    <!-- gripper main fixed joint-->
     <joint name="robot${id}/end_link_fixed" type="fixed">
       <parent link="robot${id}/end_link"/>
@@ -366,4 +368,32 @@
         <origin xyz="0.0 0.0 0.0" rpy="0 0 0" />
         <mass value="0.001" />
+        <inertia ixx="1.0" ixy="0.0" ixz="0.0" iyy="1.0" iyz="0.0" izz="1.0" />
+      </inertial>
+    </link>
+  </xacro:macro>
+  <xacro:macro name="omp_camera" params="id">
+    <!-- camera link fixed joint -->
+    <joint name="robot${id}/camera_fixed_joint" type="fixed">
+      <parent link="robot${id}/gripper_main_link"/>
+      <child link="robot${id}/camera_link"/>
+      <origin xyz="0.0592 0.0167 0.04452" rpy="0 0 0" />
+    </joint>
+    <!-- Camera Link -->
+    <link name="robot${id}/camera_link">
+      <visual>
+        <origin xyz="0 0 0" rpy="0 0 0" />
+        <geometry>
+          <mesh filename="package://open_manipulator_p_description/meshes/camera_mount.stl"/>
+        </geometry>
+      </visual>
+      <collision>
+        <origin xyz="0 0 0" rpy="0 0 0" />
+        <geometry>
+          <mesh filename="package://open_manipulator_p_description/meshes/camera_mount_simple.stl"/>
+        </geometry>
+      </collision>
+      <inertial>
+        <origin xyz="0 0 0" rpy="0 0 0"/>
+        <mass value="0.088"/>
         <inertia ixx="1.0" ixy="0.0" ixz="0.0" iyy="1.0" iyz="0.0" izz="1.0" />
       </inertial>
@@ -393,6 +423,11 @@
   <!-- Arms -->
   <xacro:omp_arm id="1"/>
+  <xacro:omp_gripper id="1"/>
+  <xacro:omp_camera id="1"/>
   <xacro:omp_arm id="2"/>
   <xacro:omp_arm id="3"/>
+  <xacro:omp_gripper id="3"/>
   <xacro:omp_arm id="4"/>
+  <xacro:omp_gripper id="4"/>
+  <xacro:omp_camera id="4"/>
 </robot>
