Commit message: add realsense depth sensor to coffee urdf, visualized on rviz but wrong transform from camera link to world

File: papras_description/urdf/coffee_camera.gazebo.xacro (robot description, xacro)
@@ -55,6 +55,6 @@
   </gazebo>
   <!-- camera_link -->
-  <gazebo reference="robot1/camera_link"/>
-  <gazebo reference="robot3/camera_link"/>
+  <!-- <gazebo reference="robot1/camera_link"/>
+  <gazebo reference="robot3/camera_link"/> -->
   <!-- ros_control plugin -->
   <gazebo>
@@ -81,3 +81,81 @@
     </plugin>
   </gazebo>
+  <!-- rgb camera -->
+  <!-- <gazebo reference="robot1/camera_link">
+    <sensor type="camera" name="camera1">
+      <update_rate>0</update_rate>
+      <camera name="head">
+        <horizontal_fov>1.02974</horizontal_fov>
+        <image>
+          <width>1920</width>
+          <height>1080</height>
+          <format>R8G8B8</format>
+        </image>
+        <clip>
+          <near>0.02</near>
+          <far>300</far>
+        </clip>
+        <noise>
+          <type>gaussian</type>
+          <mean>0.0</mean>
+          <stddev>0.007</stddev>
+        </noise>
+      </camera>
+      <plugin name="camera_controller" filename="libgazebo_ros_camera.so">
+        <alwaysOn>true</alwaysOn>
+        <updateRate>0.0</updateRate>
+        <cameraName>robot1/camera</cameraName>
+        <imageTopicName>image_raw</imageTopicName>
+        <cameraInfoTopicName>camera_info</cameraInfoTopicName>
+        <frameName>robot1/camera_link</frameName>
+        <hackBaseline>0.07</hackBaseline>
+        <distortionK1>0.0</distortionK1>
+        <distortionK2>0.0</distortionK2>
+        <distortionK3>0.0</distortionK3>
+        <distortionT1>0.0</distortionT1>
+        <distortionT2>0.0</distortionT2>
+      </plugin>
+    </sensor>
+  </gazebo> -->
+  <gazebo reference="robot1/camera_link">
+    <sensor name="camera1" type="depth">
+      <update_rate>20</update_rate>
+      <camera>
+        <horizontal_fov>1.047198</horizontal_fov>
+        <image>
+          <width>640</width>
+          <height>480</height>
+          <format>R8G8B8</format>
+        </image>
+        <clip>
+          <near>0.01</near>
+          <far>3</far>
+        </clip>
+      </camera>
+      <plugin name="camera1_controller" filename="libgazebo_ros_openni_kinect.so">
+        <baseline>0.2</baseline>
+        <alwaysOn>true</alwaysOn>
+        <updateRate>1.0</updateRate>
+        <cameraName>robot1/camera_ir</cameraName>
+        <imageTopicName>/color/image_raw</imageTopicName>
+        <cameraInfoTopicName>/color/camera_info</cameraInfoTopicName>
+        <depthImageTopicName>/depth/image_raw</depthImageTopicName>
+        <depthImageInfoTopicName>/depth/camera_info</depthImageInfoTopicName>
+        <pointCloudTopicName>/depth/points</pointCloudTopicName>
+        <frameName>robot1/camera_link</frameName>
+        <pointCloudCutoff>0.01</pointCloudCutoff>
+        <pointCloudCutoffMax>3.0</pointCloudCutoffMax>
+        <distortionK1>0.00000001</distortionK1>
+        <distortionK2>0.00000001</distortionK2>
+        <distortionK3>0.00000001</distortionK3>
+        <distortionT1>0.00000001</distortionT1>
+        <distortionT2>0.00000001</distortionT2>
+        <CxPrime>0</CxPrime>
+        <Cx>0</Cx>
+        <Cy>0</Cy>
+        <focalLength>0</focalLength>
+        <hackBaseline>0</hackBaseline>
+      </plugin>
+    </sensor>
+  </gazebo>
 </robot>

File: papras_description/urdf/coffee_camera.urdf.xacro (robot description, xacro)
@@ -363,4 +363,5 @@
     <!-- camera link fixed joint -->
     <joint name="robot${id}/camera_fixed_joint" type="fixed">
+      <axis xyz="0 1 0" />
       <parent link="robot${id}/gripper_main_link"/>
       <child link="robot${id}/camera_link"/>

Commit message: fix point cloud localization error, add dummy camera depth joint in coffee urdf with roll yaw rotations

File: papras_description/urdf/coffee_camera.gazebo.xacro (robot description, xacro)
@@ -82,6 +82,6 @@
   </gazebo>
   <!-- rgb camera -->
-  <!-- <gazebo reference="robot1/camera_link">
-    <sensor type="camera" name="camera1">
+  <gazebo reference="robot1/camera_link">
+    <sensor name="rgb_camera1" type="camera">
       <update_rate>0</update_rate>
       <camera name="head">
@@ -117,7 +117,7 @@
       </plugin>
     </sensor>
-  </gazebo> -->
+  </gazebo>
   <gazebo reference="robot1/camera_link">
-    <sensor name="camera1" type="depth">
+    <sensor name="depth_camera1" type="depth">
       <update_rate>20</update_rate>
       <camera>
@@ -143,5 +143,5 @@
         <depthImageInfoTopicName>/depth/camera_info</depthImageInfoTopicName>
         <pointCloudTopicName>/depth/points</pointCloudTopicName>
-        <frameName>robot1/camera_link</frameName>
+        <frameName>robot1/camera_depth_link</frameName>
         <pointCloudCutoff>0.01</pointCloudCutoff>
         <pointCloudCutoffMax>3.0</pointCloudCutoffMax>

File: papras_description/urdf/coffee_camera.urdf.xacro (robot description, xacro)
@@ -388,4 +388,12 @@
       </inertial>
     </link>
+    <!-- Empty link to fix depth sensor transform -->
+    <!-- https://answers.ros.org/question/218395/libgazebo_ros_openni_kinectso-depth-pointcloud-wrong-tf/ -->
+    <joint name="robot${id}/camera_depth_joint" type="fixed">
+      <origin xyz="0 0 0" rpy="${-pi/2} 0 ${-pi/2} "/>
+      <parent link="robot${id}/camera_link"/>
+      <child link="robot${id}/camera_depth_link"/>
+    </joint>
+    <link name="robot${id}/camera_depth_link"></link>
   </xacro:macro>
   <!-- World with PAPRAS Desk-->
