Commit message: pick_place: add urdf and stl model spawn in gazebo

File: papras_description/urdf/spot_mount.urdf.xacro (robot description, xacro)
@@ -2,9 +2,9 @@
 <robot name="open_manipulator_p" xmlns:xacro="http://www.ros.org/wiki/xacro">
   <!-- Import Rviz colors -->
-  <xacro:include filename="$(find open_manipulator_p_description)/urdf/materials.xacro"/>
+  <xacro:include filename="$(find papras_description)/urdf/materials.xacro"/>
   <!-- Import all Gazebo-customization elements, including Gazebo colors -->
-  <xacro:include filename="$(find open_manipulator_p_description)/urdf/spot_mount.gazebo.xacro"/>
+  <xacro:include filename="$(find papras_description)/urdf/spot_mount.gazebo.xacro"/>
   <!-- Import Transmission -->
-  <xacro:include filename="$(find open_manipulator_p_description)/urdf/spot_mount.transmission.xacro"/>
+  <xacro:include filename="$(find papras_description)/urdf/spot_mount.transmission.xacro"/>
   <xacro:arg name="robot1_base_x" default="0.0"/>
   <xacro:arg name="robot1_base_y" default="0.05049"/>
@@ -31,12 +31,12 @@
         <origin xyz="0 0 0" rpy="0 0 0"/>
         <geometry>
-          <mesh filename="package://open_manipulator_p_description/meshes/link1.stl" scale="0.001 0.001 0.001"/>
-        </geometry>
-        <material name="grey"/>
-      </visual>
-      <collision>
-        <origin xyz="0 0 0" rpy="0 0 0"/>
-        <geometry>
-          <mesh filename="package://open_manipulator_p_description/meshes/link1.stl" scale="0.001 0.001 0.001"/>
+          <mesh filename="package://papras_description/meshes/link1.stl" scale="0.001 0.001 0.001"/>
+        </geometry>
+        <material name="grey"/>
+      </visual>
+      <collision>
+        <origin xyz="0 0 0" rpy="0 0 0"/>
+        <geometry>
+          <mesh filename="package://papras_description/meshes/link1.stl" scale="0.001 0.001 0.001"/>
         </geometry>
       </collision>
@@ -62,12 +62,12 @@
         <origin xyz="0 0 0" rpy="0 0 0"/>
         <geometry>
-          <mesh filename="package://open_manipulator_p_description/meshes/link2.stl" scale="0.001 0.001 0.001"/>
-        </geometry>
-        <material name="grey"/>
-      </visual>
-      <collision>
-        <origin xyz="0 0 0" rpy="0 0 0"/>
-        <geometry>
-          <mesh filename="package://open_manipulator_p_description/meshes/link2.stl" scale="0.001 0.001 0.001"/>
+          <mesh filename="package://papras_description/meshes/link2.stl" scale="0.001 0.001 0.001"/>
+        </geometry>
+        <material name="grey"/>
+      </visual>
+      <collision>
+        <origin xyz="0 0 0" rpy="0 0 0"/>
+        <geometry>
+          <mesh filename="package://papras_description/meshes/link2.stl" scale="0.001 0.001 0.001"/>
         </geometry>
       </collision>
@@ -94,5 +94,5 @@
         <origin xyz="0.067 0.008 -0.019" rpy="0 0 3.14"/>
         <geometry>
-          <mesh filename="package://open_manipulator_p_description/meshes/link3_papras.stl" scale="0.001 0.001 0.001"/>
+          <mesh filename="package://papras_description/meshes/link3_papras.stl" scale="0.001 0.001 0.001"/>
         </geometry>
         <material name="grey"/>
@@ -101,5 +101,5 @@
         <origin xyz="0.067 0.008 -0.019" rpy="0 0 3.14"/>
         <geometry>
-          <mesh filename="package://open_manipulator_p_description/meshes/link3_papras_simple.stl" scale="0.001 0.001 0.001"/>
+          <mesh filename="package://papras_description/meshes/link3_papras_simple.stl" scale="0.001 0.001 0.001"/>
         </geometry>
       </collision>
@@ -126,5 +126,5 @@
         <origin xyz="0.227 0.0085 -0.024" rpy="0 0 3.14"/>
         <geometry>
-          <mesh filename="package://open_manipulator_p_description/meshes/link4_papras.stl" scale="0.001 0.001 0.001"/>
+          <mesh filename="package://papras_description/meshes/link4_papras.stl" scale="0.001 0.001 0.001"/>
         </geometry>
         <material name="grey"/>
@@ -133,5 +133,5 @@
         <origin xyz="0.227 0.0085 -0.024" rpy="0 0 3.14"/>
         <geometry>
-          <mesh filename="package://open_manipulator_p_description/meshes/link4_papras_simple.stl" scale="0.001 0.001 0.001"/>
+          <mesh filename="package://papras_description/meshes/link4_papras_simple.stl" scale="0.001 0.001 0.001"/>
         </geometry>
       </collision>
@@ -158,12 +158,12 @@
         <origin xyz="0 0 0" rpy="0 0 0"/>
         <geometry>
-          <mesh filename="package://open_manipulator_p_description/meshes/link5.stl" scale="0.001 0.001 0.001"/>
-        </geometry>
-        <material name="grey"/>
-      </visual>
-      <collision>
-        <origin xyz="0 0 0" rpy="0 0 0"/>
-        <geometry>
-          <mesh filename="package://open_manipulator_p_description/meshes/link5.stl" scale="0.001 0.001 0.001"/>
+          <mesh filename="package://papras_description/meshes/link5.stl" scale="0.001 0.001 0.001"/>
+        </geometry>
+        <material name="grey"/>
+      </visual>
+      <collision>
+        <origin xyz="0 0 0" rpy="0 0 0"/>
+        <geometry>
+          <mesh filename="package://papras_description/meshes/link5.stl" scale="0.001 0.001 0.001"/>
         </geometry>
       </collision>
@@ -190,5 +190,5 @@
         <origin xyz="-0.034 -0.098 -0.028" rpy="0 0 0"/>
         <geometry>
-          <mesh filename="package://open_manipulator_p_description/meshes/link6_papras.stl" scale="0.001 0.001 0.001"/>
+          <mesh filename="package://papras_description/meshes/link6_papras.stl" scale="0.001 0.001 0.001"/>
         </geometry>
         <material name="grey"/>
@@ -197,5 +197,5 @@
         <origin xyz="-0.034 -0.098 -0.028" rpy="0 0 0"/>
         <geometry>
-          <mesh filename="package://open_manipulator_p_description/meshes/link6_papras_simple.stl" scale="0.001 0.001 0.001"/>
+          <mesh filename="package://papras_description/meshes/link6_papras_simple.stl" scale="0.001 0.001 0.001"/>
         </geometry>
       </collision>
@@ -222,5 +222,5 @@
         <origin xyz="0.0 0.0 0.0" rpy="0 0 0" />
         <geometry>
-          <mesh filename="package://open_manipulator_p_description/meshes/end_link.stl" scale="0.001 0.001 0.001"/>
+          <mesh filename="package://papras_description/meshes/end_link.stl" scale="0.001 0.001 0.001"/>
         </geometry>
         <material name="grey"/>
@@ -229,5 +229,5 @@
         <origin xyz="0.0 0.0 0.0" rpy="0 0 0" />
         <geometry>
-          <mesh filename="package://open_manipulator_p_description/meshes/end_link.stl" scale="0.001 0.001 0.001"/>
+          <mesh filename="package://papras_description/meshes/end_link.stl" scale="0.001 0.001 0.001"/>
         </geometry>
       </collision>
@@ -252,12 +252,12 @@
         <origin xyz="0 0 0" rpy="0 0 0" />
         <geometry>
-          <mesh filename="package://open_manipulator_p_description/meshes/gripper_main_link.stl" scale="0.001 0.001 0.001"/>
-        </geometry>
-        <material name="grey"/>
-      </visual>
-      <collision>
-        <origin xyz="0 0 0" rpy="0 0 0" />
-        <geometry>
-          <mesh filename="package://open_manipulator_p_description/meshes/gripper_main_link.stl" scale="0.001 0.001 0.001"/>
+          <mesh filename="package://papras_description/meshes/gripper_main_link.stl" scale="0.001 0.001 0.001"/>
+        </geometry>
+        <material name="grey"/>
+      </visual>
+      <collision>
+        <origin xyz="0 0 0" rpy="0 0 0" />
+        <geometry>
+          <mesh filename="package://papras_description/meshes/gripper_main_link.stl" scale="0.001 0.001 0.001"/>
         </geometry>
       </collision>
@@ -282,12 +282,12 @@
         <origin xyz="0 0 0" rpy="0 0 0" />
         <geometry>
-          <mesh filename="package://open_manipulator_p_description/meshes/gripper_link.stl" scale="0.001 0.001 0.001"/>
-        </geometry>
-        <material name="grey"/>
-      </visual>
-      <collision>
-        <origin xyz="0 0 0" rpy="0 0 0" />
-        <geometry>
-          <mesh filename="package://open_manipulator_p_description/meshes/gripper_link.stl" scale="0.001 0.001 0.001"/>
+          <mesh filename="package://papras_description/meshes/gripper_link.stl" scale="0.001 0.001 0.001"/>
+        </geometry>
+        <material name="grey"/>
+      </visual>
+      <collision>
+        <origin xyz="0 0 0" rpy="0 0 0" />
+        <geometry>
+          <mesh filename="package://papras_description/meshes/gripper_link.stl" scale="0.001 0.001 0.001"/>
         </geometry>
         <material name="grey"/>
@@ -314,12 +314,12 @@
         <origin xyz="0 0 0" rpy="0 0 0" />
         <geometry>
-          <mesh filename="package://open_manipulator_p_description/meshes/gripper_sub_link.stl" scale="0.001 0.001 0.001"/>
-        </geometry>
-        <material name="grey"/>
-      </visual>
-      <collision>
-        <origin xyz="0 0 0" rpy="0 0 0" />
-        <geometry>
-          <mesh filename="package://open_manipulator_p_description/meshes/gripper_sub_link.stl" scale="0.001 0.001 0.001"/>
+          <mesh filename="package://papras_description/meshes/gripper_sub_link.stl" scale="0.001 0.001 0.001"/>
+        </geometry>
+        <material name="grey"/>
+      </visual>
+      <collision>
+        <origin xyz="0 0 0" rpy="0 0 0" />
+        <geometry>
+          <mesh filename="package://papras_description/meshes/gripper_sub_link.stl" scale="0.001 0.001 0.001"/>
         </geometry>
         <material name="grey"/>
@@ -372,11 +372,11 @@
         <origin xyz="0 0 0" rpy="0 0 0" />
         <geometry>
-          <mesh filename="package://open_manipulator_p_description/meshes/camera_mount.stl"/>
-        </geometry>
-      </visual>
-      <collision>
-        <origin xyz="0 0 0" rpy="0 0 0" />
-        <geometry>
-          <mesh filename="package://open_manipulator_p_description/meshes/camera_mount_simple.stl"/>
+          <mesh filename="package://papras_description/meshes/camera_mount.stl"/>
+        </geometry>
+      </visual>
+      <collision>
+        <origin xyz="0 0 0" rpy="0 0 0" />
+        <geometry>
+          <mesh filename="package://papras_description/meshes/camera_mount_simple.stl"/>
         </geometry>
       </collision>
@@ -399,5 +399,5 @@
       <origin xyz="0.0 0.0 0.0" rpy="0 0 0" />
       <geometry>
-        <mesh filename="package://open_manipulator_p_description/meshes/spot_mount.stl"/>
+        <mesh filename="package://papras_description/meshes/spot_mount.stl"/>
       </geometry>
     </visual>
@@ -405,5 +405,5 @@
       <origin xyz="0.0 0.0 0.0" rpy="0 0 0" />
       <geometry>
-        <mesh filename="package://open_manipulator_p_description/meshes/spot_mount_simple.stl"/>
+        <mesh filename="package://papras_description/meshes/spot_mount_simple.stl"/>
       </geometry>
     </collision>
