Commit message: spot candy demo tested in sim

File: papras_description/urdf/spot_mount.urdf.xacro (robot description, xacro)
@@ -1,401 +1,15 @@
 <?xml version="1.0"?>
-<robot name="open_manipulator_p" xmlns:xacro="http://www.ros.org/wiki/xacro">
-  <!-- Import Rviz colors -->
-  <xacro:include filename="$(find papras_description)/urdf/materials.xacro"/>
-  <!-- Import all Gazebo-customization elements, including Gazebo colors -->
-  <xacro:include filename="$(find papras_description)/urdf/spot_mount.gazebo.xacro"/>
-  <!-- Import Transmission -->
-  <xacro:include filename="$(find papras_description)/urdf/spot_mount.transmission.xacro"/>
-  <xacro:arg name="robot1_base_x" default="0.0"/>
-  <xacro:arg name="robot1_base_y" default="0.05049"/>
-  <xacro:arg name="robot1_base_z" default="0.09003"/>
-  <xacro:arg name="robot1_base_roll" default="0.0"/>
-  <xacro:arg name="robot1_base_pitch" default="$(eval ${pi*0.25})"/>
-  <xacro:arg name="robot1_base_yaw" default="$(eval ${pi*0.5})"/>
-  <xacro:arg name="robot2_base_x" default="0.0"/>
-  <xacro:arg name="robot2_base_y" default="-0.05049"/>
-  <xacro:arg name="robot2_base_z" default="0.09003"/>
-  <xacro:arg name="robot2_base_roll" default="0.0"/>
-  <xacro:arg name="robot2_base_pitch" default="$(eval ${pi*0.25})"/>
-  <xacro:arg name="robot2_base_yaw" default="$(eval ${-pi*0.5})"/>
-  <xacro:macro name="omp_arm" params="id">
-    <joint name="robot${id}/arm_spot_mount_fixed" type="fixed">
-        <parent link="spot_mount" />
-        <child link="robot${id}/link1" />
-        <origin xyz="$(eval robot${id}_base_x) $(eval robot${id}_base_y) $(eval robot${id}_base_z)"
-                rpy="$(eval robot${id}_base_roll) $(eval robot${id}_base_pitch) $(eval robot${id}_base_yaw)"/>
-    </joint>
-    <!-- link 1 -->
-    <link name="robot${id}/link1">
-      <visual>
-        <origin xyz="0 0 0" rpy="0 0 0"/>
-        <geometry>
-          <mesh filename="package://papras_description/meshes/link1.stl" scale="0.001 0.001 0.001"/>
-        </geometry>
-        <material name="grey"/>
-      </visual>
-      <collision>
-        <origin xyz="0 0 0" rpy="0 0 0"/>
-        <geometry>
-          <mesh filename="package://papras_description/meshes/link1.stl" scale="0.001 0.001 0.001"/>
-        </geometry>
-      </collision>
-      <inertial>
-        <origin xyz="0.00023 0.00000 0.06223" rpy="0 0 0"/>
-        <mass value="0.85644"/>
-        <inertia ixx="1.0" ixy="0.0" ixz="0.0" iyy="1.0" iyz="0.0" izz="1.0" />
-        <!--<inertia ixx="0.00121064" ixy="0.0" ixz="0.00001100" iyy="0.00120886" iyz="0.0" izz="0.00038103" />-->
-      </inertial>
-    </link>
-    <!-- Joint 1 -->
-    <joint name="robot${id}/joint1" type="revolute">
-      <parent link="robot${id}/link1"/>
-      <child link="robot${id}/link2"/>
-      <origin xyz="0.0 0.0 0.126" rpy="0 0 0"/>
-      <axis xyz="0 0 1"/>
-      <limit velocity="6.5" effort="1000" lower="${-pi*1.0}" upper="${pi*1.0}" />
-      <dynamics damping="0.7"/>
-    </joint>
-    <!-- link 2 -->
-    <link name="robot${id}/link2">
-      <visual>
-        <origin xyz="0 0 0" rpy="0 0 0"/>
-        <geometry>
-          <mesh filename="package://papras_description/meshes/link2.stl" scale="0.001 0.001 0.001"/>
-        </geometry>
-        <material name="grey"/>
-      </visual>
-      <collision>
-        <origin xyz="0 0 0" rpy="0 0 0"/>
-        <geometry>
-          <mesh filename="package://papras_description/meshes/link2.stl" scale="0.001 0.001 0.001"/>
-        </geometry>
-      </collision>
-      <inertial>
-        <origin xyz="0.00000 0.00080 0.03183" rpy="0 0 0"/>
-        <!--<origin xyz="0.00000 -0.06820 -0.00117" rpy="0 0 0"/>-->
-        <mass value="0.94658"/>
-        <inertia ixx="1.0" ixy="0.0" ixz="0.0" iyy="1.0" iyz="0.0" izz="1.0" />
-        <!--<inertia ixx="0.00152547" ixy="0.0" ixz="0.0" iyy="0.00045954" iyz="-0.00001086" izz="0.00151740" />-->
-      </inertial>
-    </link>
-    <!-- Joint 2 -->
-    <joint name="robot${id}/joint2" type="revolute">
-      <parent link="robot${id}/link2"/>
-      <child link="robot${id}/link3"/>
-      <origin xyz="0.0 0.069 0.033" rpy="0 0 0"/>
-      <axis xyz="0 1 0"/>
-      <limit velocity="6.5" effort="1000" lower="-2.0" upper="2.0" />
-      <dynamics damping="0.7"/>
-    </joint>
-    <!-- link 3 -->
-    <link name="robot${id}/link3">
-      <visual>
-        <origin xyz="0.067 0.008 -0.019" rpy="0 0 3.14"/>
-        <geometry>
-          <mesh filename="package://papras_description/meshes/link3_papras.stl" scale="0.001 0.001 0.001"/>
-        </geometry>
-        <material name="grey"/>
-      </visual>
-      <collision>
-        <origin xyz="0.067 0.008 -0.019" rpy="0 0 3.14"/>
-        <geometry>
-          <mesh filename="package://papras_description/meshes/link3_papras_simple.stl" scale="0.001 0.001 0.001"/>
-        </geometry>
-      </collision>
-      <inertial>
-        <origin xyz="0.01768 -0.06881 0.20524" rpy="0 0 0"/>
-        <!--<origin xyz="-0.01232 -0.05731 -0.05876" rpy="0 0 0"/>-->
-        <mass value="1.30260"/>
-        <inertia ixx="1.0" ixy="0.0" ixz="0.0" iyy="1.0" iyz="0.0" izz="1.0" />
-        <!--<inertia ixx="0.01111021" ixy="0.00001331" ixz="-0.00134208" iyy="0.01046642" iyz="0.00016235" izz="0.00202081" />-->
-      </inertial>
-    </link>
-    <!-- Joint 3 -->
-    <joint name="robot${id}/joint3" type="revolute">
-      <parent link="robot${id}/link3"/>
-      <child link="robot${id}/link4"/>
-      <origin xyz="0.03000 -0.01150 0.26400" rpy="0 0 0"/>
-      <axis xyz="0 1 0"/>
-      <limit velocity="6.5" effort="1000" lower="${-pi*1.0}" upper="${pi*0.5}" />
-      <dynamics damping="0.7"/>
-    </joint>
-    <!-- link 4 -->
-    <link name="robot${id}/link4">
-      <visual>
-        <origin xyz="0.227 0.0085 -0.024" rpy="0 0 3.14"/>
-        <geometry>
-          <mesh filename="package://papras_description/meshes/link4_papras.stl" scale="0.001 0.001 0.001"/>
-        </geometry>
-        <material name="grey"/>
-      </visual>
-      <collision>
-        <origin xyz="0.227 0.0085 -0.024" rpy="0 0 3.14"/>
-        <geometry>
-          <mesh filename="package://papras_description/meshes/link4_papras_simple.stl" scale="0.001 0.001 0.001"/>
-        </geometry>
-      </collision>
-      <inertial>
-        <origin xyz="0.12475 -0.05716 0.02979" rpy="0 0 0"/>
-        <!--<origin xyz="-0.07025 0.00034 -0.00021" rpy="0 0 0"/>-->
-        <mass value="1.15977"/>
-        <inertia ixx="1.0" ixy="0.0" ixz="0.0" iyy="1.0" iyz="0.0" izz="1.0" />
-        <!--<inertia ixx="0.00096726" ixy="0.00004383" ixz="-0.00002771" iyy="0.00318801" iyz="0.00000627" izz="0.00341484" />-->
-      </inertial>
-    </link>
-    <!-- Joint 4 -->
-    <joint name="robot${id}/joint4" type="revolute">
-      <parent link="robot${id}/link4"/>
-      <child link="robot${id}/link5"/>
-      <origin xyz="0.19500 -0.05750 0.03000" rpy="0 0 0"/>
-      <axis xyz="1 0 0"/>
-      <limit velocity="6.5" effort="1000" lower="${-pi*0.875}" upper="${pi*0.875}" />
-      <dynamics damping="0.7"/>
-    </joint>
-    <!-- link 5 -->
-    <link name="robot${id}/link5">
-      <visual>
-        <origin xyz="0 0 0" rpy="0 0 0"/>
-        <geometry>
-          <mesh filename="package://papras_description/meshes/link5.stl" scale="0.001 0.001 0.001"/>
-        </geometry>
-        <material name="grey"/>
-      </visual>
-      <collision>
-        <origin xyz="0 0 0" rpy="0 0 0"/>
-        <geometry>
-          <mesh filename="package://papras_description/meshes/link5.stl" scale="0.001 0.001 0.001"/>
-        </geometry>
-      </collision>
-      <inertial>
-        <origin xyz="0.05642 -0.00217 0.00002" rpy="0 0 0"/>
-        <!--<origin xyz="-0.00658 -0.04717 0.00002" rpy="0 0 0"/>-->
-        <mass value="0.44688"/>
-        <inertia ixx="1.0" ixy="0.0" ixz="0.0" iyy="1.0" iyz="0.0" izz="1.0" />
-        <!--<inertia ixx="0.00030285" ixy="0.00000761" ixz="0.00000031" iyy="0.00022339" iyz="-0.00000001" izz="0.00039766" />-->
-      </inertial>
-    </link>
-    <!-- Joint 5 -->
-    <joint name="robot${id}/joint5" type="revolute">
-      <parent link="robot${id}/link5"/>
-      <child link="robot${id}/link6"/>
-      <origin xyz="0.06300 0.04500 0.00000" rpy="0 0 0"/>
-      <axis xyz="0 1 0"/>
-      <limit velocity="6.5" effort="1000" lower="${-pi*0.5}" upper="${pi*0.5}" />
-      <dynamics damping="0.7"/>
-    </joint>
-    <!-- link 6 -->
-    <link name="robot${id}/link6">
-      <visual>
-        <origin xyz="-0.034 -0.098 -0.028" rpy="0 0 0"/>
-        <geometry>
-          <mesh filename="package://papras_description/meshes/link6_papras.stl" scale="0.001 0.001 0.001"/>
-        </geometry>
-        <material name="grey"/>
-      </visual>
-      <collision>
-        <origin xyz="-0.034 -0.098 -0.028" rpy="0 0 0"/>
-        <geometry>
-          <mesh filename="package://papras_description/meshes/link6_papras_simple.stl" scale="0.001 0.001 0.001"/>
-        </geometry>
-      </collision>
-      <inertial>
-        <origin xyz="0.06831 -0.04457 0.00000" rpy="0 0 0"/>
-        <!--<origin xyz="-0.05469 0.00043 0.00000" rpy="0 0 0"/>-->
-        <mass value="0.43273"/>
-        <inertia ixx="1.0" ixy="0.0" ixz="0.0" iyy="1.0" iyz="0.0" izz="1.0" />
-        <!--<inertia ixx="0.00021512" ixy="0.00001009" ixz="0.00000000" iyy="0.00042827" iyz="0.00000000" izz="0.00051436" />-->
-      </inertial>
-    </link>
-    <!-- Joint 6 -->
-    <joint name="robot${id}/joint6" type="revolute">
-      <parent link="robot${id}/link6"/>
-      <child link="robot${id}/end_link"/>
-      <origin xyz="0.12300 -0.04500 0.00000" rpy="0 0 0"/>
-      <axis xyz="1 0 0"/>
-      <limit velocity="6.5" effort="1000" lower="${-pi*1.0}" upper="${pi*1.0}" />
-      <dynamics damping="0.7"/>
-    </joint>
-    <!-- end link -->
-    <link name="robot${id}/end_link">
-      <visual>
-        <origin xyz="0.0 0.0 0.0" rpy="0 0 0" />
-        <geometry>
-          <mesh filename="package://papras_description/meshes/end_link.stl" scale="0.001 0.001 0.001"/>
-        </geometry>
-        <material name="grey"/>
-      </visual>
-      <collision>
-        <origin xyz="0.0 0.0 0.0" rpy="0 0 0" />
-        <geometry>
-          <mesh filename="package://papras_description/meshes/end_link.stl" scale="0.001 0.001 0.001"/>
-        </geometry>
-      </collision>
-      <inertial>
-        <origin xyz="0.00337 0.00000 0.00000" rpy="0 0 0"/>
-        <mass value="0.01919"/>
-        <inertia ixx="1.0" ixy="0.0" ixz="0.0" iyy="1.0" iyz="0.0" izz="1.0" />
-        <!--<inertia ixx="0.00000938" ixy="0.0" ixz="0.0" iyy="0.00000338" iyz="0.0" izz="0.00000635" />-->
-      </inertial>
-    </link>
-  </xacro:macro>
-  <xacro:macro name="omp_gripper" params="id">
-    <!-- gripper main fixed joint-->
-    <joint name="robot${id}/end_link_fixed" type="fixed">
-      <parent link="robot${id}/end_link"/>
-      <child link="robot${id}/gripper_main_link"/>
-      <origin xyz="0.007 0.0 0.0" rpy="0 0 0" />
-    </joint>
-    <!-- gripper main link -->
-    <link name="robot${id}/gripper_main_link">
-      <visual>
-        <origin xyz="0 0 0" rpy="0 0 0" />
-        <geometry>
-          <mesh filename="package://papras_description/meshes/gripper_main_link.stl" scale="0.001 0.001 0.001"/>
-        </geometry>
-        <material name="grey"/>
-      </visual>
-      <collision>
-        <origin xyz="0 0 0" rpy="0 0 0" />
-        <geometry>
-          <mesh filename="package://papras_description/meshes/gripper_main_link.stl" scale="0.001 0.001 0.001"/>
-        </geometry>
-      </collision>
-      <inertial>
-        <origin xyz="0.0 0.0 0.0" rpy="0 0 0"/>
-        <mass value="0.509"/>
-        <inertia ixx="1.0" ixy="0.0" ixz="0.0" iyy="1.0" iyz="0.0" izz="1.0" />
-      </inertial>
-    </link>
-    <!-- gripper joint -->
-    <joint name="robot${id}/gripper" type="revolute">
-      <axis xyz="0 0 1" />
-      <origin xyz="0.0552 -0.0400 0" rpy="0 0 -0.4"/>
-      <parent link="robot${id}/gripper_main_link"/>
-      <child link="robot${id}/gripper_link"/>
-      <limit velocity="6.5" effort="1000" lower="0.0" upper="1.1" />
-      <dynamics damping="0.1" friction="0.0" />
-    </joint>
-    <!-- gripper link -->
-    <link name="robot${id}/gripper_link">
-      <visual>
-        <origin xyz="0 0 0" rpy="0 0 0" />
-        <geometry>
-          <mesh filename="package://papras_description/meshes/gripper_link.stl" scale="0.001 0.001 0.001"/>
-        </geometry>
-        <material name="grey"/>
-      </visual>
-      <collision>
-        <origin xyz="0 0 0" rpy="0 0 0" />
-        <geometry>
-          <mesh filename="package://papras_description/meshes/gripper_link.stl" scale="0.001 0.001 0.001"/>
-        </geometry>
-        <material name="grey"/>
-      </collision>
-      <inertial>
-        <origin xyz="0 0 0" rpy="0 0 0"/>
-        <mass value="0.013"/>
-        <inertia ixx="1.0" ixy="0.0" ixz="0.0" iyy="1.0" iyz="0.0" izz="1.0" />
-      </inertial>
-    </link>
-    <!-- gripper joint 1 -->
-    <joint name="robot${id}/gripper_sub" type="revolute">
-      <axis xyz="0 0 -1" />
-      <origin xyz="0.0552 0.0400 0" rpy="0 0 0.4"/>
-      <parent link="robot${id}/gripper_main_link"/>
-      <child link="robot${id}/gripper_sub_link"/>
-      <limit velocity="6.5" effort="1000" lower="0.0" upper="1.1" />
-      <dynamics damping="0.1" friction="0.0" />
-      <mimic joint="robot${id}/gripper" multiplier="1"/>
-    </joint>
-    <!-- gripper 1 link -->
-    <link name="robot${id}/gripper_sub_link">
-      <visual>
-        <origin xyz="0 0 0" rpy="0 0 0" />
-        <geometry>
-          <mesh filename="package://papras_description/meshes/gripper_sub_link.stl" scale="0.001 0.001 0.001"/>
-        </geometry>
-        <material name="grey"/>
-      </visual>
-      <collision>
-        <origin xyz="0 0 0" rpy="0 0 0" />
-        <geometry>
-          <mesh filename="package://papras_description/meshes/gripper_sub_link.stl" scale="0.001 0.001 0.001"/>
-        </geometry>
-        <material name="grey"/>
-      </collision>
-      <inertial>
-        <origin xyz="0 0 0" rpy="0 0 0"/>
-        <mass value="0.013"/>
-        <inertia ixx="1.0" ixy="0.0" ixz="0.0" iyy="1.0" iyz="0.0" izz="1.0" />
-      </inertial>
-    </link>
-    <!-- gripper main fixed joint-->
-    <joint name="robot${id}/end_effector_joint" type="fixed">
-      <parent link="robot${id}/gripper_main_link"/>
-      <child link="robot${id}/end_effector_link"/>
-      <origin xyz="0.14 0.0 0.0" rpy="0 0 0" />
-    </joint>
-    <!-- End Effector -->
-    <link name="robot${id}/end_effector_link">
-      <visual>
-        <origin xyz="0.0 0.0 0.0" rpy="0 0 0" />
-        <geometry>
-          <box size = "0.01 0.01 0.01"/>
-        </geometry>
-        <material name="red"/>
-      </visual>
-      <collision>
-        <origin xyz="0.0 0.0 0.0" rpy="0 0 0" />
-        <geometry>
-          <box size = "0.01 0.01 0.01"/>
-        </geometry>
-        <material name="red"/>
-      </collision>
-      <inertial>
-        <origin xyz="0.0 0.0 0.0" rpy="0 0 0" />
-        <mass value="0.001" />
-        <inertia ixx="1.0" ixy="0.0" ixz="0.0" iyy="1.0" iyz="0.0" izz="1.0" />
-      </inertial>
-    </link>
-  </xacro:macro>
-  <xacro:macro name="omp_camera" params="id">
-    <!-- camera link fixed joint -->
-    <joint name="robot${id}/camera_fixed_joint" type="fixed">
-      <parent link="robot${id}/gripper_main_link"/>
-      <child link="robot${id}/camera_link"/>
-      <origin xyz="0.0592 0.0167 0.04452" rpy="0 0 0" />
-    </joint>
-    <!-- Camera Link -->
-    <link name="robot${id}/camera_link">
-      <visual>
-        <origin xyz="0 0 0" rpy="0 0 0" />
-        <geometry>
-          <mesh filename="package://papras_description/meshes/camera_mount.stl"/>
-        </geometry>
-      </visual>
-      <collision>
-        <origin xyz="0 0 0" rpy="0 0 0" />
-        <geometry>
-          <mesh filename="package://papras_description/meshes/camera_mount_simple.stl"/>
-        </geometry>
-      </collision>
-      <inertial>
-        <origin xyz="0 0 0" rpy="0 0 0"/>
-        <mass value="0.088"/>
-        <inertia ixx="1.0" ixy="0.0" ixz="0.0" iyy="1.0" iyz="0.0" izz="1.0" />
-      </inertial>
-    </link>
-  </xacro:macro>
-  <!-- World with PAPRAS Desk-->
+<robot name="spot_mount" xmlns:xacro="http://www.ros.org/wiki/xacro">
+  <!-- Import PAPRAS Macros -->
+  <xacro:include filename="$(find papras_description)/urdf/papras_macros.xacro"/>
   <link name="world"/>
-  <joint name="spot_mount_world_fixed" type="fixed">
-      <parent link="world" />
-      <child link="spot_mount" />
-      <origin xyz="0 0 0" rpy="0 0 0"/>
+  <joint name="world_env_fixed" type="fixed">
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
File: papras_description/urdf/tea_table.urdf.xacro (robot description, xacro)
@@ -11,5 +11,5 @@
   <link name="env">
     <visual>
-      <origin xyz="0.0 0.0 00" rpy="0 0 0"/>
+      <origin xyz="0.0 0.0 0.0" rpy="0 0 0"/>
       <geometry>
         <mesh filename="package://papras_description/meshes/tea_table.stl"/>
