Commit message: add pkg perception sim utils

File: papras_description/urdf/kitchen.urdf.xacro (robot description, xacro)
@@ -1,10 +1,10 @@
 <?xml version="1.0"?>
-<robot name="open_manipulator_p" xmlns:xacro="http://www.ros.org/wiki/xacro">
+<robot name="papras kitchen" xmlns:xacro="http://www.ros.org/wiki/xacro">
   <!-- Import Rviz colors -->
-  <xacro:include filename="$(find open_manipulator_p_description)/urdf/materials.xacro"/>
+  <xacro:include filename="$(find papras_description)/urdf/materials.xacro"/>
   <!-- Import all Gazebo-customization elements, including Gazebo colors -->
-  <xacro:include filename="$(find open_manipulator_p_description)/urdf/kitchen.gazebo.xacro"/>
+  <xacro:include filename="$(find papras_description)/urdf/kitchen.gazebo.xacro"/>
   <!-- Import Transmission -->
-  <xacro:include filename="$(find open_manipulator_p_description)/urdf/kitchen.transmission.xacro"/>
+  <xacro:include filename="$(find papras_description)/urdf/kitchen.transmission.xacro"/>
   <xacro:arg name="robot1_base_x" default="-0.02394"/>
   <xacro:arg name="robot1_base_y" default="0.04497"/>
@@ -25,12 +25,12 @@
         <origin xyz="0 0 0" rpy="0 0 0"/>
         <geometry>
-          <mesh filename="package://open_manipulator_p_description/meshes/link1.stl" scale="0.001 0.001 0.001"/>
-        </geometry>
-        <material name="grey"/>
-      </visual>
-      <collision>
-        <origin xyz="0 0 0" rpy="0 0 0"/>
-        <geometry>
-          <mesh filename="package://open_manipulator_p_description/meshes/link1.stl" scale="0.001 0.001 0.001"/>
+          <mesh filename="package://papras_description/meshes/link1.stl" scale="0.001 0.001 0.001"/>
+        </geometry>
+        <material name="grey"/>
+      </visual>
+      <collision>
+        <origin xyz="0 0 0" rpy="0 0 0"/>
+        <geometry>
+          <mesh filename="package://papras_description/meshes/link1.stl" scale="0.001 0.001 0.001"/>
         </geometry>
       </collision>
@@ -56,12 +56,12 @@
         <origin xyz="0 0 0" rpy="0 0 0"/>
         <geometry>
-          <mesh filename="package://open_manipulator_p_description/meshes/link2.stl" scale="0.001 0.001 0.001"/>
-        </geometry>
-        <material name="grey"/>
-      </visual>
-      <collision>
-        <origin xyz="0 0 0" rpy="0 0 0"/>
-        <geometry>
-          <mesh filename="package://open_manipulator_p_description/meshes/link2.stl" scale="0.001 0.001 0.001"/>
+          <mesh filename="package://papras_description/meshes/link2.stl" scale="0.001 0.001 0.001"/>
+        </geometry>
+        <material name="grey"/>
+      </visual>
+      <collision>
+        <origin xyz="0 0 0" rpy="0 0 0"/>
+        <geometry>
+          <mesh filename="package://papras_description/meshes/link2.stl" scale="0.001 0.001 0.001"/>
         </geometry>
       </collision>
@@ -88,5 +88,5 @@
         <origin xyz="0.067 0.008 -0.019" rpy="0 0 3.14"/>
         <geometry>
-          <mesh filename="package://open_manipulator_p_description/meshes/link3_papras.stl" scale="0.001 0.001 0.001"/>
+          <mesh filename="package://papras_description/meshes/link3_papras.stl" scale="0.001 0.001 0.001"/>
         </geometry>
         <material name="grey"/>
@@ -95,5 +95,5 @@
         <origin xyz="0.067 0.008 -0.019" rpy="0 0 3.14"/>
         <geometry>
-          <mesh filename="package://open_manipulator_p_description/meshes/link3_papras_simple.stl" scale="0.001 0.001 0.001"/>
+          <mesh filename="package://papras_description/meshes/link3_papras_simple.stl" scale="0.001 0.001 0.001"/>
         </geometry>
       </collision>
@@ -120,5 +120,5 @@
         <origin xyz="0.227 0.0085 -0.024" rpy="0 0 3.14"/>
         <geometry>
-          <mesh filename="package://open_manipulator_p_description/meshes/link4_papras.stl" scale="0.001 0.001 0.001"/>
+          <mesh filename="package://papras_description/meshes/link4_papras.stl" scale="0.001 0.001 0.001"/>
         </geometry>
         <material name="grey"/>
@@ -127,5 +127,5 @@
         <origin xyz="0.227 0.0085 -0.024" rpy="0 0 3.14"/>
         <geometry>
-          <mesh filename="package://open_manipulator_p_description/meshes/link4_papras_simple.stl" scale="0.001 0.001 0.001"/>
+          <mesh filename="package://papras_description/meshes/link4_papras_simple.stl" scale="0.001 0.001 0.001"/>
         </geometry>
       </collision>
@@ -152,12 +152,12 @@
         <origin xyz="0 0 0" rpy="0 0 0"/>
         <geometry>
-          <mesh filename="package://open_manipulator_p_description/meshes/link5.stl" scale="0.001 0.001 0.001"/>
-        </geometry>
-        <material name="grey"/>
-      </visual>
-      <collision>
-        <origin xyz="0 0 0" rpy="0 0 0"/>
-        <geometry>
-          <mesh filename="package://open_manipulator_p_description/meshes/link5.stl" scale="0.001 0.001 0.001"/>
+          <mesh filename="package://papras_description/meshes/link5.stl" scale="0.001 0.001 0.001"/>
+        </geometry>
+        <material name="grey"/>
+      </visual>
+      <collision>
+        <origin xyz="0 0 0" rpy="0 0 0"/>
+        <geometry>
+          <mesh filename="package://papras_description/meshes/link5.stl" scale="0.001 0.001 0.001"/>
         </geometry>
       </collision>
@@ -184,5 +184,5 @@
         <origin xyz="-0.034 -0.098 -0.028" rpy="0 0 0"/>
         <geometry>
-          <mesh filename="package://open_manipulator_p_description/meshes/link6_papras.stl" scale="0.001 0.001 0.001"/>
+          <mesh filename="package://papras_description/meshes/link6_papras.stl" scale="0.001 0.001 0.001"/>
         </geometry>
         <material name="grey"/>
@@ -191,5 +191,5 @@
         <origin xyz="-0.034 -0.098 -0.028" rpy="0 0 0"/>
         <geometry>
-          <mesh filename="package://open_manipulator_p_description/meshes/link6_papras_simple.stl" scale="0.001 0.001 0.001"/>
+          <mesh filename="package://papras_description/meshes/link6_papras_simple.stl" scale="0.001 0.001 0.001"/>
         </geometry>
       </collision>
@@ -216,12 +216,12 @@
         <origin xyz="0.0 0.0 0.0" rpy="0 0 0" />
         <geometry>
-          <mesh filename="package://open_manipulator_p_description/meshes/end_link.stl" scale="0.001 0.001 0.001"/>
-        </geometry>
-        <material name="grey"/>
-      </visual>
-      <collision>
-        <origin xyz="0.0 0.0 0.0" rpy="0 0 0" />
-        <geometry>
-          <mesh filename="package://open_manipulator_p_description/meshes/end_link.stl" scale="0.001 0.001 0.001"/>
+          <mesh filename="package://papras_description/meshes/end_link.stl" scale="0.001 0.001 0.001"/>
+        </geometry>
+        <material name="grey"/>
+      </visual>
+      <collision>
+        <origin xyz="0.0 0.0 0.0" rpy="0 0 0" />
+        <geometry>
+          <mesh filename="package://papras_description/meshes/end_link.stl" scale="0.001 0.001 0.001"/>
         </geometry>
       </collision>
@@ -244,12 +244,12 @@
         <origin xyz="0 0 0" rpy="0 0 0" />
         <geometry>
-          <mesh filename="package://open_manipulator_p_description/meshes/gripper_main_link.stl" scale="0.001 0.001 0.001"/>
-        </geometry>
-        <material name="grey"/>
-      </visual>
-      <collision>
-        <origin xyz="0 0 0" rpy="0 0 0" />
-        <geometry>
-          <mesh filename="package://open_manipulator_p_description/meshes/gripper_main_link.stl" scale="0.001 0.001 0.001"/>
+          <mesh filename="package://papras_description/meshes/gripper_main_link.stl" scale="0.001 0.001 0.001"/>
+        </geometry>
+        <material name="grey"/>
+      </visual>
+      <collision>
+        <origin xyz="0 0 0" rpy="0 0 0" />
+        <geometry>
+          <mesh filename="package://papras_description/meshes/gripper_main_link.stl" scale="0.001 0.001 0.001"/>
         </geometry>
       </collision>
@@ -274,12 +274,12 @@
         <origin xyz="0 0 0" rpy="0 0 0" />
         <geometry>
-          <mesh filename="package://open_manipulator_p_description/meshes/gripper_link.stl" scale="0.001 0.001 0.001"/>
-        </geometry>
-        <material name="grey"/>
-      </visual>
-      <collision>
-        <origin xyz="0 0 0" rpy="0 0 0" />
-        <geometry>
-          <mesh filename="package://open_manipulator_p_description/meshes/gripper_link.stl" scale="0.001 0.001 0.001"/>
+          <mesh filename="package://papras_description/meshes/gripper_link.stl" scale="0.001 0.001 0.001"/>
+        </geometry>
+        <material name="grey"/>
+      </visual>
+      <collision>
+        <origin xyz="0 0 0" rpy="0 0 0" />
+        <geometry>
+          <mesh filename="package://papras_description/meshes/gripper_link.stl" scale="0.001 0.001 0.001"/>
         </geometry>
         <material name="grey"/>
@@ -306,12 +306,12 @@
         <origin xyz="0 0 0" rpy="0 0 0" />
         <geometry>
-          <mesh filename="package://open_manipulator_p_description/meshes/gripper_sub_link.stl" scale="0.001 0.001 0.001"/>
-        </geometry>
-        <material name="grey"/>
-      </visual>
-      <collision>
-        <origin xyz="0 0 0" rpy="0 0 0" />
-        <geometry>
-          <mesh filename="package://open_manipulator_p_description/meshes/gripper_sub_link.stl" scale="0.001 0.001 0.001"/>
+          <mesh filename="package://papras_description/meshes/gripper_sub_link.stl" scale="0.001 0.001 0.001"/>
+        </geometry>
+        <material name="grey"/>
+      </visual>
+      <collision>
+        <origin xyz="0 0 0" rpy="0 0 0" />
+        <geometry>
+          <mesh filename="package://papras_description/meshes/gripper_sub_link.stl" scale="0.001 0.001 0.001"/>
         </geometry>
         <material name="grey"/>
@@ -363,5 +363,5 @@
       <origin xyz="0.0 0.0 0.0" rpy="0 0 0" />
       <geometry>
-        <mesh filename="package://open_manipulator_p_description/meshes/kitchen.stl"/>
+        <mesh filename="package://papras_description/meshes/kitchen.stl"/>
       </geometry>
     </visual>
@@ -369,5 +369,5 @@
       <origin xyz="0.0 0.0 0.0" rpy="0 0 0" />
       <geometry>
-        <mesh filename="package://open_manipulator_p_description/meshes/kitchen_simple.stl"/>
+        <mesh filename="package://papras_description/meshes/kitchen_simple.stl"/>
       </geometry>
     </collision>

Commit message: initial inertia data from sw2urdf

File: papras_description/urdf/kitchen.urdf.xacro (robot description, xacro)
@@ -36,7 +36,7 @@
       </collision>
       <inertial>
-        <origin xyz="0.00023 0.00000 0.06223" rpy="0 0 0"/>
-        <mass value="0.85644"/>
-        <inertia ixx="1.0" ixy="0.0" ixz="0.0" iyy="1.0" iyz="0.0" izz="1.0" />
+        <origin xyz="0 0 0.06092" rpy="0 0 0"/>
+        <mass value="0.9023"/>
+        <inertia ixx="0.0013454" ixy="0.0" ixz="0.0" iyy="0.0013426" iyz="0.0" izz="0.00039686" />
         <!--<inertia ixx="0.00121064" ixy="0.0" ixz="0.00001100" iyy="0.00120886" iyz="0.0" izz="0.00038103" />-->
       </inertial>
@@ -67,8 +67,8 @@
       </collision>
       <inertial>
-        <origin xyz="0.00000 0.00080 0.03183" rpy="0 0 0"/>
+        <origin xyz="0 0.0025574 0.032618" rpy="0 0 0"/>
         <!--<origin xyz="0.00000 -0.06820 -0.00117" rpy="0 0 0"/>-->
-        <mass value="0.94658"/>
-        <inertia ixx="1.0" ixy="0.0" ixz="0.0" iyy="1.0" iyz="0.0" izz="1.0" />
+        <mass value="0.93297"/>
+        <inertia ixx="0.0013554" ixy="0.0" ixz="0.0" iyy="0.00041526" iyz="0.0" izz="0.0013588" />
         <!--<inertia ixx="0.00152547" ixy="0.0" ixz="0.0" iyy="0.00045954" iyz="-0.00001086" izz="0.00151740" />-->
       </inertial>
@@ -99,8 +99,8 @@
       </collision>
       <inertial>
-        <origin xyz="0.01768 -0.06881 0.20524" rpy="0 0 0"/>
+        <origin xyz="0.014245 -0.069376 0.20003" rpy="0 0 0"/>
         <!--<origin xyz="-0.01232 -0.05731 -0.05876" rpy="0 0 0"/>-->
-        <mass value="1.30260"/>
-        <inertia ixx="1.0" ixy="0.0" ixz="0.0" iyy="1.0" iyz="0.0" izz="1.0" />
+        <mass value="0.65312"/>
+        <inertia ixx="0.0027586" ixy="0.0" ixz="0.0" iyy="0.0021267" iyz="0.0" izz="0.00095197" />
         <!--<inertia ixx="0.01111021" ixy="0.00001331" ixz="-0.00134208" iyy="0.01046642" iyz="0.00016235" izz="0.00202081" />-->
       </inertial>
@@ -131,8 +131,8 @@
       </collision>
       <inertial>
-        <origin xyz="0.12475 -0.05716 0.02979" rpy="0 0 0"/>
+        <origin xyz="0.11815 -0.057014 0.027875" rpy="0 0 0"/>
         <!--<origin xyz="-0.07025 0.00034 -0.00021" rpy="0 0 0"/>-->
-        <mass value="1.15977"/>
-        <inertia ixx="1.0" ixy="0.0" ixz="0.0" iyy="1.0" iyz="0.0" izz="1.0" />
+        <mass value="0.5869"/>
+        <inertia ixx="0.00076095" ixy="0.0" ixz="0.0" iyy="0.0015481" iyz="0.0" izz="0.0018522" />
         <!--<inertia ixx="0.00096726" ixy="0.00004383" ixz="-0.00002771" iyy="0.00318801" iyz="0.00000627" izz="0.00341484" />-->
       </inertial>
@@ -163,8 +163,8 @@
       </collision>
       <inertial>
-        <origin xyz="0.05642 -0.00217 0.00002" rpy="0 0 0"/>
+        <origin xyz="0.055523 0.0014518 0" rpy="0 0 0"/>
         <!--<origin xyz="-0.00658 -0.04717 0.00002" rpy="0 0 0"/>-->
-        <mass value="0.44688"/>
-        <inertia ixx="1.0" ixy="0.0" ixz="0.0" iyy="1.0" iyz="0.0" izz="1.0" />
+        <mass value="0.17671"/>
+        <inertia ixx="0.00010999" ixy="0.0" ixz="0.0" iyy="0.000050887" iyz="0.0" izz="0.00010417" />
         <!--<inertia ixx="0.00030285" ixy="0.00000761" ixz="0.00000031" iyy="0.00022339" iyz="-0.00000001" izz="0.00039766" />-->
       </inertial>
@@ -195,8 +195,8 @@
       </collision>
       <inertial>
-        <origin xyz="0.06831 -0.04457 0.00000" rpy="0 0 0"/>
+        <origin xyz="0.061664 -0.044945 0" rpy="0 0 0"/>
         <!--<origin xyz="-0.05469 0.00043 0.00000" rpy="0 0 0"/>-->
-        <mass value="0.43273"/>
-        <inertia ixx="1.0" ixy="0.0" ixz="0.0" iyy="1.0" iyz="0.0" izz="1.0" />
+        <mass value="0.20465"/>
+        <inertia ixx="0.00013742" ixy="0.0" ixz="0.0" iyy="0.00015856" iyz="0.0" izz="0.00021625" />
         <!--<inertia ixx="0.00021512" ixy="0.00001009" ixz="0.00000000" iyy="0.00042827" iyz="0.00000000" izz="0.00051436" />-->
       </inertial>
@@ -227,7 +227,7 @@
       </collision>
       <inertial>
-        <origin xyz="0.00337 0.00000 0.00000" rpy="0 0 0"/>
-        <mass value="0.01919"/>
-        <inertia ixx="1.0" ixy="0.0" ixz="0.0" iyy="1.0" iyz="0.0" izz="1.0" />
+        <origin xyz="0.003365 0 0" rpy="0 0 0"/>
+        <mass value="0.015"/>
+        <inertia ixx="0.00001106" ixy="0.0" ixz="0.0" iyy="0.00000399" iyz="0.0" izz="0.00000749" />
         <!--<inertia ixx="0.00000938" ixy="0.0" ixz="0.0" iyy="0.00000338" iyz="0.0" izz="0.00000635" />-->
       </inertial>
@@ -255,7 +255,7 @@
       </collision>
       <inertial>
-        <origin xyz="0.0 0.0 0.0" rpy="0 0 0"/>
-        <mass value="0.509"/>
-        <inertia ixx="1.0" ixy="0.0" ixz="0.0" iyy="1.0" iyz="0.0" izz="1.0" />
+        <origin xyz="0.036472 0 0" rpy="0 0 0"/>
+        <mass value="0.400"/>
+        <inertia ixx="0.00041299" ixy="0.0" ixz="0.0" iyy="0.00035504" iyz="0.0" izz="0.00044011" />
       </inertial>
     </link>
@@ -286,7 +286,7 @@
       </collision>
       <inertial>
-        <origin xyz="0 0 0" rpy="0 0 0"/>
-        <mass value="0.013"/>
-        <inertia ixx="1.0" ixy="0.0" ixz="0.0" iyy="1.0" iyz="0.0" izz="1.0" />
+        <origin xyz="0.030630 -0.013802 0" rpy="0 0 0"/>
+        <mass value="0.050"/>
+        <inertia ixx="0.00002894" ixy="0.00003550" ixz="0.0" iyy="0.00010484" iyz="0.0" izz="0.00011795" />
       </inertial>
     </link>
@@ -318,7 +318,7 @@
       </collision>
       <inertial>
-        <origin xyz="0 0 0" rpy="0 0 0"/>
-        <mass value="0.013"/>
-        <inertia ixx="1.0" ixy="0.0" ixz="0.0" iyy="1.0" iyz="0.0" izz="1.0" />
+        <origin xyz="0.030630 0.013802 0" rpy="0 0 0"/>
+        <mass value="0.050"/>
+        <inertia ixx="0.00002894" ixy="-0.00003550" ixz="0.0" iyy="0.00010484" iyz="0.0" izz="0.00011795" />
       </inertial>
     </link>
@@ -357,5 +357,5 @@
       <parent link="world" />
       <child link="kitchen_link" />
-      <origin xyz="0 0 0.04" rpy="0 0 0"/>
+      <origin xyz="0 0 0.1" rpy="0 0 0"/>
   </joint>
   <link name="kitchen_link">
@@ -372,4 +372,9 @@
       </geometry>
     </collision>
+    <inertial>
+      <origin xyz="0.0 0.0 0.5" rpy="0 0 0" />
+      <mass value="100.0" />
+      <inertia ixx="1.0" ixy="0.0" ixz="0.0" iyy="1.0" iyz="0.0" izz="1.0" />
+    </inertial>
   </link>
   <!-- Arms -->

Commit message: removed inertial data from gripper links, arm breaks when it stops

File: papras_description/urdf/kitchen.urdf.xacro (robot description, xacro)
@@ -255,7 +255,7 @@
       </collision>
       <inertial>
-        <origin xyz="0.036472 0 0" rpy="0 0 0"/>
-        <mass value="0.400"/>
-        <inertia ixx="0.00041299" ixy="0.0" ixz="0.0" iyy="0.00035504" iyz="0.0" izz="0.00044011" />
+        <origin xyz="0.0 0.0 0.0" rpy="0 0 0"/>
+        <mass value="0.509"/>
+        <inertia ixx="1.0" ixy="0.0" ixz="0.0" iyy="1.0" iyz="0.0" izz="1.0" />
       </inertial>
     </link>
@@ -286,7 +286,7 @@
       </collision>
       <inertial>
-        <origin xyz="0.030630 -0.013802 0" rpy="0 0 0"/>
-        <mass value="0.050"/>
-        <inertia ixx="0.00002894" ixy="0.00003550" ixz="0.0" iyy="0.00010484" iyz="0.0" izz="0.00011795" />
+        <origin xyz="0 0 0" rpy="0 0 0"/>
+        <mass value="0.013"/>
+        <inertia ixx="1.0" ixy="0.0" ixz="0.0" iyy="1.0" iyz="0.0" izz="1.0" />
       </inertial>
     </link>
@@ -318,7 +318,7 @@
       </collision>
       <inertial>
-        <origin xyz="0.030630 0.013802 0" rpy="0 0 0"/>
-        <mass value="0.050"/>
-        <inertia ixx="0.00002894" ixy="-0.00003550" ixz="0.0" iyy="0.00010484" iyz="0.0" izz="0.00011795" />
+        <origin xyz="0 0 0" rpy="0 0 0"/>
+        <mass value="0.013"/>
+        <inertia ixx="1.0" ixy="0.0" ixz="0.0" iyy="1.0" iyz="0.0" izz="1.0" />
       </inertial>
     </link>

Commit message: fixed kitchen mesh, arm still vibrates at end of motion

File: papras_description/urdf/kitchen.urdf.xacro (robot description, xacro)
@@ -357,5 +357,5 @@
       <parent link="world" />
       <child link="kitchen_link" />
-      <origin xyz="0 0 0.1" rpy="0 0 0"/>
+      <origin xyz="0 0 0" rpy="0 0 0"/>
   </joint>
   <link name="kitchen_link">
@@ -363,5 +363,5 @@
       <origin xyz="0.0 0.0 0.0" rpy="0 0 0" />
       <geometry>
-        <mesh filename="package://papras_description/meshes/kitchen.stl"/>
+        <mesh filename="package://papras_description/meshes/kitchen_new.stl"/>
       </geometry>
     </visual>
@@ -369,5 +369,5 @@
       <origin xyz="0.0 0.0 0.0" rpy="0 0 0" />
       <geometry>
-        <mesh filename="package://papras_description/meshes/kitchen_simple.stl"/>
+        <mesh filename="package://papras_description/meshes/kitchen_new_simple.stl"/>
       </geometry>
     </collision>
