Commit message: fixed kitchen shaking issues

File: papras_description/urdf/kitchen.urdf.xacro (robot description, xacro)
@@ -1,382 +1,33 @@
 <?xml version="1.0"?>
-<robot name="papras kitchen" xmlns:xacro="http://www.ros.org/wiki/xacro">
-  <!-- Import Rviz colors -->
-  <xacro:include filename="$(find papras_description)/urdf/materials.xacro"/>
-  <!-- Import all Gazebo-customization elements, including Gazebo colors -->
-  <xacro:include filename="$(find papras_description)/urdf/kitchen.gazebo.xacro"/>
-  <!-- Import Transmission -->
-  <xacro:include filename="$(find papras_description)/urdf/kitchen.transmission.xacro"/>
-  <xacro:arg name="robot1_base_x" default="-0.02394"/>
-  <xacro:arg name="robot1_base_y" default="0.04497"/>
-  <xacro:arg name="robot1_base_z" default="0.78851"/>
-  <xacro:arg name="robot1_base_roll" default="$(eval ${pi*1.0})"/>
-  <xacro:arg name="robot1_base_pitch" default="$(eval ${-pi*0.5})"/>
-  <xacro:arg name="robot1_base_yaw" default="0.0"/>
-  <xacro:macro name="omp_arm" params="id">
-    <joint name="robot${id}/arm_kitchen_fixed" type="fixed">
-        <parent link="kitchen_link" />
-        <child link="robot${id}/link1" />
-        <origin xyz="$(eval robot${id}_base_x) $(eval robot${id}_base_y) $(eval robot${id}_base_z)"
-                rpy="$(eval robot${id}_base_roll) $(eval robot${id}_base_pitch) $(eval robot${id}_base_yaw)"/>
-    </joint>
-    <!-- link 1 -->
-    <link name="robot${id}/link1">
-      <visual>
-        <origin xyz="0 0 0" rpy="0 0 0"/>
-        <geometry>
-          <mesh filename="package://papras_description/meshes/link1.stl" scale="0.001 0.001 0.001"/>
-        </geometry>
-        <material name="grey"/>
-      </visual>
-      <collision>
-        <origin xyz="0 0 0" rpy="0 0 0"/>
-        <geometry>
-          <mesh filename="package://papras_description/meshes/link1.stl" scale="0.001 0.001 0.001"/>
-        </geometry>
-      </collision>
-      <inertial>
-        <origin xyz="0 0 0.06092" rpy="0 0 0"/>
-        <mass value="0.9023"/>
-        <inertia ixx="0.0013454" ixy="0.0" ixz="0.0" iyy="0.0013426" iyz="0.0" izz="0.00039686" />
-        <!--<inertia ixx="0.00121064" ixy="0.0" ixz="0.00001100" iyy="0.00120886" iyz="0.0" izz="0.00038103" />-->
-      </inertial>
-    </link>
-    <!-- Joint 1 -->
-    <joint name="robot${id}/joint1" type="revolute">
-      <parent link="robot${id}/link1"/>
-      <child link="robot${id}/link2"/>
-      <origin xyz="0.0 0.0 0.126" rpy="0 0 0"/>
-      <axis xyz="0 0 1"/>
-      <limit velocity="6.5" effort="1000" lower="${-pi*1.0}" upper="${pi*1.0}" />
-      <dynamics damping="0.7"/>
-    </joint>
-    <!-- link 2 -->
-    <link name="robot${id}/link2">
-      <visual>
-        <origin xyz="0 0 0" rpy="0 0 0"/>
-        <geometry>
-          <mesh filename="package://papras_description/meshes/link2.stl" scale="0.001 0.001 0.001"/>
-        </geometry>
-        <material name="grey"/>
-      </visual>
-      <collision>
-        <origin xyz="0 0 0" rpy="0 0 0"/>
-        <geometry>
-          <mesh filename="package://papras_description/meshes/link2.stl" scale="0.001 0.001 0.001"/>
-        </geometry>
-      </collision>
-      <inertial>
-        <origin xyz="0 0.0025574 0.032618" rpy="0 0 0"/>
-        <!--<origin xyz="0.00000 -0.06820 -0.00117" rpy="0 0 0"/>-->
-        <mass value="0.93297"/>
-        <inertia ixx="0.0013554" ixy="0.0" ixz="0.0" iyy="0.00041526" iyz="0.0" izz="0.0013588" />
-        <!--<inertia ixx="0.00152547" ixy="0.0" ixz="0.0" iyy="0.00045954" iyz="-0.00001086" izz="0.00151740" />-->
-      </inertial>
-    </link>
-    <!-- Joint 2 -->
-    <joint name="robot${id}/joint2" type="revolute">
-      <parent link="robot${id}/link2"/>
-      <child link="robot${id}/link3"/>
-      <origin xyz="0.0 0.069 0.033" rpy="0 0 0"/>
-      <axis xyz="0 1 0"/>
-      <limit velocity="6.5" effort="1000" lower="-2.0" upper="2.0" />
-      <dynamics damping="0.7"/>
-    </joint>
-    <!-- link 3 -->
-    <link name="robot${id}/link3">
-      <visual>
-        <origin xyz="0.067 0.008 -0.019" rpy="0 0 3.14"/>
-        <geometry>
-          <mesh filename="package://papras_description/meshes/link3_papras.stl" scale="0.001 0.001 0.001"/>
-        </geometry>
-        <material name="grey"/>
-      </visual>
-      <collision>
-        <origin xyz="0.067 0.008 -0.019" rpy="0 0 3.14"/>
-        <geometry>
-          <mesh filename="package://papras_description/meshes/link3_papras_simple.stl" scale="0.001 0.001 0.001"/>
-        </geometry>
-      </collision>
-      <inertial>
-        <origin xyz="0.014245 -0.069376 0.20003" rpy="0 0 0"/>
-        <!--<origin xyz="-0.01232 -0.05731 -0.05876" rpy="0 0 0"/>-->
-        <mass value="0.65312"/>
-        <inertia ixx="0.0027586" ixy="0.0" ixz="0.0" iyy="0.0021267" iyz="0.0" izz="0.00095197" />
-        <!--<inertia ixx="0.01111021" ixy="0.00001331" ixz="-0.00134208" iyy="0.01046642" iyz="0.00016235" izz="0.00202081" />-->
-      </inertial>
-    </link>
-    <!-- Joint 3 -->
-    <joint name="robot${id}/joint3" type="revolute">
-      <parent link="robot${id}/link3"/>
-      <child link="robot${id}/link4"/>
-      <origin xyz="0.03000 -0.01150 0.26400" rpy="0 0 0"/>
-      <axis xyz="0 1 0"/>
-      <limit velocity="6.5" effort="1000" lower="${-pi*1.0}" upper="${pi*0.5}" />
-      <dynamics damping="0.7"/>
-    </joint>
-    <!-- link 4 -->
-    <link name="robot${id}/link4">
-      <visual>
-        <origin xyz="0.227 0.0085 -0.024" rpy="0 0 3.14"/>
-        <geometry>
-          <mesh filename="package://papras_description/meshes/link4_papras.stl" scale="0.001 0.001 0.001"/>
-        </geometry>
-        <material name="grey"/>
-      </visual>
-      <collision>
-        <origin xyz="0.227 0.0085 -0.024" rpy="0 0 3.14"/>
-        <geometry>
-          <mesh filename="package://papras_description/meshes/link4_papras_simple.stl" scale="0.001 0.001 0.001"/>
-        </geometry>
-      </collision>
-      <inertial>
-        <origin xyz="0.11815 -0.057014 0.027875" rpy="0 0 0"/>
-        <!--<origin xyz="-0.07025 0.00034 -0.00021" rpy="0 0 0"/>-->
-        <mass value="0.5869"/>
-        <inertia ixx="0.00076095" ixy="0.0" ixz="0.0" iyy="0.0015481" iyz="0.0" izz="0.0018522" />
-        <!--<inertia ixx="0.00096726" ixy="0.00004383" ixz="-0.00002771" iyy="0.00318801" iyz="0.00000627" izz="0.00341484" />-->
-      </inertial>
-    </link>
-    <!-- Joint 4 -->
-    <joint name="robot${id}/joint4" type="revolute">
-      <parent link="robot${id}/link4"/>
-      <child link="robot${id}/link5"/>
-      <origin xyz="0.19500 -0.05750 0.03000" rpy="0 0 0"/>
-      <axis xyz="1 0 0"/>
-      <limit velocity="6.5" effort="1000" lower="${-pi*0.875}" upper="${pi*0.875}" />
-      <dynamics damping="0.7"/>
-    </joint>
-    <!-- link 5 -->
-    <link name="robot${id}/link5">
-      <visual>
-        <origin xyz="0 0 0" rpy="0 0 0"/>
-        <geometry>
-          <mesh filename="package://papras_description/meshes/link5.stl" scale="0.001 0.001 0.001"/>
-        </geometry>
-        <material name="grey"/>
-      </visual>
-      <collision>
-        <origin xyz="0 0 0" rpy="0 0 0"/>
-        <geometry>
-          <mesh filename="package://papras_description/meshes/link5.stl" scale="0.001 0.001 0.001"/>
-        </geometry>
-      </collision>
-      <inertial>
-        <origin xyz="0.055523 0.0014518 0" rpy="0 0 0"/>
-        <!--<origin xyz="-0.00658 -0.04717 0.00002" rpy="0 0 0"/>-->
-        <mass value="0.17671"/>
-        <inertia ixx="0.00010999" ixy="0.0" ixz="0.0" iyy="0.000050887" iyz="0.0" izz="0.00010417" />
-        <!--<inertia ixx="0.00030285" ixy="0.00000761" ixz="0.00000031" iyy="0.00022339" iyz="-0.00000001" izz="0.00039766" />-->
-      </inertial>
-    </link>
-    <!-- Joint 5 -->
-    <joint name="robot${id}/joint5" type="revolute">
-      <parent link="robot${id}/link5"/>
-      <child link="robot${id}/link6"/>
-      <origin xyz="0.06300 0.04500 0.00000" rpy="0 0 0"/>
-      <axis xyz="0 1 0"/>
-      <limit velocity="6.5" effort="1000" lower="${-pi*0.5}" upper="${pi*0.5}" />
-      <dynamics damping="0.7"/>
-    </joint>
-    <!-- link 6 -->
-    <link name="robot${id}/link6">
-      <visual>
-        <origin xyz="-0.034 -0.098 -0.028" rpy="0 0 0"/>
-        <geometry>
-          <mesh filename="package://papras_description/meshes/link6_papras.stl" scale="0.001 0.001 0.001"/>
-        </geometry>
-        <material name="grey"/>
-      </visual>
-      <collision>
-        <origin xyz="-0.034 -0.098 -0.028" rpy="0 0 0"/>
-        <geometry>
-          <mesh filename="package://papras_description/meshes/link6_papras_simple.stl" scale="0.001 0.001 0.001"/>
-        </geometry>
-      </collision>
-      <inertial>
-        <origin xyz="0.061664 -0.044945 0" rpy="0 0 0"/>
-        <!--<origin xyz="-0.05469 0.00043 0.00000" rpy="0 0 0"/>-->
-        <mass value="0.20465"/>
-        <inertia ixx="0.00013742" ixy="0.0" ixz="0.0" iyy="0.00015856" iyz="0.0" izz="0.00021625" />
-        <!--<inertia ixx="0.00021512" ixy="0.00001009" ixz="0.00000000" iyy="0.00042827" iyz="0.00000000" izz="0.00051436" />-->
-      </inertial>
-    </link>
-    <!-- Joint 6 -->
-    <joint name="robot${id}/joint6" type="revolute">
-      <parent link="robot${id}/link6"/>
-      <child link="robot${id}/end_link"/>
-      <origin xyz="0.12300 -0.04500 0.00000" rpy="0 0 0"/>
-      <axis xyz="1 0 0"/>
-      <limit velocity="6.5" effort="1000" lower="${-pi*1.0}" upper="${pi*1.0}" />
-      <dynamics damping="0.7"/>
-    </joint>
-    <!-- end link -->
-    <link name="robot${id}/end_link">
-      <visual>
-        <origin xyz="0.0 0.0 0.0" rpy="0 0 0" />
-        <geometry>
-          <mesh filename="package://papras_description/meshes/end_link.stl" scale="0.001 0.001 0.001"/>
-        </geometry>
-        <material name="grey"/>
-      </visual>
-      <collision>
-        <origin xyz="0.0 0.0 0.0" rpy="0 0 0" />
-        <geometry>
-          <mesh filename="package://papras_description/meshes/end_link.stl" scale="0.001 0.001 0.001"/>
-        </geometry>
-      </collision>
-      <inertial>
-        <origin xyz="0.003365 0 0" rpy="0 0 0"/>
-        <mass value="0.015"/>
-        <inertia ixx="0.00001106" ixy="0.0" ixz="0.0" iyy="0.00000399" iyz="0.0" izz="0.00000749" />
-        <!--<inertia ixx="0.00000938" ixy="0.0" ixz="0.0" iyy="0.00000338" iyz="0.0" izz="0.00000635" />-->
-      </inertial>
-    </link>
-     <!-- gripper main fixed joint-->
-    <joint name="robot${id}/end_link_fixed" type="fixed">
-      <parent link="robot${id}/end_link"/>
-      <child link="robot${id}/gripper_main_link"/>
-      <origin xyz="0.007 0.0 0.0" rpy="0 0 0" />
-    </joint>
-    <!-- gripper main link -->
-    <link name="robot${id}/gripper_main_link">
-      <visual>
-        <origin xyz="0 0 0" rpy="0 0 0" />
-        <geometry>
-          <mesh filename="package://papras_description/meshes/gripper_main_link.stl" scale="0.001 0.001 0.001"/>
-        </geometry>
-        <material name="grey"/>
-      </visual>
-      <collision>
-        <origin xyz="0 0 0" rpy="0 0 0" />
-        <geometry>
-          <mesh filename="package://papras_description/meshes/gripper_main_link.stl" scale="0.001 0.001 0.001"/>
-        </geometry>
-      </collision>
-      <inertial>
-        <origin xyz="0.0 0.0 0.0" rpy="0 0 0"/>
-        <mass value="0.509"/>
-        <inertia ixx="1.0" ixy="0.0" ixz="0.0" iyy="1.0" iyz="0.0" izz="1.0" />
-      </inertial>
-    </link>
-    <!-- gripper joint -->
-    <joint name="robot${id}/gripper" type="revolute">
-      <axis xyz="0 0 1" />
-      <origin xyz="0.0552 -0.0400 0" rpy="0 0 -0.4"/>
-      <parent link="robot${id}/gripper_main_link"/>
-      <child link="robot${id}/gripper_link"/>
-      <limit velocity="6.5" effort="1000" lower="0.0" upper="1.1" />
-      <dynamics damping="0.1" friction="0.0" />
-    </joint>
-    <!-- gripper link -->
-    <link name="robot${id}/gripper_link">
-      <visual>
-        <origin xyz="0 0 0" rpy="0 0 0" />
-        <geometry>
-          <mesh filename="package://papras_description/meshes/gripper_link.stl" scale="0.001 0.001 0.001"/>
-        </geometry>
-        <material name="grey"/>
-      </visual>
-      <collision>
-        <origin xyz="0 0 0" rpy="0 0 0" />
-        <geometry>
-          <mesh filename="package://papras_description/meshes/gripper_link.stl" scale="0.001 0.001 0.001"/>
-        </geometry>
-        <material name="grey"/>
-      </collision>
-      <inertial>
-        <origin xyz="0 0 0" rpy="0 0 0"/>
-        <mass value="0.013"/>
-        <inertia ixx="1.0" ixy="0.0" ixz="0.0" iyy="1.0" iyz="0.0" izz="1.0" />
-      </inertial>
-    </link>
-    <!-- gripper joint 1 -->
-    <joint name="robot${id}/gripper_sub" type="revolute">
-      <axis xyz="0 0 -1" />
-      <origin xyz="0.0552 0.0400 0" rpy="0 0 0.4"/>
-      <parent link="robot${id}/gripper_main_link"/>
-      <child link="robot${id}/gripper_sub_link"/>
-      <limit velocity="6.5" effort="1000" lower="0.0" upper="1.1" />
-      <dynamics damping="0.1" friction="0.0" />
-      <mimic joint="robot${id}/gripper" multiplier="1"/>
-    </joint>
-    <!-- gripper 1 link -->
-    <link name="robot${id}/gripper_sub_link">
-      <visual>
-        <origin xyz="0 0 0" rpy="0 0 0" />
-        <geometry>
-          <mesh filename="package://papras_description/meshes/gripper_sub_link.stl" scale="0.001 0.001 0.001"/>
-        </geometry>
-        <material name="grey"/>
-      </visual>
-      <collision>
-        <origin xyz="0 0 0" rpy="0 0 0" />
-        <geometry>
-          <mesh filename="package://papras_description/meshes/gripper_sub_link.stl" scale="0.001 0.001 0.001"/>
-        </geometry>
-        <material name="grey"/>
-      </collision>
-      <inertial>
-        <origin xyz="0 0 0" rpy="0 0 0"/>
-        <mass value="0.013"/>
-        <inertia ixx="1.0" ixy="0.0" ixz="0.0" iyy="1.0" iyz="0.0" izz="1.0" />
-      </inertial>
-    </link>
-    <!-- gripper main fixed joint-->
-    <joint name="robot${id}/end_effector_joint" type="fixed">
-      <parent link="robot${id}/gripper_main_link"/>
-      <child link="robot${id}/end_effector_link"/>
-      <origin xyz="0.14 0.0 0.0" rpy="0 0 0" />
-    </joint>
-    <!-- End Effector -->
-    <link name="robot${id}/end_effector_link">
-      <visual>
-        <origin xyz="0.0 0.0 0.0" rpy="0 0 0" />
-        <geometry>
-          <box size = "0.01 0.01 0.01"/>
-        </geometry>
-        <material name="red"/>
-      </visual>
-      <collision>
-        <origin xyz="0.0 0.0 0.0" rpy="0 0 0" />
-        <geometry>
-          <box size = "0.01 0.01 0.01"/>
-        </geometry>
-        <material name="red"/>
-      </collision>
-      <inertial>
-        <origin xyz="0.0 0.0 0.0" rpy="0 0 0" />
-        <mass value="0.001" />
-        <inertia ixx="1.0" ixy="0.0" ixz="0.0" iyy="1.0" iyz="0.0" izz="1.0" />
-      </inertial>
-    </link>
-  </xacro:macro>
-  <!-- World with kitchen-->
+<robot name="kitchen" xmlns:xacro="http://www.ros.org/wiki/xacro">
+  <!-- Import PAPRAS Macros -->
+  <xacro:include filename="$(find papras_description)/urdf/papras_macros.xacro"/>
   <link name="world"/>
-  <joint name="kitchen_world_fixed" type="fixed">
-      <parent link="world" />
-      <child link="kitchen_link" />
-      <origin xyz="0 0 0" rpy="0 0 0"/>
+  <joint name="world_env_fixed" type="fixed">
+    <parent link="world"/>
+    <child link="env"/>
+    <origin xyz="0 0 0" rpy="0 0 0"/>
   </joint>
-  <link name="kitchen_link">
+  <link name="env">
     <visual>
-      <origin xyz="0.0 0.0 0.0" rpy="0 0 0" />
+      <origin xyz="0.0 0.0 0.0" rpy="0 0 0"/>
       <geometry>
-        <mesh filename="package://papras_description/meshes/kitchen_new.stl"/>
+        <mesh filename="package://papras_description/meshes/kitchen.stl"/>
       </geometry>
     </visual>
     <collision>
-      <origin xyz="0.0 0.0 0.0" rpy="0 0 0" />
+      <origin xyz="0.0 0.0 0.0" rpy="0 0 0"/>
       <geometry>
-        <mesh filename="package://papras_description/meshes/kitchen_new_simple.stl"/>
+        <mesh filename="package://papras_description/meshes/kitchen_simple.stl"/>
       </geometry>
     </collision>
-    <inertial>
-      <origin xyz="0.0 0.0 0.5" rpy="0 0 0" />
-      <mass value="100.0" />
-      <inertia ixx="1.0" ixy="0.0" ixz="0.0" iyy="1.0" iyz="0.0" izz="1.0" />
-    </inertial>
   </link>
-  <!-- Arms -->
-  <xacro:omp_arm id="1"/>
+  <joint name="robot1/env_arm_fixed" type="fixed">
+    <parent link="env"/>
+    <child link="robot1/link1"/>
+    <origin xyz="-0.07009 0.03648 0.78111" rpy="${pi} ${-0.5*pi} 0"/>
+  </joint>
+  <xacro:papras_arm_long id="1"/>
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
Commit message: updated kitchen stl to be accurate w.r.t. sink cavity

File: papras_description/urdf/kitchen.urdf.xacro (robot description, xacro)
@@ -26,5 +26,5 @@
     <parent link="env"/>
     <child link="robot1/link1"/>
-    <origin xyz="-0.07009 0.03648 0.78111" rpy="${pi} ${-0.5*pi} 0"/>
+    <origin xyz="-0.06229 0.01597 0.85252" rpy="${pi} ${-0.5*pi} 0"/>
   </joint>
   <xacro:papras_arm_long id="1"/>
