Commit message: soft gripper experiment works for all objects

File: papras_description/urdf/papras_macros.xacro (robot description, xacro)
@@ -681,5 +681,5 @@
     <xacro:RefLink ref="robot${id}/gripper_body"/>
     <!-- jaw joint -->
-    <joint name="robot${id}/jaw" type="revolute">
+    <joint name="robot${id}/soft_gripper_jaw" type="revolute">
       <axis xyz="0 1 0" />
       <origin xyz="0.06625 -0.019 0.01425" rpy="0 0 0"/>
@@ -714,5 +714,5 @@
     <xacro:RefLink ref="robot${id}/gripper_jaw"/>
     <!-- pulley joint -->
-    <joint name="robot${id}/pulley" type="revolute">
+    <joint name="robot${id}/soft_gripper_pulley" type="revolute">
       <axis xyz="0 0 1" />
       <origin xyz="0.01675 0 0.015" rpy="0 0 0"/>
@@ -817,5 +817,5 @@
     <xacro:RefLink ref="robot${id}/gripper_body"/>
     <!-- jaw joint -->
-    <joint name="robot${id}/jaw" type="revolute">
+    <joint name="robot${id}/soft_gripper_jaw" type="revolute">
       <axis xyz="0 1 0" />
       <origin xyz="0.06625 0.019 0.00975" rpy="0 0 0"/>
@@ -850,5 +850,5 @@
     <xacro:RefLink ref="robot${id}/gripper_jaw"/>
     <!-- pulley joint -->
-    <joint name="robot${id}/pulley" type="revolute">
+    <joint name="robot${id}/soft_gripper_pulley" type="revolute">
       <axis xyz="0 0 -1" />
       <origin xyz="0.01675 0 -0.015" rpy="0 0 0"/>
@@ -917,5 +917,5 @@
       <parent link="robot${id}/gripper_body"/>
       <child link="robot${id}/camera_link"/>
-      <origin xyz="0.07755 0 0.0545" rpy="-1.57 0 0"/>
+      <origin xyz="0.07755 0 0.0545" rpy="0 -1.57 3.14"/>
     </joint>
     <!-- Camera Link -->

Commit message: Added cameras to tea table
- Rotated camera_link frame to match OpenCV conventions

File: papras_description/urdf/papras_macros.xacro (robot description, xacro)
@@ -927,10 +927,10 @@
       <parent link="robot${id}/gripper_main_link"/>
       <child link="robot${id}/camera_link"/>
-      <origin xyz="0.0592 0.0167 0.04452" rpy="0 0 0" />
+      <origin xyz="0.0592 0.0167 0.04452" rpy="${-0.5*pi} 0 ${-0.5*pi}" />
     </joint>
     <!-- Camera Link -->
     <link name="robot${id}/camera_link">
       <visual>
-        <origin xyz="0 0 0" rpy="0 0 0" />
+        <origin xyz="0 0 0" rpy="${0.5*pi} ${-0.5*pi} 0" />
         <geometry>
           <mesh filename="package://papras_description/meshes/camera_mount.stl"/>
@@ -938,5 +938,5 @@
       </visual>
       <collision>
-        <origin xyz="0 0 0" rpy="0 0 0" />
+        <origin xyz="0 0 0" rpy="${0.5*pi} ${-0.5*pi} 0" />
         <geometry>
           <mesh filename="package://papras_description/meshes/camera_mount_simple.stl"/>
@@ -944,5 +944,5 @@
       </collision>
       <inertial>
-        <origin xyz="0 0 0" rpy="0 0 0"/>
+        <origin xyz="0 0 0" rpy="${0.5*pi} ${-0.5*pi} 0"/>
         <mass value="0.088"/>
         <inertia ixx="1.0" ixy="0.0" ixz="0.0" iyy="1.0" iyz="0.0" izz="1.0" />

File: papras_description/urdf/tea_table.urdf.xacro (robot description, xacro)
@@ -35,5 +35,7 @@
   <xacro:papras_arm id="1"/>
   <xacro:papras_gripper id="1"/>
+  <xacro:papras_camera id="1"/>
   <xacro:papras_arm id="2"/>
   <xacro:papras_gripper id="2"/>
+  <xacro:papras_camera id="2"/>
 </robot>

Commit message: change long arm joint 3 limits from [-pi, pi/2]  to [-pi/2, pi/2]

File: papras_description/urdf/papras_macros.xacro (robot description, xacro)
@@ -384,5 +384,5 @@
       <origin xyz="0.03000 -0.01200 0.31400" rpy="0 0 0"/>
       <axis xyz="0 1 0"/>
-      <limit velocity="6.5" effort="1000" lower="${-pi*1.0}" upper="${pi*0.5}" />
+      <limit velocity="6.5" effort="1000" lower="${-pi*0.5}" upper="${pi*0.5}" />
       <dynamics damping="0.7"/>
     </joint>

Commit message: multi-arm pick and place to roomba working on big table

File: papras_description/urdf/papras_macros.xacro (robot description, xacro)
@@ -625,5 +625,5 @@
         <material name="red"/>
       </visual>
-      <collision>
+      <!-- <collision>
         <origin xyz="0.0 0.0 0.0" rpy="0 0 0" />
         <geometry>
@@ -631,5 +631,5 @@
         </geometry>
         <material name="red"/>
-      </collision>
+      </collision> -->
       <inertial>
         <origin xyz="0.0 0.0 0.0" rpy="0 0 0" />

Commit message: add stl files

File: papras_description/urdf/papras_macros.xacro (robot description, xacro)
@@ -651,140 +651,4 @@
     </gazebo>
   </xacro:macro>
-  <xacro:macro name="papras_soft_gripper" params="id">
-    <!-- gripper main fixed joint-->
-    <joint name="robot${id}/end_link_fixed" type="fixed">
-      <parent link="robot${id}/end_link"/>
-      <child link="robot${id}/gripper_body"/>
-      <origin xyz="0.006 0.0 0.0" rpy="0 0 0" />
-    </joint>
-    <!-- gripper body -->
-    <link name="robot${id}/gripper_body">
-      <visual>
-        <origin xyz="0 0 0" rpy="1.57 0 0" />
-        <geometry>
-          <mesh filename="package://papras_description/meshes/soft_gripper_body.stl"/>
-        </geometry>
-        <material name="grey"/>
-      </visual>
-      <collision>
-        <origin xyz="0 0 0" rpy="1.57 0 0" />
-        <geometry>
-          <mesh filename="package://papras_description/meshes/soft_gripper_body_simple.stl"/>
-        </geometry>
-      </collision>
-      <inertial>
-        <origin xyz="0.0 0.0 0.0" rpy="0 0 0"/>
-        <mass value="0.343"/>
-        <inertia ixx="1.0" ixy="0.0" ixz="0.0" iyy="1.0" iyz="0.0" izz="1.0" />
-      </inertial>
-    </link>
-    <xacro:RefLink ref="robot${id}/gripper_body"/>
-    <!-- jaw joint -->
-    <joint name="robot${id}/soft_gripper_jaw" type="revolute">
-      <axis xyz="0 1 0" />
-      <origin xyz="0.06625 -0.019 0.01425" rpy="0 0 0"/>
-      <parent link="robot${id}/gripper_body"/>
-      <child link="robot${id}/gripper_jaw"/>
-      <limit velocity="6.5" effort="1000" lower="0.0" upper="1.4" />
-      <dynamics damping="0.1" friction="0.0" />
-    </joint>
-    <xacro:SimpleTransmissionEffort n="jaw" joint="jaw" id="${id}"/>
-    <!-- gripper jaw link -->
-    <link name="robot${id}/gripper_jaw">
-      <visual>
-        <origin xyz="0 0 0" rpy="1.57 -1.4 0" />
-        <geometry>
-          <mesh filename="package://papras_description/meshes/soft_gripper_jaw.stl"/>
-        </geometry>
-        <material name="grey"/>
-      </visual>
-      <collision>
-        <origin xyz="0 0 0" rpy="1.57 -1.4 0" />
-        <geometry>
-          <mesh filename="package://papras_description/meshes/soft_gripper_jaw_simple.stl"/>
-        </geometry>
-        <material name="grey"/>
-      </collision>
-      <inertial>
-        <origin xyz="0 0 0" rpy="0 0 0"/>
-        <mass value="0.034"/>
-        <inertia ixx="1.0" ixy="0.0" ixz="0.0" iyy="1.0" iyz="0.0" izz="1.0" />
-      </inertial>
-    </link>
-    <xacro:RefLink ref="robot${id}/gripper_jaw"/>
-    <!-- pulley joint -->
-    <joint name="robot${id}/soft_gripper_pulley" type="revolute">
-      <axis xyz="0 0 1" />
-      <origin xyz="0.01675 0 0.015" rpy="0 0 0"/>
-      <parent link="robot${id}/gripper_body"/>
-      <child link="robot${id}/gripper_pulley"/>
-      <limit velocity="6.5" effort="1000" lower="0.0" upper="0.9" />
-      <dynamics damping="0.1" friction="0.0" />
-    </joint>
-    <xacro:SimpleTransmissionEffort n="pulley" joint="pulley" id="${id}"/>
-    <!-- gripper pulley link -->
-    <link name="robot${id}/gripper_pulley">
-      <visual>
-        <origin xyz="0 0 0" rpy="0 0 0" />
-        <geometry>
-          <mesh filename="package://papras_description/meshes/soft_gripper_pulley.stl"/>
-        </geometry>
-        <material name="grey"/>
-      </visual>
-      <collision>
-        <origin xyz="0 0 0" rpy="0 0 0" />
-        <geometry>
-          <mesh filename="package://papras_description/meshes/soft_gripper_pulley_simple.stl"/>
-        </geometry>
-        <material name="grey"/>
-      </collision>
-      <inertial>
-        <origin xyz="0 0 0" rpy="0 0 0"/>
-        <mass value="0.007"/>
-        <inertia ixx="1.0" ixy="0.0" ixz="0.0" iyy="1.0" iyz="0.0" izz="1.0" />
-      </inertial>
-    </link>
-    <xacro:RefLink ref="robot${id}/gripper_sub_link"/>
-    <!-- gripper main fixed joint-->
-    <joint name="robot${id}/end_effector_joint" type="fixed">
-      <parent link="robot${id}/gripper_body"/>
-      <child link="robot${id}/end_effector_link"/>
-      <origin xyz="0.17 0.0 0.02" rpy="0 0 0" />
-    </joint>
-    <!-- End Effector -->
-    <link name="robot${id}/end_effector_link">
-      <visual>
-        <origin xyz="0.0 0.0 0.0" rpy="0 0 0" />
-        <geometry>
-          <box size = "0.01 0.01 0.01"/>
-        </geometry>
-        <material name="red"/>
-      </visual>
-      <collision>
-        <origin xyz="0.0 0.0 0.0" rpy="0 0 0" />
-        <geometry>
-          <box size = "0.01 0.01 0.01"/>
-        </geometry>
-        <material name="red"/>
-      </collision>
-      <inertial>
-        <origin xyz="0.0 0.0 0.0" rpy="0 0 0" />
-        <mass value="0.001" />
-        <inertia ixx="1.0" ixy="0.0" ixz="0.0" iyy="1.0" iyz="0.0" izz="1.0" />
-      </inertial>
-    </link>
-    <gazebo reference="robot${id}/end_effector_link">
-      <material>Gazebo/Red</material>
-    </gazebo>
-    <gazebo>
-      <!-- loading plugin: mimic joints works in gazebo now -->
-      <plugin name="gazebo_gripper${id}_ros_control" filename="libroboticsgroup_gazebo_mimic_joint_plugin.so">
-        <joint>robot${id}/gripper</joint>
-        <mimicJoint>robot${id}/gripper_sub</mimicJoint>
-        <multiplier>1.0</multiplier>
-        <offset>0.0</offset>
-      </plugin>
-    </gazebo>
-  </xacro:macro>
   <xacro:macro name="papras_soft_gripper_v2" params="id">
     <!-- gripper main fixed joint-->
@@ -822,8 +686,8 @@
       <parent link="robot${id}/gripper_body"/>
       <child link="robot${id}/gripper_jaw"/>
-      <limit velocity="6.5" effort="1000" lower="0.0" upper="1.7" />
+      <limit velocity="6.5" effort="1000" lower="0.0" upper="1.78" />
       <dynamics damping="0.1" friction="0.0" />
     </joint>
-    <xacro:SimpleTransmissionEffort n="jaw" joint="jaw" id="${id}"/>
+    <xacro:SimpleTransmissionEffort n="soft_gripper_jaw" joint="soft_gripper_jaw" id="${id}"/>
     <!-- gripper jaw link -->
     <link name="robot${id}/gripper_jaw">
@@ -858,5 +722,5 @@
       <dynamics damping="0.1" friction="0.0" />
     </joint>
-    <xacro:SimpleTransmissionEffort n="pulley" joint="pulley" id="${id}"/>
+    <xacro:SimpleTransmissionEffort n="soft_gripper_pulley" joint="soft_gripper_pulley" id="${id}"/>
     <!-- gripper pulley link -->
     <link name="robot${id}/gripper_pulley">

Commit message: changed camera color to grey

File: papras_description/urdf/papras_macros.xacro (robot description, xacro)
@@ -800,4 +800,5 @@
           <mesh filename="package://papras_description/meshes/camera_mount.stl"/>
         </geometry>
+        <material name="grey"/>
       </visual>
       <collision>

Commit message: add multiturn urdf macro

File: papras_description/urdf/papras_macros.xacro (robot description, xacro)
@@ -514,4 +514,232 @@
     <xacro:RefLink ref="robot${id}/end_link"/>
   </xacro:macro>
+  <xacro:macro name="papras_arm_multiturn" params="id">
+    <!-- link 1 -->
+    <link name="robot${id}/link1">
+      <visual>
+        <origin xyz="0 0 0" rpy="0 0 0"/>
+        <geometry>
+          <mesh filename="package://papras_description/meshes/link1.stl" scale="0.001 0.001 0.001"/>
+        </geometry>
+        <material name="grey"/>
+      </visual>
+      <collision>
+        <origin xyz="0 0 0" rpy="0 0 0"/>
+        <geometry>
+          <mesh filename="package://papras_description/meshes/link1.stl" scale="0.001 0.001 0.001"/>
+        </geometry>
+      </collision>
+      <inertial>
+        <origin xyz="0.00023 0.00000 0.06223" rpy="0 0 0"/>
+        <mass value="0.85644"/>
+        <inertia ixx="1.0" ixy="0.0" ixz="0.0" iyy="1.0" iyz="0.0" izz="1.0" />
+        <!--<inertia ixx="0.00121064" ixy="0.0" ixz="0.00001100" iyy="0.00120886" iyz="0.0" izz="0.00038103" />-->
+      </inertial>
+    </link>
+    <xacro:RefLink ref="robot${id}/link1"/>
+    <!-- Joint 1 -->
+    <joint name="robot${id}/joint1" type="revolute">
+      <parent link="robot${id}/link1"/>
+      <child link="robot${id}/link2"/>
+      <origin xyz="0.0 0.0 0.126" rpy="0 0 0"/>
+      <axis xyz="0 0 1"/>
+      <limit velocity="6.5" effort="1000" lower="${-pi*1.0}" upper="${pi*1.0}" />
+      <dynamics damping="0.7"/>
+    </joint>
+    <xacro:SimpleTransmissionPosition n="1" joint="joint1" id="${id}" />
+    <!-- link 2 -->
+    <link name="robot${id}/link2">
+      <visual>
+        <origin xyz="0 0 0" rpy="0 0 0"/>
+        <geometry>
+          <mesh filename="package://papras_description/meshes/link2.stl" scale="0.001 0.001 0.001"/>
+        </geometry>
+        <material name="grey"/>
+      </visual>
+      <collision>
+        <origin xyz="0 0 0" rpy="0 0 0"/>
+        <geometry>
+          <mesh filename="package://papras_description/meshes/link2.stl" scale="0.001 0.001 0.001"/>
+        </geometry>
+      </collision>
+      <inertial>
+        <origin xyz="0.00000 0.00080 0.03183" rpy="0 0 0"/>
+        <!--<origin xyz="0.00000 -0.06820 -0.00117" rpy="0 0 0"/>-->
+        <mass value="0.94658"/>
+        <inertia ixx="1.0" ixy="0.0" ixz="0.0" iyy="1.0" iyz="0.0" izz="1.0" />
+        <!--<inertia ixx="0.00152547" ixy="0.0" ixz="0.0" iyy="0.00045954" iyz="-0.00001086" izz="0.00151740" />-->
+      </inertial>
+    </link>
+    <xacro:RefLink ref="robot${id}/link2"/>
+    <!-- Joint 2 -->
+    <joint name="robot${id}/joint2" type="revolute">
+      <parent link="robot${id}/link2"/>
+      <child link="robot${id}/link3"/>
+      <origin xyz="0.0 0.069 0.033" rpy="0 0 0"/>
+      <axis xyz="0 1 0"/>
+      <limit velocity="6.5" effort="1000" lower="-2.0" upper="2.0" />
+      <dynamics damping="0.7"/>
+    </joint>
+    <xacro:SimpleTransmissionPosition n="2" joint="joint2" id="${id}" />
+    <!-- link 3 -->
+    <link name="robot${id}/link3">
+      <visual>
+        <origin xyz="0.067 0.008 -0.019" rpy="0 0 3.14"/>
+        <geometry>
+          <mesh filename="package://papras_description/meshes/link3_papras.stl" scale="0.001 0.001 0.001"/>
+        </geometry>
+        <material name="grey"/>
+      </visual>
+      <collision>
+        <origin xyz="0.067 0.008 -0.019" rpy="0 0 3.14"/>
+        <geometry>
+          <mesh filename="package://papras_description/meshes/link3_papras_simple.stl" scale="0.001 0.001 0.001"/>
+        </geometry>
+      </collision>
+      <inertial>
+        <origin xyz="0.01768 -0.06881 0.20524" rpy="0 0 0"/>
+        <!--<origin xyz="-0.01232 -0.05731 -0.05876" rpy="0 0 0"/>-->
+        <mass value="1.30260"/>
+        <inertia ixx="1.0" ixy="0.0" ixz="0.0" iyy="1.0" iyz="0.0" izz="1.0" />
+        <!--<inertia ixx="0.01111021" ixy="0.00001331" ixz="-0.00134208" iyy="0.01046642" iyz="0.00016235" izz="0.00202081" />-->
+      </inertial>
+    </link>
+    <xacro:RefLink ref="robot${id}/link3"/>
+    <!-- Joint 3 -->
+    <joint name="robot${id}/joint3" type="revolute">
+      <parent link="robot${id}/link3"/>
+      <child link="robot${id}/link4"/>
+      <origin xyz="0.03000 -0.01150 0.26400" rpy="0 0 0"/>
+      <axis xyz="0 1 0"/>
+      <limit velocity="6.5" effort="1000" lower="${-pi*1.0}" upper="${pi*0.5}" />
+      <dynamics damping="0.7"/>
+    </joint>
+    <xacro:SimpleTransmissionPosition n="3" joint="joint3" id="${id}" />
+    <!-- link 4 -->
+    <link name="robot${id}/link4">
+      <visual>
+        <origin xyz="0.227 0.0085 -0.024" rpy="0 0 3.14"/>
+        <geometry>
+          <mesh filename="package://papras_description/meshes/link4_papras.stl" scale="0.001 0.001 0.001"/>
+        </geometry>
+        <material name="grey"/>
+      </visual>
+      <collision>
+        <origin xyz="0.227 0.0085 -0.024" rpy="0 0 3.14"/>
+        <geometry>
+          <mesh filename="package://papras_description/meshes/link4_papras_simple.stl" scale="0.001 0.001 0.001"/>
+        </geometry>
+      </collision>
+      <inertial>
+        <origin xyz="0.12475 -0.05716 0.02979" rpy="0 0 0"/>
+        <!--<origin xyz="-0.07025 0.00034 -0.00021" rpy="0 0 0"/>-->
+        <mass value="1.15977"/>
+        <inertia ixx="1.0" ixy="0.0" ixz="0.0" iyy="1.0" iyz="0.0" izz="1.0" />
+        <!--<inertia ixx="0.00096726" ixy="0.00004383" ixz="-0.00002771" iyy="0.00318801" iyz="0.00000627" izz="0.00341484" />-->
+      </inertial>
+    </link>
+    <xacro:RefLink ref="robot${id}/link4"/>
+    <!-- Joint 4 -->
+    <joint name="robot${id}/joint4" type="revolute">
+      <parent link="robot${id}/link4"/>
+      <child link="robot${id}/link5"/>
+      <origin xyz="0.19500 -0.05750 0.03000" rpy="0 0 0"/>
+      <axis xyz="1 0 0"/>
+      <limit velocity="6.5" effort="1000" lower="${-pi*0.875}" upper="${pi*0.875}" />
+      <dynamics damping="0.7"/>
+    </joint>
+    <xacro:SimpleTransmissionPosition n="4" joint="joint4" id="${id}" />
+    <!-- link 5 -->
+    <link name="robot${id}/link5">
+      <visual>
+        <origin xyz="0 0 0" rpy="0 0 0"/>
+        <geometry>
+          <mesh filename="package://papras_description/meshes/link5.stl" scale="0.001 0.001 0.001"/>
+        </geometry>
+        <material name="grey"/>
+      </visual>
+      <collision>
+        <origin xyz="0 0 0" rpy="0 0 0"/>
+        <geometry>
+          <mesh filename="package://papras_description/meshes/link5.stl" scale="0.001 0.001 0.001"/>
+        </geometry>
+      </collision>
+      <inertial>
+        <origin xyz="0.05642 -0.00217 0.00002" rpy="0 0 0"/>
+        <!--<origin xyz="-0.00658 -0.04717 0.00002" rpy="0 0 0"/>-->
+        <mass value="0.44688"/>
+        <inertia ixx="1.0" ixy="0.0" ixz="0.0" iyy="1.0" iyz="0.0" izz="1.0" />
+        <!--<inertia ixx="0.00030285" ixy="0.00000761" ixz="0.00000031" iyy="0.00022339" iyz="-0.00000001" izz="0.00039766" />-->
+      </inertial>
+    </link>
+    <xacro:RefLink ref="robot${id}/link5"/>
+    <!-- Joint 5 -->
+    <joint name="robot${id}/joint5" type="revolute">
+      <parent link="robot${id}/link5"/>
+      <child link="robot${id}/link6"/>
+      <origin xyz="0.06300 0.04500 0.00000" rpy="0 0 0"/>
+      <axis xyz="0 1 0"/>
+      <limit velocity="6.5" effort="1000" lower="${-pi*0.5}" upper="${pi*0.5}" />
+      <dynamics damping="0.7"/>
+    </joint>
+    <xacro:SimpleTransmissionPosition n="5" joint="joint5" id="${id}" />
+    <!-- link 6 -->
+    <link name="robot${id}/link6">
+      <visual>
+        <origin xyz="-0.034 -0.098 -0.028" rpy="0 0 0"/>
+        <geometry>
+          <mesh filename="package://papras_description/meshes/link6_papras.stl" scale="0.001 0.001 0.001"/>
+        </geometry>
+        <material name="grey"/>
+      </visual>
+      <collision>
+        <origin xyz="-0.034 -0.098 -0.028" rpy="0 0 0"/>
+        <geometry>
+          <mesh filename="package://papras_description/meshes/link6_papras_simple.stl" scale="0.001 0.001 0.001"/>
+        </geometry>
+      </collision>
+      <inertial>
+        <origin xyz="0.06831 -0.04457 0.00000" rpy="0 0 0"/>
+        <!--<origin xyz="-0.05469 0.00043 0.00000" rpy="0 0 0"/>-->
+        <mass value="0.43273"/>
+        <inertia ixx="1.0" ixy="0.0" ixz="0.0" iyy="1.0" iyz="0.0" izz="1.0" />
+        <!--<inertia ixx="0.00021512" ixy="0.00001009" ixz="0.00000000" iyy="0.00042827" iyz="0.00000000" izz="0.00051436" />-->
+      </inertial>
+    </link>
+    <xacro:RefLink ref="robot${id}/link6"/>
+    <!-- Joint 6 -->
+    <joint name="robot${id}/joint6" type="continuous">
+      <parent link="robot${id}/link6"/>
+      <child link="robot${id}/end_link"/>
+      <origin xyz="0.12300 -0.04500 0.00000" rpy="0 0 0"/>
+      <axis xyz="1 0 0"/>
+      <limit velocity="6.5" effort="1000"/>
+      <dynamics damping="0.7"/>
+    </joint>
+    <xacro:SimpleTransmissionPosition n="6" joint="joint6" id="${id}" />
+    <!-- end link -->
+    <link name="robot${id}/end_link">
+      <visual>
+        <origin xyz="0.0 0.0 0.0" rpy="0 0 0" />
+        <geometry>
+          <mesh filename="package://papras_description/meshes/end_link.stl" scale="0.001 0.001 0.001"/>
+        </geometry>
+        <material name="grey"/>
+      </visual>
+      <collision>
+        <origin xyz="0.0 0.0 0.0" rpy="0 0 0" />
+        <geometry>
+          <mesh filename="package://papras_description/meshes/end_link.stl" scale="0.001 0.001 0.001"/>
+        </geometry>
+      </collision>
+      <inertial>
+        <origin xyz="0.00337 0.00000 0.00000" rpy="0 0 0"/>
+        <mass value="0.01919"/>
+        <inertia ixx="1.0" ixy="0.0" ixz="0.0" iyy="1.0" iyz="0.0" izz="1.0" />
+        <!--<inertia ixx="0.00000938" ixy="0.0" ixz="0.0" iyy="0.00000338" iyz="0.0" izz="0.00000635" />-->
+      </inertial>
+    </link>
+    <xacro:RefLink ref="robot${id}/end_link"/>
+  </xacro:macro>
   <xacro:macro name="papras_gripper" params="id">
     <!-- gripper main fixed joint-->

Commit message: updated vel limit j6

File: papras_description/urdf/papras_macros.xacro (robot description, xacro)
@@ -25,4 +25,6 @@
       <minDepth>0.001</minDepth>
       <material>Gazebo/White</material>
+      <selfCollide>1</selfCollide>
+      <dampingFactor>0.01</dampingFactor>
     </gazebo>
   </xacro:macro>
@@ -714,5 +716,5 @@
       <origin xyz="0.12300 -0.04500 0.00000" rpy="0 0 0"/>
       <axis xyz="1 0 0"/>
-      <limit velocity="6.5" effort="1000"/>
+      <limit velocity="3.057" effort="1000"/>
       <dynamics damping="0.7"/>
     </joint>
