Commit message: change vel limits for all joints

File: papras_description/urdf/papras_macros.xacro (robot description, xacro)
@@ -90,5 +90,5 @@
       <origin xyz="0.0 0.0 0.126" rpy="0 0 0"/>
       <axis xyz="0 0 1"/>
-      <limit velocity="6.5" effort="1000" lower="${-pi*1.0}" upper="${pi*1.0}" />
+      <limit velocity="3.03687" effort="100" lower="${-pi*1.0}" upper="${pi*1.0}" />
       <dynamics damping="0.7"/>
     </joint>
@@ -124,5 +124,5 @@
       <origin xyz="0.0 0.069 0.033" rpy="0 0 0"/>
       <axis xyz="0 1 0"/>
-      <limit velocity="6.5" effort="1000" lower="-2.0" upper="2.0" />
+      <limit velocity="3.03687" effort="100" lower="-2.0" upper="2.0" />
       <dynamics damping="0.7"/>
     </joint>
@@ -158,5 +158,5 @@
       <origin xyz="0.03000 -0.01150 0.26400" rpy="0 0 0"/>
       <axis xyz="0 1 0"/>
-      <limit velocity="6.5" effort="1000" lower="${-pi*1.0}" upper="${pi*0.5}" />
+      <limit velocity="3.03687" effort="100" lower="${-pi*1.0}" upper="${pi*0.5}" />
       <dynamics damping="0.7"/>
     </joint>
@@ -192,5 +192,5 @@
       <origin xyz="0.19500 -0.05750 0.03000" rpy="0 0 0"/>
       <axis xyz="1 0 0"/>
-      <limit velocity="6.5" effort="1000" lower="${-pi*0.875}" upper="${pi*0.875}" />
+      <limit velocity="3.03687" effort="100" lower="${-pi*0.875}" upper="${pi*0.875}" />
       <dynamics damping="0.7"/>
     </joint>
@@ -226,5 +226,5 @@
       <origin xyz="0.06300 0.04500 0.00000" rpy="0 0 0"/>
       <axis xyz="0 1 0"/>
-      <limit velocity="6.5" effort="1000" lower="${-pi*0.5}" upper="${pi*0.5}" />
+      <limit velocity="3.03687" effort="100" lower="${-pi*0.5}" upper="${pi*0.5}" />
       <dynamics damping="0.7"/>
     </joint>
@@ -260,5 +260,5 @@
       <origin xyz="0.12300 -0.04500 0.00000" rpy="0 0 0"/>
       <axis xyz="1 0 0"/>
-      <limit velocity="6.5" effort="1000" lower="${-pi*1.0}" upper="${pi*1.0}" />
+      <limit velocity="3.03687" effort="100" lower="${-pi*1.0}" upper="${pi*1.0}" />
       <dynamics damping="0.7"/>
     </joint>
@@ -318,5 +318,5 @@
       <origin xyz="0.0 0.0 0.126" rpy="0 0 0"/>
       <axis xyz="0 0 1"/>
-      <limit velocity="6.5" effort="1000" lower="${-pi*1.0}" upper="${pi*1.0}" />
+      <limit velocity="3.03687" effort="100" lower="${-pi*1.0}" upper="${pi*1.0}" />
       <dynamics damping="0.7"/>
     </joint>
@@ -352,5 +352,5 @@
       <origin xyz="0.0 0.069 0.033" rpy="0 0 0"/>
       <axis xyz="0 1 0"/>
-      <limit velocity="6.5" effort="1000" lower="-2.0" upper="2.0" />
+      <limit velocity="3.03687" effort="100" lower="-2.0" upper="2.0" />
       <dynamics damping="0.7"/>
     </joint>
@@ -386,5 +386,5 @@
       <origin xyz="0.03000 -0.01200 0.31400" rpy="0 0 0"/>
       <axis xyz="0 1 0"/>
-      <limit velocity="6.5" effort="1000" lower="${-pi*0.5}" upper="${pi*0.5}" />
+      <limit velocity="3.03687" effort="100" lower="${-pi*0.5}" upper="${pi*0.5}" />
       <dynamics damping="0.7"/>
     </joint>
@@ -420,5 +420,5 @@
       <origin xyz="0.24500 -0.05750 0.03000" rpy="0 0 0"/>
       <axis xyz="1 0 0"/>
-      <limit velocity="6.5" effort="1000" lower="${-pi*0.875}" upper="${pi*0.875}" />
+      <limit velocity="3.03687" effort="100" lower="${-pi*0.875}" upper="${pi*0.875}" />
       <dynamics damping="0.7"/>
     </joint>
@@ -454,5 +454,5 @@
       <origin xyz="0.06300 0.04500 0.00000" rpy="0 0 0"/>
       <axis xyz="0 1 0"/>
-      <limit velocity="6.5" effort="1000" lower="${-pi*0.5}" upper="${pi*0.5}" />
+      <limit velocity="3.03687" effort="100" lower="${-pi*0.5}" upper="${pi*0.5}" />
       <dynamics damping="0.7"/>
     </joint>
@@ -488,5 +488,5 @@
       <origin xyz="0.12300 -0.04500 0.00000" rpy="0 0 0"/>
       <axis xyz="1 0 0"/>
-      <limit velocity="6.5" effort="1000" lower="${-pi*1.0}" upper="${pi*1.0}" />
+      <limit velocity="3.03687" effort="100" lower="${-pi*1.0}" upper="${pi*1.0}" />
       <dynamics damping="0.7"/>
     </joint>
@@ -546,5 +546,5 @@
       <origin xyz="0.0 0.0 0.126" rpy="0 0 0"/>
       <axis xyz="0 0 1"/>
-      <limit velocity="6.5" effort="1000" lower="${-pi*1.0}" upper="${pi*1.0}" />
+      <limit velocity="3.03687" effort="100" lower="${-pi*1.0}" upper="${pi*1.0}" />
       <dynamics damping="0.7"/>
     </joint>
@@ -580,5 +580,5 @@
       <origin xyz="0.0 0.069 0.033" rpy="0 0 0"/>
       <axis xyz="0 1 0"/>
-      <limit velocity="6.5" effort="1000" lower="-2.0" upper="2.0" />
+      <limit velocity="3.03687" effort="100" lower="-2.0" upper="2.0" />
       <dynamics damping="0.7"/>
     </joint>
@@ -614,5 +614,5 @@
       <origin xyz="0.03000 -0.01150 0.26400" rpy="0 0 0"/>
       <axis xyz="0 1 0"/>
-      <limit velocity="6.5" effort="1000" lower="${-pi*1.0}" upper="${pi*0.5}" />
+      <limit velocity="3.03687" effort="100" lower="${-pi*1.0}" upper="${pi*0.5}" />
       <dynamics damping="0.7"/>
     </joint>
@@ -648,5 +648,5 @@
       <origin xyz="0.19500 -0.05750 0.03000" rpy="0 0 0"/>
       <axis xyz="1 0 0"/>
-      <limit velocity="6.5" effort="1000" lower="${-pi*0.875}" upper="${pi*0.875}" />
+      <limit velocity="3.03687" effort="100" lower="${-pi*0.875}" upper="${pi*0.875}" />
       <dynamics damping="0.7"/>
     </joint>
@@ -682,5 +682,5 @@
       <origin xyz="0.06300 0.04500 0.00000" rpy="0 0 0"/>
       <axis xyz="0 1 0"/>
-      <limit velocity="6.5" effort="1000" lower="${-pi*0.5}" upper="${pi*0.5}" />
+      <limit velocity="3.03687" effort="100" lower="${-pi*0.5}" upper="${pi*0.5}" />
       <dynamics damping="0.7"/>
     </joint>
@@ -716,5 +716,5 @@
       <origin xyz="0.12300 -0.04500 0.00000" rpy="0 0 0"/>
       <axis xyz="1 0 0"/>
-      <limit velocity="3.057" effort="1000"/>
+      <limit velocity="3.03687" effort="100"/>
       <dynamics damping="0.7"/>
     </joint>
@@ -779,5 +779,5 @@
       <parent link="robot${id}/gripper_main_link"/>
       <child link="robot${id}/gripper_link"/>
-      <limit velocity="6.5" effort="1000" lower="0.0" upper="1.15" />
+      <limit velocity="3.03687" effort="100" lower="0.0" upper="1.15" />
       <dynamics damping="0.1" friction="0.0" />
     </joint>
@@ -812,5 +812,5 @@
       <parent link="robot${id}/gripper_main_link"/>
       <child link="robot${id}/gripper_sub_link"/>
-      <limit velocity="6.5" effort="1000" lower="0.0" upper="1.15" />
+      <limit velocity="3.03687" effort="100" lower="0.0" upper="1.15" />
       <dynamics damping="0.1" friction="0.0" />
       <mimic joint="robot${id}/gripper" multiplier="1"/>
@@ -916,5 +916,5 @@
       <parent link="robot${id}/gripper_body"/>
       <child link="robot${id}/gripper_jaw"/>
-      <limit velocity="6.5" effort="1000" lower="0.0" upper="1.78" />
+      <limit velocity="3.03687" effort="100" lower="0.0" upper="1.78" />
       <dynamics damping="0.1" friction="0.0" />
     </joint>
@@ -949,5 +949,5 @@
       <parent link="robot${id}/gripper_body"/>
       <child link="robot${id}/gripper_pulley"/>
-      <limit velocity="6.5" effort="1000" lower="0.0" upper="1.59" />
+      <limit velocity="3.03687" effort="100" lower="0.0" upper="1.59" />
       <dynamics damping="0.1" friction="0.0" />
     </joint>

Commit message: add gazebo mimic joint and depth camera plugins to papras macros

File: papras_description/urdf/papras_macros.xacro (robot description, xacro)
@@ -873,5 +873,5 @@
     <gazebo>
       <!-- loading plugin: mimic joints works in gazebo now -->
-      <plugin name="gazebo_gripper${id}_ros_control" filename="libroboticsgroup_gazebo_mimic_joint_plugin.so">
+      <plugin name="gazebo_gripper${id}_ros_control" filename="libroboticsgroup_upatras_gazebo_mimic_joint_plugin.so">
         <joint>robot${id}/gripper</joint>
         <mimicJoint>robot${id}/gripper_sub</mimicJoint>
@@ -1045,4 +1045,62 @@
     </link>
     <xacro:RefLink ref="robot${id}/camera_link"/>
+    <joint name="robot${id}/camera_fixed_plugin_joint" type="fixed">
+      <parent link="robot${id}/camera_link"/>
+      <child link="robot${id}/camera_plugin_link"/>
+      <origin xyz="0 0 0" rpy="${0.5*pi} ${-0.5*pi} 0" />
+    </joint>
+    <link name="robot${id}/camera_plugin_link"/>
+    <xacro:RefLink ref="robot${id}/camera_plugin_link"/>
+    <gazebo reference="robot${id}/camera_plugin_link">
+      <sensor type="depth" name="robot${id}/camera_sensor">
+        <update_rate>30.0</update_rate>
+        <camera name="head">
+          <horizontal_fov>1.3962634</horizontal_fov>
+          <image>
+            <width>640</width>
+            <height>480</height>
+            <format>R8G8B8</format>
+          </image>
+          <clip>
+            <near>0.02</near>
+            <far>300</far>
+          </clip>
+          <noise>
+            <type>gaussian</type>
+            <!-- Noise is sampled independently per pixel on each frame.
+                That pixel's noise value is added to each of its color
+                channels, which at that point lie in the range [0,1]. -->
+            <mean>0.0</mean>
+            <stddev>0.007</stddev>
+          </noise>
+        </camera>
+        <plugin name="camera_plugin" filename="libgazebo_ros_openni_kinect.so">
+          <baseline>0.2</baseline>
+          <alwaysOn>true</alwaysOn>
+          <!-- Keep this zero, update_rate in the parent <sensor> tag
+            will control the frame rate. -->
+          <updateRate>0.0</updateRate>
+          <cameraName>robot${id}/camera</cameraName>
+          <imageTopicName>color/image_raw</imageTopicName>
+          <cameraInfoTopicName>color/camera_info</cameraInfoTopicName>
+          <depthImageTopicName>depth/image_raw</depthImageTopicName>
+          <depthImageCameraInfoTopicName>depth/camera_info</depthImageCameraInfoTopicName>
+          <pointCloudTopicName>depth/points</pointCloudTopicName>
+          <frameName>robot${id}/camera_link</frameName>
+          <pointCloudCutoff>0.1</pointCloudCutoff>
+          <pointCloudCutoffMax>3.0</pointCloudCutoffMax>
+          <distortionK1>0</distortionK1>
+          <distortionK2>0</distortionK2>
+          <distortionK3>0</distortionK3>
+          <distortionT1>0</distortionT1>
+          <distortionT2>0</distortionT2>
+          <CxPrime>0</CxPrime>
+          <Cx>0</Cx>
+          <Cy>0</Cy>
+          <focalLength>0</focalLength>
+          <hackBaseline>0</hackBaseline>
+        </plugin>
+      </sensor>
+    </gazebo>
   </xacro:macro>
 </robot>

Commit message: Proper description folder

File: papras_description/urdf/papras_macros.xacro (robot description, xacro)
@@ -881,139 +881,4 @@
     </gazebo>
   </xacro:macro>
-  <xacro:macro name="papras_soft_gripper_v2" params="id">
-    <!-- gripper main fixed joint-->
-    <joint name="robot${id}/end_link_fixed" type="fixed">
-      <parent link="robot${id}/end_link"/>
-      <child link="robot${id}/gripper_body"/>
-      <origin xyz="0.006 0.0 0.0" rpy="0 0 0" />
-    </joint>
-    <!-- gripper body -->
-    <link name="robot${id}/gripper_body">
-      <visual>
-        <origin xyz="0 0 0" rpy="0 0 0" />
-        <geometry>
-          <mesh filename="package://papras_description/meshes/soft_gripper_body_v2.stl"/>
-        </geometry>
-        <material name="grey"/>
-      </visual>
-      <collision>
-        <origin xyz="0 0 0" rpy="0 0 0" />
-        <geometry>
-          <mesh filename="package://papras_description/meshes/soft_gripper_body_v2_simple.stl"/>
-        </geometry>
-      </collision>
-      <inertial>
-        <origin xyz="0.0 0.0 0.0" rpy="0 0 0"/>
-        <mass value="0.343"/>
-        <inertia ixx="1.0" ixy="0.0" ixz="0.0" iyy="1.0" iyz="0.0" izz="1.0" />
-      </inertial>
-    </link>
-    <xacro:RefLink ref="robot${id}/gripper_body"/>
-    <!-- jaw joint -->
-    <joint name="robot${id}/soft_gripper_jaw" type="revolute">
-      <axis xyz="0 1 0" />
-      <origin xyz="0.06625 0.019 0.00975" rpy="0 0 0"/>
-      <parent link="robot${id}/gripper_body"/>
-      <child link="robot${id}/gripper_jaw"/>
-      <limit velocity="3.03687" effort="100" lower="0.0" upper="1.78" />
-      <dynamics damping="0.1" friction="0.0" />
-    </joint>
-    <xacro:SimpleTransmissionEffort n="soft_gripper_jaw" joint="soft_gripper_jaw" id="${id}"/>
-    <!-- gripper jaw link -->
-    <link name="robot${id}/gripper_jaw">
-      <visual>
-        <origin xyz="0 0 0" rpy="3.14 0 1.57" />
-        <geometry>
-          <mesh filename="package://papras_description/meshes/soft_gripper_jaw_v2.stl"/>
-        </geometry>
-        <material name="grey"/>
-      </visual>
-      <collision>
-        <origin xyz="0 0 0" rpy="3.14 0 1.57" />
-        <geometry>
-          <mesh filename="package://papras_description/meshes/soft_gripper_jaw_v2_simple.stl"/>
-        </geometry>
-        <material name="grey"/>
-      </collision>
-      <inertial>
-        <origin xyz="0 0 0" rpy="0 0 0"/>
-        <mass value="0.034"/>
-        <inertia ixx="1.0" ixy="0.0" ixz="0.0" iyy="1.0" iyz="0.0" izz="1.0" />
-      </inertial>
-    </link>
-    <xacro:RefLink ref="robot${id}/gripper_jaw"/>
-    <!-- pulley joint -->
-    <joint name="robot${id}/soft_gripper_pulley" type="revolute">
-      <axis xyz="0 0 -1" />
-      <origin xyz="0.01675 0 -0.015" rpy="0 0 0"/>
-      <parent link="robot${id}/gripper_body"/>
-      <child link="robot${id}/gripper_pulley"/>
-      <limit velocity="3.03687" effort="100" lower="0.0" upper="1.59" />
-      <dynamics damping="0.1" friction="0.0" />
-    </joint>
-    <xacro:SimpleTransmissionEffort n="soft_gripper_pulley" joint="soft_gripper_pulley" id="${id}"/>
-    <!-- gripper pulley link -->
-    <link name="robot${id}/gripper_pulley">
-      <visual>
-        <origin xyz="0 0 0" rpy="-1.57 0 0" />
-        <geometry>
-          <mesh filename="package://papras_description/meshes/soft_gripper_pulley_v2.stl"/>
-        </geometry>
-        <material name="grey"/>
-      </visual>
-      <collision>
-        <origin xyz="0 0 0" rpy="-1.57 0 0" />
-        <geometry>
-          <mesh filename="package://papras_description/meshes/soft_gripper_pulley_v2_simple.stl"/>
-        </geometry>
-        <material name="grey"/>
-      </collision>
-      <inertial>
-        <origin xyz="0 0 0" rpy="0 0 0"/>
-        <mass value="0.007"/>
-        <inertia ixx="1.0" ixy="0.0" ixz="0.0" iyy="1.0" iyz="0.0" izz="1.0" />
-      </inertial>
-    </link>
-    <xacro:RefLink ref="robot${id}/gripper_pulley"/>
-    <!-- gripper main fixed joint-->
-    <joint name="robot${id}/end_effector_joint" type="fixed">
-      <parent link="robot${id}/gripper_body"/>
-      <child link="robot${id}/end_effector_link"/>
-      <origin xyz="0.188 0.0 -0.014" rpy="0 0 0" />
-    </joint>
-    <!-- End Effector -->
-    <link name="robot${id}/end_effector_link">
-      <visual>
-        <origin xyz="0.0 0.0 0.0" rpy="0 0 0" />
-        <geometry>
-          <box size = "0.01 0.01 0.01"/>
-        </geometry>
-        <material name="red"/>
-      </visual>
-      <collision>
-        <origin xyz="0.0 0.0 0.0" rpy="0 0 0" />
-        <geometry>
-          <box size = "0.01 0.01 0.01"/>
-        </geometry>
-        <material name="red"/>
-      </collision>
-      <inertial>
-        <origin xyz="0.0 0.0 0.0" rpy="0 0 0" />
-        <mass value="0.001" />
-        <inertia ixx="1.0" ixy="0.0" ixz="0.0" iyy="1.0" iyz="0.0" izz="1.0" />
-      </inertial>
-    </link>
-    <gazebo reference="robot${id}/end_effector_link">
-      <material>Gazebo/Red</material>
-    </gazebo>
-    <!-- camera link fixed joint -->
-    <joint name="robot${id}/camera_fixed_joint" type="fixed">
-      <parent link="robot${id}/gripper_body"/>
-      <child link="robot${id}/camera_link"/>
-      <origin xyz="0.07755 0 0.0545" rpy="0 -1.57 3.14"/>
-    </joint>
-    <!-- Camera Link -->
-    <link name="robot${id}/camera_link"/>
-  </xacro:macro>
   <xacro:macro name="papras_camera" params="id">
     <!-- camera link fixed joint -->
