Commit message: added 7dof model and demo

File: papras_description/urdf/papras_macros.xacro (robot description, xacro)
@@ -969,3 +969,937 @@
     </gazebo>
   </xacro:macro>
+  <xacro:macro name="papras_arm_7dof" params="id">
+    <!-- link 1 -->
+    <link name="robot${id}/link1">
+      <visual>
+        <origin xyz="0 0 0" rpy="0 0 0"/>
+        <geometry>
+          <mesh filename="package://papras_description/meshes/link1.stl" scale="0.001 0.001 0.001"/>
+        </geometry>
+        <material name="grey"/>
+      </visual>
+      <collision>
+        <origin xyz="0 0 0" rpy="0 0 0"/>
+        <geometry>
+          <mesh filename="package://papras_description/meshes/link1.stl" scale="0.001 0.001 0.001"/>
+        </geometry>
+      </collision>
+      <inertial>
+        <origin xyz="-0.00205616406 0.00000000 0.07012969338"/>
+        <mass value="0.91200000"/>
+        <inertia ixx="0.00140582306367" ixy="0.00000000" ixz="0.00000000" iyy="0.00140582097352" iyz="-0.00000000" izz="0.00043779331105"/>
+      </inertial>
+    </link>
+    <xacro:RefLink ref="robot${id}/link1"/>
+      <!-- Joint 1 -->
+    <joint name="robot${id}/joint1" type="revolute">
+      <parent link="robot${id}/link1"/>
+      <child link="robot${id}/link2"/>
+      <origin xyz="0.0 0.0 0.126" rpy="0 0 0"/>
+      <axis xyz="0 0 1"/>
+      <limit velocity="3.03687" effort="100" lower="${-pi*1.0}" upper="${pi*1.0}" />
+      <dynamics damping="0.7"/>
+    </joint>
+    <xacro:SimpleTransmissionPosition n="1" joint="joint1" id="${id}" />
+    <!-- link 2 -->
+    <link name="robot${id}/link2">
+      <visual>
+        <origin xyz="0 0 0" rpy="0 0 0"/>
+        <geometry>
+          <mesh filename="package://papras_description/meshes/link2.stl" scale="0.001 0.001 0.001"/>
+        </geometry>
+        <material name="grey"/>
+      </visual>
+      <collision>
+        <origin xyz="0 0 0" rpy="0 0 0"/>
+        <geometry>
+          <mesh filename="package://papras_description/meshes/link2.stl" scale="0.001 0.001 0.001"/>
+        </geometry>
+      </collision>
+      <inertial>
+        <origin xyz="-0.00000000001 -0.01570756882 0.02819237930"/>
+        <mass value="0.88500000"/>
+        <inertia ixx="0.00155754725347" ixy="-0.00000000" ixz="-0.00000000" iyy="0.00048405544236" iyz="-0.00000173296990" izz="0.00154667193282"/>
+      </inertial>
+    </link>
+    <xacro:RefLink ref="robot${id}/link2"/>
+    <!-- Joint 2 -->
+    <joint name="robot${id}/joint2" type="revolute">
+      <parent link="robot${id}/link2"/>
+      <child link="robot${id}/link3"/>
+      <origin xyz="0.0 0.00 0.033" rpy="${pi/2.0} ${-pi/2.0} 0"/>
+      <axis xyz="0 0 1"/>
+      <limit velocity="3.03687" effort="100" lower="-2.0" upper="2.0" />
+      <dynamics damping="0.7"/>
+    </joint>
+    <xacro:SimpleTransmissionPosition n="2" joint="joint2" id="${id}" />
+    <!-- link 2 -->
+    <link name="robot${id}/link3">
+      <visual>
+        <origin xyz="0.0 0.0 0.0" rpy="0 0 0"/>
+        <geometry>
+          <mesh filename="package://papras_description/meshes/7dof/link3.stl"/>
+        </geometry>
+        <material name="grey"/>
+      </visual>
+      <collision>
+        <origin xyz="0 0 0" rpy="0 0 0"/>
+        <geometry>
+          <mesh filename="package://papras_description/meshes/7dof/link3.stl"/>
+        </geometry>
+      </collision>
+      <inertial>
+        <origin xyz="0.10300488 0.00026160 0.00111164"/>
+        <mass value="1.01000000"/>
+        <inertia ixx="0.00182373" ixy="-0.00000000" ixz="-0.00000526" iyy="0.00433189" iyz="0.00000000" izz="0.00310084"/>
+      </inertial>
+    </link>
+    <xacro:RefLink ref="robot${id}/link3"/>
+    <!-- Joint 2 -->
+    <joint name="robot${id}/joint3" type="revolute">
+      <parent link="robot${id}/link3"/>
+      <child link="robot${id}/link4"/>
+      <origin xyz="0.156382198147594 0 0.000400000000010851" rpy="0 ${-pi/2.0} ${-pi/2.0}"/>
+      <axis xyz="0 1 0"/>
+      <limit velocity="3.03687" effort="100" lower="-${pi}" upper="${pi}" />
+      <dynamics damping="0.7"/>
+    </joint>
+    <xacro:SimpleTransmissionPosition n="3" joint="joint3" id="${id}" />
+        <!-- link 2 -->
+    <link name="robot${id}/link4">
+      <visual>
+        <origin xyz="0.0 0.0 0.0" rpy="0 0 0"/>
+        <geometry>
+          <mesh filename="package://papras_description/meshes/7dof/link4.stl"/>
+        </geometry>
+        <material name="grey"/>
+      </visual>
+      <collision>
+        <origin xyz="0 0 0" rpy="0 0 0"/>
+        <geometry>
+          <mesh filename="package://papras_description/meshes/7dof/link4.stl"/>
+        </geometry>
+      </collision>
+      <inertial>
+        <origin xyz="-0.00205466 0.07035925 0.01546531"/>
+        <mass value="0.96600000"/>
+        <inertia ixx="0.00180447" ixy="0.00000423" ixz="0.00000322" iyy="0.00132106" iyz="-0.00029745" izz="0.00211226"/>
+      </inertial>
+    </link>
+    <xacro:RefLink ref="robot${id}/link4"/>
+    <!-- Joint 3 -->
+    <joint name="robot${id}/joint4" type="revolute">
+      <parent link="robot${id}/link4"/>
+      <child link="robot${id}/link5"/>
+      <origin xyz="0.0575 0.10761780185239 0.0300000000000553" rpy="${pi} ${-pi/2.0} ${pi/2.0}"/>
+      <axis xyz="0 1 0"/>
+      <limit velocity="3.03687" effort="100" lower="${-pi*1.0}" upper="1.42" />
+      <dynamics damping="0.7"/>
+    </joint>
+    <xacro:SimpleTransmissionPosition n="4" joint="joint4" id="${id}" />
+    <!-- link 5 -->
+    <link name="robot${id}/link5">
+      <visual>
+        <origin xyz="0.227 0.0085 -0.024" rpy="0 0 3.14"/>
+        <geometry>
+          <mesh filename="package://papras_description/meshes/link4_papras.stl" scale="0.001 0.001 0.001"/>
+        </geometry>
+        <material name="grey"/>
+      </visual>
+      <collision>
+        <origin xyz="0.227 0.0085 -0.024" rpy="0 0 3.14"/>
+        <geometry>
+          <mesh filename="package://papras_description/meshes/link4_papras_simple.stl" scale="0.001 0.001 0.001"/>
+        </geometry>
+      </collision>
+      <inertial>
+        <origin xyz="0.133722 -0.058143 0.028408"/>
+        <!-- <origin xyz="${0.277-0.09327796} 0.06664315 0.05240824" rpy="0 0 3.14"/>                                                                   -->
+        <mass value="1.22500000"/>
+        <inertia ixx="0.00184346" ixy="0.00000031" ixz="-0.00063174" iyy="0.00588246" iyz="0.00000015" izz="0.00647638"/>
+      </inertial>
+    </link>
+    <xacro:RefLink ref="robot${id}/link5"/>
+    <!-- Joint 4 -->
+    <joint name="robot${id}/joint5" type="revolute">
+      <parent link="robot${id}/link5"/>
+      <child link="robot${id}/link6"/>
+      <origin xyz="0.19500 -0.05750 0.03000" rpy="0 0 0"/>
+      <axis xyz="1 0 0"/>
+      <limit velocity="3.03687" effort="100" lower="${-pi*0.875}" upper="${pi*0.875}" />
+      <dynamics damping="0.7"/>
+    </joint>
+    <xacro:SimpleTransmissionPosition n="5" joint="joint5" id="${id}" />
+    <!-- link 6 -->
+    <link name="robot${id}/link6">
+      <visual>
+        <origin xyz="0 0 0" rpy="0 0 0"/>
+        <geometry>
+          <mesh filename="package://papras_description/meshes/link5.stl" scale="0.001 0.001 0.001"/>
+        </geometry>
+        <material name="grey"/>
+      </visual>
+      <collision>
+        <origin xyz="0 0 0" rpy="0 0 0"/>
+        <geometry>
+          <mesh filename="package://papras_description/meshes/link5.stl" scale="0.001 0.001 0.001"/>
+        </geometry>
+      </collision>
+      <inertial>
+        <origin xyz="0.04029922252 -0.00098556287 -0.00018415947"/>
+        <mass value="0.37100000"/>
+        <inertia ixx="0.00025425095366" ixy="-0.00000045021116" ixz="-0.00000018765570" iyy="0.00024792762707" iyz="0.00000000815247" izz="0.00038245308001"/>
+      </inertial>
+    </link>
+    <xacro:RefLink ref="robot${id}/link6"/>
+    <!-- Joint 6 -->
+    <joint name="robot${id}/joint6" type="revolute">
+      <parent link="robot${id}/link6"/>
+      <child link="robot${id}/link7"/>
+      <origin xyz="0.06300 0.04500 0.00000" rpy="0 0 0"/>
+      <axis xyz="0 1 0"/>
+      <limit velocity="3.03687" effort="100" lower="${-pi*0.5}" upper="${pi*0.5}" />
+      <dynamics damping="0.7"/>
+    </joint>
+    <xacro:SimpleTransmissionPosition n="6" joint="joint6" id="${id}" />
+        <!-- link 6 -->
+    <link name="robot${id}/link7">
+      <visual>
+        <origin xyz="-0.034 -0.098 -0.028" rpy="0 0 0"/>
+        <geometry>
+          <mesh filename="package://papras_description/meshes/link6_papras.stl" scale="0.001 0.001 0.001"/>
+        </geometry>
+        <material name="grey"/>
+      </visual>
+      <collision>
+        <origin xyz="-0.034 -0.098 -0.028" rpy="0 0 0"/>
+        <geometry>
+          <mesh filename="package://papras_description/meshes/link6_papras_simple.stl" scale="0.001 0.001 0.001"/>
+        </geometry>
+      </collision>
+      <inertial>
+        <origin xyz="${-0.034+ 0.08626593672} ${-0.098 + 0.05359265979} ${-0.028 + 0.02722564800}"/>
+        <mass value="0.38500000"/>
+        <inertia ixx="0.00032088715022" ixy="0.00000000348043" ixz="-0.00000000156396" iyy="0.00056261623134" iyz="-0.00000000024514" izz="0.00074173273605"/>
+      </inertial>
+    </link>
+    <xacro:RefLink ref="robot${id}/link7"/>
+        <!-- Joint 7 -->
+    <joint name="robot${id}/joint7" type="revolute">
+      <parent link="robot${id}/link7"/>
+      <child link="robot${id}/end_link"/>
+      <origin xyz="0.12300 -0.04500 0.00000" rpy="0 0 0"/>
+      <axis xyz="1 0 0"/>
+      <limit velocity="3.03687" effort="100" lower="${-pi*1.0}" upper="${pi*1.0}" />
+      <dynamics damping="0.7"/>
+    </joint>
+    <xacro:SimpleTransmissionPosition n="7" joint="joint7" id="${id}" />
+        <!-- end link -->
+    <link name="robot${id}/end_link">
+      <visual>
+        <origin xyz="0.0 0.0 0.0" rpy="0 0 0" />
+        <geometry>
+          <mesh filename="package://papras_description/meshes/end_link.stl" scale="0.001 0.001 0.001"/>
+        </geometry>
+        <material name="grey"/>
+      </visual>
+      <collision>
+        <origin xyz="0.0 0.0 0.0" rpy="0 0 0" />
+        <geometry>
+          <mesh filename="package://papras_description/meshes/end_link.stl" scale="0.001 0.001 0.001"/>
+        </geometry>
+      </collision>
+      <inertial>
+        <origin xyz="0.00337 0.00000 0.00000" rpy="0 0 0"/>
+        <mass value="0.01919"/>
+        <!-- <inertia ixx="1.0" ixy="0.0" ixz="0.0" iyy="1.0" iyz="0.0" izz="1.0" /> -->
+        <inertia ixx="0.00000938" ixy="0.0" ixz="0.0" iyy="0.00000338" iyz="0.0" izz="0.00000635" />
+      </inertial>
+    </link>
+    <xacro:RefLink ref="robot${id}/end_link"/>
+  </xacro:macro>
+  <xacro:macro name="papras_arm_7dof_metal" params="id">
+      <!-- link 1 -->
+      <link name="robot${id}/link1">
+        <visual>
+          <origin xyz="0 0 0" rpy="0 0 0"/>
+          <geometry>
+            <mesh filename="package://papras_description/meshes/link1.stl" scale="0.001 0.001 0.001"/>
+          </geometry>
+          <material name="grey"/>
+        </visual>
+        <collision>
+          <origin xyz="0 0 0" rpy="0 0 0"/>
+          <geometry>
+            <mesh filename="package://papras_description/meshes/link1.stl" scale="0.001 0.001 0.001"/>
+          </geometry>
+        </collision>
+        <inertial>
+          <origin xyz="-0.00205616406 0.00000000 0.07012969338"/>
+          <mass value="0.91200000"/>
+          <inertia ixx="0.00140582306367" ixy="0.00000000" ixz="0.00000000" iyy="0.00140582097352" iyz="-0.00000000" izz="0.00043779331105"/>
+        </inertial>
+      </link>
+      <xacro:RefLink ref="robot${id}/link1"/>
+        <!-- Joint 1 -->
+      <joint name="robot${id}/joint1" type="revolute">
+        <parent link="robot${id}/link1"/>
+        <child link="robot${id}/link2"/>
+        <origin xyz="0.0 0.0 0.126" rpy="0 0 0"/>
+        <axis xyz="0 0 1"/>
+        <limit velocity="3.03687" effort="100" lower="${-pi*1.0}" upper="${pi*1.0}" />
+        <dynamics damping="0.7"/>
+      </joint>
+      <xacro:SimpleTransmissionPosition n="1" joint="joint1" id="${id}" />
+      <!-- link 2 -->
+      <link name="robot${id}/link2">
+        <visual>
+          <origin xyz="0 0 0" rpy="0 0 0"/>
+          <geometry>
+            <mesh filename="package://papras_description/meshes/link2.stl" scale="0.001 0.001 0.001"/>
+          </geometry>
+          <material name="grey"/>
+        </visual>
+        <collision>
+          <origin xyz="0 0 0" rpy="0 0 0"/>
+          <geometry>
+            <mesh filename="package://papras_description/meshes/link2.stl" scale="0.001 0.001 0.001"/>
+          </geometry>
+        </collision>
+        <inertial>
+          <origin xyz="-0.00000000001 -0.01570756882 0.02819237930"/>
+          <mass value="0.88500000"/>
+          <inertia ixx="0.00155754725347" ixy="-0.00000000" ixz="-0.00000000" iyy="0.00048405544236" iyz="-0.00000173296990" izz="0.00154667193282"/>
+        </inertial>
+      </link>
+      <xacro:RefLink ref="robot${id}/link2"/>
+      <!-- Joint 2 -->
+      <joint name="robot${id}/joint2" type="revolute">
+        <parent link="robot${id}/link2"/>
+        <child link="robot${id}/link3"/>
+        <origin xyz="0.0 0.00 0.033" rpy="${pi/2.0} ${-pi/2.0} 0"/>
+        <axis xyz="0 0 1"/>
+        <limit velocity="3.03687" effort="100" lower="-2.0" upper="2.0" />
+        <dynamics damping="0.7"/>
+      </joint>
+      <xacro:SimpleTransmissionPosition n="2" joint="joint2" id="${id}" />
+      <!-- link 2 -->
+      <link name="robot${id}/link3">
+        <visual>
+          <origin xyz="0.0 0.0 0.0" rpy="0 0 0"/>
+          <geometry>
+            <mesh filename="package://papras_description/meshes/7dof/link3.stl"/>
+          </geometry>
+          <material name="grey"/>
+        </visual>
+        <collision>
+          <origin xyz="0 0 0" rpy="0 0 0"/>
+          <geometry>
+            <mesh filename="package://papras_description/meshes/7dof/link3.stl"/>
+          </geometry>
+        </collision>
+        <inertial>
+          <origin xyz="0.10300488 0.00026160 0.00111164"/>
+          <mass value="1.01000000"/>
+          <inertia ixx="0.00182373" ixy="-0.00000000" ixz="-0.00000526" iyy="0.00433189" iyz="0.00000000" izz="0.00310084"/>
+        </inertial>
+      </link>
+      <xacro:RefLink ref="robot${id}/link3"/>
+      <!-- Joint 2 -->
+      <joint name="robot${id}/joint3" type="revolute">
+        <parent link="robot${id}/link3"/>
+        <child link="robot${id}/link4"/>
+        <origin xyz="0.156382198147594 0 0.000400000000010851" rpy="0 ${-pi/2.0} ${-pi/2.0}"/>
+        <axis xyz="0 1 0"/>
+        <limit velocity="3.03687" effort="100" lower="-${pi}" upper="${pi}" />
+        <dynamics damping="0.7"/>
+      </joint>
+      <xacro:SimpleTransmissionPosition n="3" joint="joint3" id="${id}" />
+          <!-- link 2 -->
+      <link name="robot${id}/link4">
+        <visual>
+          <origin xyz="0.0 0.0 0.0" rpy="0 0 0"/>
+          <geometry>
+            <mesh filename="package://papras_description/meshes/7dof/link4.stl"/>
+          </geometry>
+          <material name="grey"/>
+        </visual>
+        <collision>
+          <origin xyz="0 0 0" rpy="0 0 0"/>
+          <geometry>
+            <mesh filename="package://papras_description/meshes/7dof/link4.stl"/>
+          </geometry>
+        </collision>
+        <inertial>
+          <origin xyz="-0.00205466 0.07035925 0.01546531"/>
+          <mass value="0.96600000"/>
+          <inertia ixx="0.00180447" ixy="0.00000423" ixz="0.00000322" iyy="0.00132106" iyz="-0.00029745" izz="0.00211226"/>
+        </inertial>
+      </link>
+      <xacro:RefLink ref="robot${id}/link4"/>
+      <!-- Joint 3 -->
+      <joint name="robot${id}/joint4" type="revolute">
+        <parent link="robot${id}/link4"/>
+        <child link="robot${id}/link5"/>
+        <origin xyz="0.0575 0.10761780185239 0.0300000000000553" rpy="${pi} ${-pi/2.0} ${pi/2.0}"/>
+        <axis xyz="0 1 0"/>
+        <limit velocity="3.03687" effort="100" lower="${-pi*1.0}" upper="1.51" />
+        <dynamics damping="0.7"/>
+      </joint>
+      <xacro:SimpleTransmissionPosition n="4" joint="joint4" id="${id}" />
+      <!-- link 5 -->
+      <link name="robot${id}/link5">
+        <visual>
+          <origin xyz="0 0 0" rpy="0 0 0"/>
+          <geometry>
+            <mesh filename="package://papras_description/meshes/link4.stl" scale="0.001 0.001 0.001"/>
+          </geometry>
+          <material name="grey"/>
+        </visual>
+        <collision>
+          <origin xyz="0 0 0" rpy="0 0 0"/>
+          <geometry>
+            <mesh filename="package://papras_description/meshes/link4.stl" scale="0.001 0.001 0.001"/>
+          </geometry>
+        </collision>
+        <inertial>
+          <origin xyz="0 0 0"/>
+          <!-- <origin xyz="${0.277-0.09327796} 0.06664315 0.05240824" rpy="0 0 3.14"/>                                                                   -->
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