Commit message: roomba urdf, moveit package, working in sim with joystick option

File: papras_utils/create_robot/create_description/urdf/create_base.urdf.xacro (robot description, xacro)
@@ -37,5 +37,5 @@
         <box size="0.001 0.001 0.001" />
       </geometry>
-      <material name="Green" />
+      <material name="green" />
     </visual>
     <collision>
@@ -101,5 +101,5 @@
     </link>
     <joint name="base_footprint_joint" type="fixed">
-      <origin xyz="0 0 0.017" rpy="0 0 0" />
+      <origin xyz="0 0 0.01" rpy="0 0 0" />
       <parent link="base_footprint" />
       <child link="base_link" />

File: papras_utils/create_robot/create_description/urdf/create_base_gazebo.urdf.xacro (robot description, xacro)
@@ -16,4 +16,6 @@
         <odometryFrame>roomba/odom</odometryFrame>
         <robotBaseFrame>roomba/base_footprint</robotBaseFrame>
+        <!-- <publishWheelTF>true</publishWheelTF> -->
+        <publishWheelJointState>true</publishWheelJointState>
       </plugin>
       <plugin name="p3d_base_controller" filename="libgazebo_ros_p3d.so">
