Commit message: checked with hw

File: papras_simple_demo/urdf/simple_robot.urdf.xacro (robot description, xacro)
@@ -18,6 +18,6 @@
   </joint>
   <xacro:papras_arm_7dof id="1"/>
-  <xacro:papras_gripper id="1"/>
-  <xacro:papras_camera id="1"/>
+  <xacro:rh_p12_rn_gripper id="1"/>
+  <xacro:papras_camera_rh12 id="1"/>
   <xacro:papras_ros2_control_hw systems="${systems}" system_prefix="${system_prefix}" arm_ids= "${arm_ids}"
                             usb_port_location='$(arg usb_port)' baud_rate_val="$(arg baud_rate)" yaml_file="${yaml_file}"/>

File: papras_simple_moveit_config/config/simple_robot.ros2_control.xacro (robot description, xacro)
@@ -2,5 +2,5 @@
 <robot xmlns:xacro="http://www.ros.org/wiki/xacro">
     <xacro:macro name="simple_robot_ros2_control" params="name initial_positions_file">
-        <xacro:property name="initial_positions" value="${xacro.load_yaml(initial_positions_file)['initial_positions']}"/>
+        <xacro:property name="initial_positions" value="${load_yaml(initial_positions_file)['initial_positions']}"/>
         <ros2_control name="${name}" type="system">
             <hardware>
@@ -14,4 +14,5 @@
                 </state_interface>
                 <state_interface name="velocity"/>
+                <state_interface name="effort"/>
             </joint>
             <joint name="robot1/joint2">
@@ -21,4 +22,5 @@
                 </state_interface>
                 <state_interface name="velocity"/>
+                <state_interface name="effort"/>
             </joint>
             <joint name="robot1/joint3">
@@ -28,4 +30,5 @@
                 </state_interface>
                 <state_interface name="velocity"/>
+                <state_interface name="effort"/>
             </joint>
             <joint name="robot1/joint4">
@@ -35,4 +38,5 @@
                 </state_interface>
                 <state_interface name="velocity"/>
+                <state_interface name="effort"/>
             </joint>
             <joint name="robot1/joint5">
@@ -42,4 +46,5 @@
                 </state_interface>
                 <state_interface name="velocity"/>
+                <state_interface name="effort"/>
             </joint>
             <joint name="robot1/joint6">
@@ -49,4 +54,5 @@
                 </state_interface>
                 <state_interface name="velocity"/>
+                <state_interface name="effort"/>
             </joint>
             <joint name="robot1/joint7">
@@ -56,4 +62,5 @@
                 </state_interface>
                 <state_interface name="velocity"/>
+                <state_interface name="effort"/>
             </joint>
             <joint name="robot1/gripper">
@@ -63,4 +70,5 @@
                 </state_interface>
                 <state_interface name="velocity"/>
+                <state_interface name="effort"/>
             </joint>
         </ros2_control>
